File: Controls-PedalsDaughter.kicad_sch (KiCad schematic)
At the start: 21 parts, among them J2 Accel Pos. Sensor, J3 PeripheralCANConnector, J4 Conn_01x02, J5 PeripheralCANConnector, U1 RI3-1205S, U2 PeripheralSOM

Commit message: Added comments
Connections:
- net GND: no longer C1.2, D5.2 (A), J4.1 (Pin_1), R1.2
- net GNDPWR: now also C1.2, D5.2 (A), J4.1 (Pin_1), R1.2
Other:
- note added: "Neads to be isolated :)"
Changed lines of the file:
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@@
 		)
 	)
+	(text "Neads to be isolated :)\n"
+		(exclude_from_sim no)
+		(at 223.266 136.144 0)
+		(effects
+			(font
+				(size 1.27 1.27)
+			)
+		)
+	)
 	(text "Break Sensor to ADC"
 		(exclude_from_sim no)
-		(at 177.038 116.078 0)
+		(at 183.134 117.348 0)
 		(effects
 			(font
@@
 	)
 	(symbol
+		(lib_id "power:GNDPWR")
+		(at 166.37 140.97 0)
+		(unit 1)
+		(exclude_from_sim no)
+		(in_bom yes)
+		(on_board yes)
+		(dnp no)
+		(fields_autoplaced yes)
+		(property "Reference" "#PWR09"
+			(at 166.37 146.05 0)
+			(effects
+				(font
+					(size 1.27 1.27)
+				)
+				(hide yes)
+			)
+		)
+		(property "Value" "GNDPWR"
+			(at 166.243 144.78 0)
+			(effects
+				(font
+					(size 1.27 1.27)
+				)
+			)
+		)
+		(property "Footprint" ""
+			(at 166.37 142.24 0)
+			(effects
+				(font
+					(size 1.27 1.27)
+				)
+				(hide yes)
+			)
+		)
+		(property "Datasheet" ""
+			(at 166.37 142.24 0)
+			(effects
+				(font
+					(size 1.27 1.27)
+				)
+				(hide yes)
+			)
+		)
+		(property "Description" "Power symbol creates a global label with name \"GNDPWR\" , global ground"
+			(at 166.37 140.97 0)
+			(effects
+				(font
+					(size 1.27 1.27)
+				)
+				(hide yes)
+			)
+		)
+		(pin "1"
+		)
+		(instances
+			(project "Controls-PedalsDaughter"
+				(path "/30d77876-714b-4f1b-9bad-b74eb43ddcf6"
+					(reference "#PWR09")
+					(unit 1)
+				)
+			)
+		)
+	)
+	(symbol
 		(lib_id "power:+5V")
 		(at 66.04 130.81 270)
@@
 	)
 	(symbol
-		(lib_id "power:+5V")
-		(at 92.71 125.73 0)
+		(lib_id "power:GNDPWR")
+		(at 173.99 143.51 0)
 		(unit 1)
 		(exclude_from_sim no)
@@
 		(on_board yes)
 		(dnp no)
-		(property "Reference" "#PWR018"
-			(at 92.71 129.54 0)
+		(fields_autoplaced yes)
+		(property "Reference" "#PWR010"
+			(at 173.99 148.59 0)
 			(effects
 				(font
@@
 			)
 		)
-		(property "Value" "+3.3V"
-			(at 92.71 120.65 0)
+		(property "Value" "GNDPWR"
+			(at 173.863 147.32 0)
 			(effects
 				(font
@@
 		)
 		(property "Footprint" ""
-			(at 92.71 125.73 0)
+			(at 173.99 144.78 0)
 			(effects
 				(font
@@
 		)
 		(property "Datasheet" ""
-			(at 92.71 125.73 0)
+			(at 173.99 144.78 0)
 			(effects
 				(font
@@
 			)
 		)
-		(property "Description" "Power symbol creates a global label with name \"+5V\""
-			(at 92.71 125.73 0)
+		(property "Description" "Power symbol creates a global label with name \"GNDPWR\" , global ground"
+			(at 173.99 143.51 0)
 			(effects
 				(font
@@
 			(project "Controls-PedalsDaughter"
 				(path "/30d77876-714b-4f1b-9bad-b74eb43ddcf6"
-					(reference "#PWR018")
+					(reference "#PWR010")
 					(unit 1)
 				)
@@
 	)
 	(symbol
-		(lib_id "power:GND")
-		(at 195.58 143.51 0)
+		(lib_id "power:+5V")
+		(at 92.71 125.73 0)
 		(unit 1)
 		(exclude_from_sim no)
@@
 		(on_board yes)
 		(dnp no)
-		(fields_autoplaced yes)
-		(property "Reference" "#PWR013"
-			(at 195.58 149.86 0)
+		(property "Reference" "#PWR018"
+			(at 92.71 129.54 0)
 			(effects
 				(font
@@
 			)
 		)
-		(property "Value" "GND"
-			(at 195.58 148.59 0)
+		(property "Value" "+3.3V"
+			(at 92.71 120.65 0)
 			(effects
 				(font
@@
 		)
 		(property "Footprint" ""
-			(at 195.58 143.51 0)
+			(at 92.71 125.73 0)
 			(effects
 				(font
@@
 		)
 		(property "Datasheet" ""
-			(at 195.58 143.51 0)
+			(at 92.71 125.73 0)
 			(effects
 				(font
@@
 			)
 		)
-		(property "Description" "Power symbol creates a global label with name \"GND\" , ground"
-			(at 195.58 143.51 0)
+		(property "Description" "Power symbol creates a global label with name \"+5V\""
+			(at 92.71 125.73 0)
 			(effects
 				(font
@@
 			(project "Controls-PedalsDaughter"
 				(path "/30d77876-714b-4f1b-9bad-b74eb43ddcf6"
-					(reference "#PWR013")
+					(reference "#PWR018")
 					(unit 1)
 				)
@@
 	)
 	(symbol
-		(lib_id "power:GND")
-		(at 166.37 140.97 0)
+		(lib_id "power:GNDPWR")
+		(at 195.58 143.51 0)
 		(unit 1)
 		(exclude_from_sim no)
@@
 		(dnp no)
 		(fields_autoplaced yes)
-		(property "Reference" "#PWR09"
-			(at 166.37 147.32 0)
+		(property "Reference" "#PWR013"
+			(at 195.58 148.59 0)
 			(effects
 				(font
@@
 			)
 		)
-		(property "Value" "GND"
-			(at 166.37 146.05 0)
+		(property "Value" "GNDPWR"
+			(at 195.453 147.32 0)
 			(effects
 				(font
@@
 		)
 		(property "Footprint" ""
-			(at 166.37 140.97 0)
+			(at 195.58 144.78 0)
 			(effects
 				(font
@@
 		)
 		(property "Datasheet" ""
-			(at 166.37 140.97 0)
+			(at 195.58 144.78 0)
 			(effects
 				(font
@@
 			)
 		)
-		(property "Description" "Power symbol creates a global label with name \"GND\" , ground"
-			(at 166.37 140.97 0)
+		(property "Description" "Power symbol creates a global label with name \"GNDPWR\" , global ground"
+			(at 195.58 143.51 0)
 			(effects
 				(font
@@
 			(project "Controls-PedalsDaughter"
 				(path "/30d77876-714b-4f1b-9bad-b74eb43ddcf6"
-					(reference "#PWR09")
+					(reference "#PWR013")
 					(unit 1)
 				)
@@
 	)
 	(symbol
+		(lib_id "power:GNDPWR")
+		(at 184.15 143.51 0)
+		(unit 1)
+		(exclude_from_sim no)
+		(in_bom yes)
+		(on_board yes)
+		(dnp no)
+		(fields_autoplaced yes)
+		(property "Reference" "#PWR011"
+			(at 184.15 148.59 0)
+			(effects
+				(font
+					(size 1.27 1.27)
+				)
+				(hide yes)
+			)
+		)
+		(property "Value" "GNDPWR"
+			(at 184.023 147.32 0)
+			(effects
+				(font
+					(size 1.27 1.27)
+				)
+			)
+		)
+		(property "Footprint" ""
+			(at 184.15 144.78 0)
+			(effects
+				(font
+					(size 1.27 1.27)
+				)
+				(hide yes)
+			)
+		)
+		(property "Datasheet" ""
+			(at 184.15 144.78 0)
+			(effects
+				(font
+					(size 1.27 1.27)
+				)
+				(hide yes)
+			)
+		)
+		(property "Description" "Power symbol creates a global label with name \"GNDPWR\" , global ground"
+			(at 184.15 143.51 0)
+			(effects
+				(font
+					(size 1.27 1.27)
+				)
+				(hide yes)
+			)
+		)
+		(pin "1"
+		)
+		(instances
+			(project "Controls-PedalsDaughter"
+				(path "/30d77876-714b-4f1b-9bad-b74eb43ddcf6"
+					(reference "#PWR011")
+					(unit 1)
+				)
+			)
+		)
+	)
+	(symbol
 		(lib_id "Device:D")
 		(at 92.71 137.16 270)
@@
 			)
 		)
-		(property "Datasheet" "~"
+		(property "Datasheet" "https://kulite.com//assets/media/2017/06/ETL-200-375.pdf"
 			(at 161.29 138.43 0)
 			(effects
@@
 	(symbol
 		(lib_id "power:GND")
-		(at 173.99 143.51 0)
-		(unit 1)
-		(exclude_from_sim no)
-		(in_bom yes)
-		(on_board yes)
-		(dnp no)
-		(fields_autoplaced yes)
-		(property "Reference" "#PWR010"
-			(at 173.99 149.86 0)
-			(effects
-				(font
-					(size 1.27 1.27)
-				)
-				(hide yes)
-			)
-		)
-		(property "Value" "GND"
-			(at 173.99 148.59 0)
-			(effects
-				(font
-					(size 1.27 1.27)
-				)
-			)
-		)
-		(property "Footprint" ""
-			(at 173.99 143.51 0)
-			(effects
-				(font
-					(size 1.27 1.27)
-				)
-				(hide yes)
-			)
-		)
-		(property "Datasheet" ""
-			(at 173.99 143.51 0)
-			(effects
-				(font
-					(size 1.27 1.27)
-				)
-				(hide yes)
-			)
-		)
-		(property "Description" "Power symbol creates a global label with name \"GND\" , ground"
-			(at 173.99 143.51 0)
-			(effects
-				(font
-					(size 1.27 1.27)
-				)
-				(hide yes)
-			)
-		)
-		(pin "1"
-		)
-		(instances
-			(project "Controls-PedalsDaughter"
-				(path "/30d77876-714b-4f1b-9bad-b74eb43ddcf6"
-					(reference "#PWR010")
-					(unit 1)
-				)
-			)
-		)
-	)
-	(symbol
-		(lib_id "power:GND")
 		(at 92.71 140.97 0)
 		(unit 1)
@@
 					(unit 1)
 				)
-			)
-		)
-	)
-	(symbol
-		(lib_id "power:GND")
-		(at 184.15 143.51 0)
-		(unit 1)
-		(exclude_from_sim no)
-		(in_bom yes)
-		(on_board yes)
-		(dnp no)
-		(fields_autoplaced yes)
-		(property "Reference" "#PWR011"
-			(at 184.15 149.86 0)
-			(effects
-				(font
-					(size 1.27 1.27)
-				)
-				(hide yes)
-			)
-		)
-		(property "Value" "GND"
-			(at 184.15 148.59 0)
-			(effects
-				(font
-					(size 1.27 1.27)
-				)
-			)
-		)
-		(property "Footprint" ""
-			(at 184.15 143.51 0)
-			(effects
-				(font
-					(size 1.27 1.27)
-				)
-				(hide yes)
-			)
-		)
-		(property "Datasheet" ""
-			(at 184.15 143.51 0)
-			(effects
-				(font
-					(size 1.27 1.27)
-				)
-				(hide yes)
-			)
-		)
-		(property "Description" "Power symbol creates a global label with name \"GND\" , ground"
-			(at 184.15 143.51 0)
-			(effects
-				(font
-					(size 1.27 1.27)
-				)
-				(hide yes)
-			)
-		)
-		(pin "1"
-		)
-		(instances
-			(project "Controls-PedalsDaughter"
-				(path "/30d77876-714b-4f1b-9bad-b74eb43ddcf6"
-					(reference "#PWR011")
-					(unit 1)
-				)

Commit message: Added isolation n stuff
Parts:
- removed D5: D, symbol Device:D
- added C10: 1nF, Capacitor_SMD:C_0805_2012Metric, symbol Device:C
- added C11: 100nF, Capacitor_SMD:C_0805_2012Metric, symbol Device:C
- added C12: 0.1uf, symbol Device:C
- added C4, C5: 10uf, symbol Device:C
- added C6, C9: 100uF, symbol Device:C
- added C7, C8: 1uF, symbol Device:C
- added D6: SMD_805, symbol Device:LED
- added D7: PESD15VL1BA, Diode_SMD:D_SOD-323, symbol Diode:SD12_SOD323
- added R3: 1.5k, symbol Device:R_US
- added U3: TLV9301xDCK, Package_TO_SOT_SMD:SOT-353_SC-70-5, symbol Amplifier_Operational:TLV9301xDCK
- added U4: AMC1300BDWV, Package_SO:SOIC-8_7.5x5.85mm_P1.27mm, symbol Amplifier_Difference:AMC1300BDWV
- added U5: TLV70130DBVR, UTSVT_Power:TLV70130DBVR, symbol 2025-01-18_20-51-31:TLV70130DBVR
- C1: value 1F -> 1nF
- C2: value 10u -> 10uF
- C3: value C -> 1uf
- D1: value TVS -> MBR; footprint Diode_SMD:D_SOD-323 -> (none); P/N (none) -> MBR0520LT1G
- D2, D3, D4: value D -> MBR; P/N (none) -> MBR0520LT1G
- R1: value 160 -> 20
Connections:
- net +12V: now also C11.1, D7.2 (A2), U5.3 (IN); no longer D1.1 (K)
- net +3.3V: now also D1.1 (K), D3.1 (K); no longer D2.1 (K), D4.1 (K)
- net +5V: now also C12.2, C4.1, C5.1, R3.1, U3.5 (V+)
- net Accel: now also D1.2 (A), D2.1 (K), U3.3 (-), U3.4; no longer D2.2 (A), D3.1 (K), R2.1, R4.1
- net Brake: now also D3.2 (A), D4.1 (K), U4.7 (+); no longer D4.2 (A), J4.2 (Pin_2), R1.1
- net GND: now also C1.2, D2.2 (A), D4.2 (A), C12.1, C4.2, C5.2, C8.2, C9.2, D6.1 (K), U3.2 (V-), U4.5 (V-), U4.6 (-); no longer D3.2 (A)
- net GNDPWR: now also C10.2, C11.2, C6.2, C7.2, D7.1 (A1), U4.3 (-), U4.4 (V-), U5.2 (GND); no longer C1.2, D1.2 (A)
- new net: R2.1, R4.1, U3.1 (+)
- new net: D6.2 (A), R3.2
- new net +3V3: C8.1, C9.1, U4.8 (V+)
- new net +3V3PWR: C10.1, C6.1, C7.1, U4.1 (V+), U5.1 (OUT)
- new net INP: J4.2 (Pin_2), R1.1, U4.2 (+)
- no-connect marks 15 -> 17
Other:
- note added: "20ma -> ~0.4V (*8.2) -> 3.28v"
- note added: "3V3 Pwr for Isolated Amp"
- note added: "Accel Pedal"
- note added: "Break Pedal"
- note added: "Isolated Amp"
- note added: "PSOM"
- note added: "Pedal Board"
- note added: "Power"
- note added: "Pwr LED"
- note added: "bypass :)"
- note added: "x8.2 gain"
- note removed: "Brake Line Fluid Sensor"
- note removed: "Break Sensor to ADC"
- note removed: "Neads to be isolated :)"
- moved on the sheet: C2, J2, J3, J4, J5, R1, R2, R4, TP1, TP2, TP3, TP4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

Commit message: wop
Parts:
- C3: value 1uf -> 1nf
Changed lines of the file:
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@@
 			)
 		)
-		(property "Value" "1uf"
+		(property "Value" "1nf"
 			(at 110.998 140.97 0)
 			(effects

Commit message: Assigned footprints for Power Sector
Parts:
- C4, C5: footprint (none) -> Capacitor_SMD:C_0805_2012Metric
- D6: value SMD_805 -> SMD_0805; footprint (none) -> Diode_SMD:D_0805_2012Metric
- R3: footprint (none) -> Resistor_SMD:R_0805_2012Metric
Changed lines of the file:
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@@
 			)
 		)
-		(property "Footprint" ""
+		(property "Footprint" "Capacitor_SMD:C_0805_2012Metric"
 			(at 134.3152 57.15 0)
 			(effects
@@
 			)
 		)
-		(property "Datasheet" "~"
+		(property "Datasheet" "https://www.mouser.com/datasheet/2/396/taiyo_yuden_12132018_mlcc11_hq_e-1510082.pdf"
 			(at 133.35 53.34 0)
 			(effects
@@
 			)
 		)
-		(property "Footprint" ""
+		(property "Footprint" "Capacitor_SMD:C_0805_2012Metric"
 			(at 121.6152 57.15 0)
 			(effects
@@
 			)
 		)
-		(property "Datasheet" "~"
+		(property "Datasheet" "https://www.mouser.com/datasheet/2/396/taiyo_yuden_12132018_mlcc11_hq_e-1510082.pdf"
 			(at 120.65 53.34 0)
 			(effects
@@
 			)
 		)
-		(property "Value" "SMD_805"
+		(property "Value" "SMD_0805"
 			(at 129.54 87.9474 90)
 			(effects
@@
 			)
 		)
-		(property "Footprint" ""
+		(property "Footprint" "Diode_SMD:D_0805_2012Metric"
 			(at 125.73 85.09 0)
 			(effects
@@
 			)
 		)
-		(property "Footprint" ""
+		(property "Footprint" "Resistor_SMD:R_0805_2012Metric"
 			(at 126.746 77.724 90)
 			(effects
@@
 			)
 		)
-		(property "Datasheet" "~"
+		(property "Datasheet" "https://www.vishay.com/docs/20035/dcrcwe3.pdf"
 			(at 125.73 77.47 0)
 			(effects

Commit message: Assigned footprints
Parts:
- C1, C12, C3, C6, C7, C8, C9: footprint (none) -> Capacitor_SMD:C_0805_2012Metric
- C2: footprint UTSVT_Passive:C_2220_5750Metric -> Capacitor_SMD:C_0805_2012Metric
- D1, D2, D3, D4: footprint (none) -> Diode_SMD:D_0805_2012Metric
- J2: footprint (none) -> Connector_Molex:Molex_Micro-Fit_3.0_43045-1200_2x06_P3.00mm_Horizontal
- J4: footprint (none) -> Connector_Molex:Molex_Micro-Fit_3.0_43045-0200_2x01_P3.00mm_Horizontal
- R1, R2, R4: footprint (none) -> Resistor_SMD:R_0805_2012Metric
Changed lines of the file:
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@@
 			)
 		)
-		(property "Footprint" ""
+		(property "Footprint" "Capacitor_SMD:C_0805_2012Metric"
 			(at 106.9848 135.89 0)
 			(effects
@@
 			)
 		)
-		(property "Footprint" ""
+		(property "Footprint" "Capacitor_SMD:C_0805_2012Metric"
 			(at 188.9252 163.83 0)
 			(effects
@@
 			)
 		)
-		(property "Footprint" ""
+		(property "Footprint" "Capacitor_SMD:C_0805_2012Metric"
 			(at 229.5652 163.83 0)
 			(effects
@@
 			)
 		)
-		(property "Footprint" ""
+		(property "Footprint" "Connector_Molex:Molex_Micro-Fit_3.0_43045-1200_2x06_P3.00mm_Horizontal"
 			(at 57.15 133.35 0)
 			(effects
@@
 			)
 		)
-		(property "Footprint" ""
+		(property "Footprint" "Diode_SMD:D_0805_2012Metric"
 			(at 237.49 125.73 0)
 			(effects
@@
 			)
 		)
-		(property "Footprint" ""
+		(property "Footprint" "Resistor_SMD:R_0805_2012Metric"
 			(at 75.946 134.366 90)
 			(effects
@@
 			)
 		)
-		(property "Footprint" ""
+		(property "Footprint" "Resistor_SMD:R_0805_2012Metric"
 			(at 82.296 138.684 90)
 			(effects
@@
 			)
 		)
-		(property "Footprint" ""
+		(property "Footprint" "Capacitor_SMD:C_0805_2012Metric"
 			(at 93.98 126.6952 0)
 			(effects
@@
 			)
 		)
-		(property "Footprint" ""
+		(property "Footprint" "Diode_SMD:D_0805_2012Metric"
 			(at 116.84 139.7 0)
 			(effects
@@
 			)
 		)
-		(property "Footprint" ""
+		(property "Footprint" "Resistor_SMD:R_0805_2012Metric"
 			(at 164.846 157.734 90)
 			(effects
@@
 			)
 		)
-		(property "Footprint" ""
+		(property "Footprint" "Capacitor_SMD:C_0805_2012Metric"
 			(at 182.5752 163.83 0)
 			(effects
@@
 			)
 		)
-		(property "Footprint" ""
+		(property "Footprint" "Connector_Molex:Molex_Micro-Fit_3.0_43045-0200_2x01_P3.00mm_Horizontal"
 			(at 151.13 156.21 0)
 			(effects
@@
 			)
 		)
-		(property "Footprint" ""
+		(property "Footprint" "Diode_SMD:D_0805_2012Metric"
 			(at 237.49 118.11 0)
 			(effects
@@
 			)
 		)
-		(property "Footprint" ""
+		(property "Footprint" "Capacitor_SMD:C_0805_2012Metric"
 			(at 239.7252 163.83 0)
 			(effects
@@
 			)
 		)
-		(property "Footprint" ""
+		(property "Footprint" "Diode_SMD:D_0805_2012Metric"
 			(at 116.84 132.08 0)
 			(effects
@@
 			)
 		)
-		(property "Footprint" "UTSVT_Passive:C_2220_5750Metric"
+		(property "Footprint" "Capacitor_SMD:C_0805_2012Metric"
 			(at 58.1152 74.93 0)
 			(effects
@@
 			)
 		)
-		(property "Footprint" ""
+		(property "Footprint" "Capacitor_SMD:C_0805_2012Metric"
 			(at 225.7552 129.54 0)
 			(effects

Commit message: Added P/Ns
Parts:
- C1, C10, C12, C2, C3, C4, C5, C6, C7, C8, C9, D6, R3, R4: P/N (none) -> pickle
- C11: P/N C0805C104M5RACTU -> pickle
- J2: footprint Connector_Molex:Molex_Micro-Fit_3.0_43045-1200_2x06_P3.00mm_Horizontal -> Connector_Molex:Molex_Micro-Fit_3.0_43045-0612_2x03_P3.00mm_Vertical; P/N (none) -> 430450626
- J4: footprint Connector_Molex:Molex_Micro-Fit_3.0_43045-0200_2x01_P3.00mm_Horizontal -> Connector_Molex:Molex_Micro-Fit_3.0_43045-0212_2x01_P3.00mm_Vertical; P/N (none) -> 430450200
- R1: P/N (none) -> ERJ-UP6D20R0V
- R2: P/N (none) -> ERA-3ARB822V
- U1: P/N (none) -> RI3-1205S
- U3: P/N (none) -> TLV9301xDCK
- U4: P/N (none) -> AMC1300BDWV
Changed lines of the file:
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@@
 			)
 		)
+		(property "P/N" "pickle"
+			(at 107.95 139.7 0)
+			(effects
+				(font
+					(size 1.27 1.27)
+				)
+				(hide yes)
+			)
+		)
 		(pin "2"
 		)
@@
 			)
 		)
+		(property "P/N" "pickle"
+			(at 187.96 160.02 0)
+			(effects
+				(font
+					(size 1.27 1.27)
+				)
+				(hide yes)
+			)
+		)
 		(pin "2"
 		)
@@
 			)
 		)
+		(property "P/N" "AMC1300BDWV"
+			(at 210.82 160.02 0)
+			(effects
+				(font
+					(size 1.27 1.27)
+				)
+				(hide yes)
+			)
+		)
 		(pin "8"
 		)
@@
 			)
 		)
+		(property "P/N" "pickle"
+			(at 228.6 160.02 0)
+			(effects
+				(font
+					(size 1.27 1.27)
+				)
+				(hide yes)
+			)
+		)
 		(pin "2"
 		)
@@
 			)
 		)
-		(property "Footprint" "Connector_Molex:Molex_Micro-Fit_3.0_43045-1200_2x06_P3.00mm_Horizontal"
+		(property "Footprint" "Connector_Molex:Molex_Micro-Fit_3.0_43045-0612_2x03_P3.00mm_Vertical"
 			(at 57.15 133.35 0)
 			(effects
@@
 			)
 		)
+		(property "P/N" "430450626"
+			(at 57.15 133.35 0)
+			(effects
+				(font
+					(size 1.27 1.27)
+				)
+				(hide yes)
+			)
+		)
 		(pin "3"
 		)
@@
 			)
 		)
+		(property "P/N" "RI3-1205S"
+			(at 78.74 66.04 0)
+			(effects
+				(font
+					(size 1.27 1.27)
+				)
+				(hide yes)
+			)
+		)
 		(pin "1"
 		)
@@
 			)
 		)
+		(property "P/N" "pickle"
+			(at 193.04 123.19 0)
+			(effects
+				(font
+					(size 1.27 1.27)
+				)
+				(hide yes)
+			)
+		)
 		(pin "1"
 		)
@@
 			)
 		)
+		(property "P/N" "ERA-3ARB822V"
+			(at 76.2 133.35 0)
+			(effects
+				(font
+					(size 1.27 1.27)
+				)
+				(hide yes)
+			)
+		)
 		(pin "2"
 		)
@@
 			)
 		)
+		(property "P/N" "pickle"
+			(at 81.28 138.43 0)
+			(effects
+				(font
+					(size 1.27 1.27)
+				)
+				(hide yes)
+			)
+		)
 		(pin "2"
 		)
@@
 			)
 		)
+		(property "P/N" "pickle"
+			(at 133.35 53.34 0)
+			(effects
+				(font
+					(size 1.27 1.27)
+				)
+				(hide yes)
+			)
+		)
 		(pin "1"
 		)
@@
 			)
 		)
+		(property "P/N" "pickle"
+			(at 97.79 125.73 0)
+			(effects
+				(font
+					(size 1.27 1.27)
+				)
+				(hide yes)
+			)
+		)
 		(pin "2"
 		)
@@
 			)
 		)
+		(property "P/N" "pickle"
+			(at 120.65 53.34 0)
+			(effects
+				(font
+					(size 1.27 1.27)
+				)
+				(hide yes)
+			)
+		)
 		(pin "1"
 		)
@@
 			)
 		)
+		(property "P/N" "ERJ-UP6D20R0V"
+			(at 163.83 157.48 0)
+			(effects
+				(font
+					(size 1.27 1.27)
+				)
+				(hide yes)
+			)
+		)
 		(pin "2"
 		)
@@
 			)
 		)
-		(property "P/N" "C0805C104M5RACTU"
+		(property "P/N" "pickle"
 			(at 151.13 125.73 0)
 			(effects
@@
 			)
 		)
+		(property "P/N" "TLV9301xDCK"
+			(at 93.98 135.89 0)
+			(effects
+				(font
+					(size 1.27 1.27)
+				)
+				(hide yes)
+			)
+		)
 		(pin "2"
 		)
@@
 			)
 		)
+		(property "P/N" "pickle"
+			(at 181.61 160.02 0)
+			(effects
+				(font
+					(size 1.27 1.27)
+				)
+				(hide yes)
+			)
+		)
 		(pin "2"
 		)
@@
 			)
 		)
-		(property "Footprint" "Connector_Molex:Molex_Micro-Fit_3.0_43045-0200_2x01_P3.00mm_Horizontal"
+		(property "Footprint" "Connector_Molex:Molex_Micro-Fit_3.0_43045-0212_2x01_P3.00mm_Vertical"
 			(at 151.13 156.21 0)
 			(effects
@@
 			)
 		)
+		(property "P/N" "430450200"
+			(at 151.13 156.21 0)
+			(effects
+				(font
+					(size 1.27 1.27)
+				)
+				(hide yes)
+			)
+		)
 		(pin "2"
 		)
@@
 			)
 		)
+		(property "P/N" "pickle"
+			(at 125.73 85.09 0)
+			(effects
+				(font
+					(size 1.27 1.27)
+				)
+				(hide yes)
+			)
+		)
 		(pin "1"
 		)
@@
 			)
 		)
+		(property "P/N" "pickle"
+			(at 238.76 160.02 0)
+			(effects
+				(font
+					(size 1.27 1.27)
+				)
+				(hide yes)
+			)
+		)
 		(pin "2"
 		)
@@
 			)
 		)
+		(property "P/N" "pickle"
+			(at 57.15 71.12 0)
+			(effects
+				(font
+					(size 1.27 1.27)
+				)
+				(hide yes)
+			)
+		)
 		(pin "1"
 		)
@@
 			)
 		)
+		(property "P/N" "pickle"
+			(at 224.79 125.73 0)
+			(effects
+				(font
+					(size 1.27 1.27)
+				)
+				(hide yes)
+			)
+		)
 		(pin "2"
 		)
@@
 			(at 125.73 77.47 0)
 			(effects
+				(font
+					(size 1.27 1.27)
+				)
+				(hide yes)
+			)
+		)
+		(property "P/N" "pickle"
+			(at 125.73 77.47 0)
+			(effects
