File: Controls-PedalsDaughter.kicad_sch (KiCad schematic)
At the start: 35 parts, among them J2 Accel Pos. Sensor, J3 PeripheralCANConnector, J4 Conn_01x02, J5 PeripheralCANConnector, U1 RI3-1205S, U2 PeripheralSOM, U3 TLV9301xDCK, U4 AMC1300BDWV, U5 TLV70130DBVR

Commit message: Schem done, prelim pcb, added 3d models
Parts:
- added TP_3V3PWR1: +3V3PWR, TestPoint:TestPoint_Pad_1.5x1.5mm, symbol Connector:TestPoint
- U5: footprint UTSVT_Power:TLV70130DBVR -> Package_TO_SOT_SMD:SOT-353_SC-70-5
- renumbered TP1 to +12V1, TP3 to +5V1, TP4 to GND1, TP2 to GNDPWR1
Connections:
- net +12V: now also U5.1 (IN); no longer U5.3 (IN)
- net +3V3PWR: now also U5.5 (OUT), TP_3V3PWR1.1; no longer U5.1 (OUT)
- net GNDPWR: now also U5.4 (GND); no longer U5.2 (GND)
Other:
- note added: "Break sensor gives current reading 4ma - 20ma"
Changed lines of the file:
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@@
 	)
 	(junction
+		(at 190.5 119.38)
+		(diameter 0)
+		(color 0 0 0 0)
+	)
+	(junction
 		(at 127 57.15)
 		(diameter 0)
@@
 	(wire
 		(pts
-			(xy 187.96 119.38) (xy 193.04 119.38)
+			(xy 187.96 119.38) (xy 190.5 119.38)
 		)
 		(stroke
@@
 	(wire
 		(pts
+			(xy 190.5 119.38) (xy 193.04 119.38)
+		)
+		(stroke
+			(width 0)
+			(type default)
+		)
+	)
+	(wire
+		(pts
 			(xy 156.21 153.67) (xy 163.83 153.67)
 		)
@@
 		)
 	)
+	(text "Break sensor gives current\nreading 4ma - 20ma"
+		(exclude_from_sim no)
+		(at 154.178 170.434 0)
+		(effects
+			(font
+				(size 1.27 1.27)
+			)
+		)
+	)
 	(text "Based on:\nhttps://www.akao.co.uk/manuals/Link%20G4+%20Manual/nissan_vq35.htm"
 		(exclude_from_sim no)
@@
 		(on_board yes)
 		(dnp no)
-		(property "Reference" "TP3"
+		(property "Reference" "+5V1"
 			(at 104.3432 61.722 0)
 			(effects
@@
 			(project "Controls-PedalsDaughter"
 				(path "/30d77876-714b-4f1b-9bad-b74eb43ddcf6"
-					(reference "TP3")
+					(reference "+5V1")
 					(unit 1)
 				)
@@
 		(on_board yes)
 		(dnp no)
-		(property "Reference" "TP1"
+		(property "Reference" "+12V1"
 			(at 46.99 55.88 0)
 			(effects
@@
 			(project "Controls-PedalsDaughter"
 				(path "/30d77876-714b-4f1b-9bad-b74eb43ddcf6"
-					(reference "TP1")
+					(reference "+12V1")
 					(unit 1)
 				)
@@
 		(on_board yes)
 		(dnp no)
-		(property "Reference" "TP4"
+		(property "Reference" "GND1"
 			(at 104.3432 79.4258 0)
 			(effects
@@
 			(project "Controls-PedalsDaughter"
 				(path "/30d77876-714b-4f1b-9bad-b74eb43ddcf6"
-					(reference "TP4")
+					(reference "GND1")
 					(unit 1)
 				)
@@
 			)
 		)
-		(property "Footprint" "UTSVT_Power:TLV70130DBVR"
+		(property "Footprint" "Package_TO_SOT_SMD:SOT-353_SC-70-5"
 			(at 158.496 102.362 0)
 			(effects
@@
 		(on_board yes)
 		(dnp no)
-		(property "Reference" "TP2"
+		(property "Reference" "GNDPWR1"
 			(at 48.4632 78.1558 0)
 			(effects
@@
 			(project "Controls-PedalsDaughter"
 				(path "/30d77876-714b-4f1b-9bad-b74eb43ddcf6"
-					(reference "TP2")
+					(reference "GNDPWR1")
 					(unit 1)
 				)
@@
 					(unit 1)
 				)
+			)
+		)
+	)
+	(symbol
+		(lib_id "Connector:TestPoint")
+		(at 190.5 119.38 0)
+		(unit 1)
+		(exclude_from_sim no)
+		(in_bom yes)
+		(on_board yes)
+		(dnp no)
+		(property "Reference" "TP_3V3PWR1"
+			(at 189.0268 118.6942 0)
+			(effects
+				(font
+					(size 1.27 1.27)
+				)
+				(justify right)
+			)
+		)
+		(property "Value" "+3V3PWR"
+			(at 189.0268 116.3828 0)
+			(effects
+				(font
+					(size 1.27 1.27)
+				)
+				(justify right)
+			)
+		)
+		(property "Footprint" "TestPoint:TestPoint_Pad_1.5x1.5mm"
+			(at 195.58 119.38 0)
+			(effects
+				(font
+					(size 1.27 1.27)
+				)
+				(hide yes)
+			)
+		)
+		(property "Datasheet" "~"
+			(at 195.58 119.38 0)
+			(effects
+				(font
+					(size 1.27 1.27)
+				)
+				(hide yes)
+			)
+		)
+		(property "Description" ""
+			(at 190.5 119.38 0)
+			(effects
+				(font
+					(size 1.27 1.27)
+				)
+				(hide yes)
+			)
+		)
+		(pin "1"
+		)
+		(instances
+			(project "Controls-PedalsDaughter"
+				(path "/30d77876-714b-4f1b-9bad-b74eb43ddcf6"
+					(reference "TP_3V3PWR1")
+					(unit 1)
+				)

Commit message: Fixed 3V3 :P
Connections:
- net +3.3V is gone; now on net +3V3: D1.1 (K), D3.1 (K), U2.2 (+3.3V), U2.9 (+3.3V)
Changed lines of the file:
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@@
 			)
 		)
-		(property "Value" "+3.3V"
+		(property "Value" "+3V3"
 			(at 116.84 123.19 0)
 			(effects
@@
 			)
 		)
-		(property "Value" "+3.3V"
+		(property "Value" "+3V3"
 			(at 250.19 41.9099 0)
 			(effects
@@
 			)
 		)
-		(property "Value" "+3.3V"
+		(property "Value" "+3V3"
 			(at 237.49 109.22 0)
 			(effects
