File: Controls-PedalsDaughter.kicad_sch (KiCad schematic)
At the start: 36 parts, among them J2 Accel Pos. Sensor, J3 PeripheralCANConnector, J4 Conn_01x02, J5 PeripheralCANConnector, U1 RI3-1205S, U2 PeripheralSOM, U3 TLV9301xDCK, U4 AMC1300BDWV, U5 TLV70130DBVR

Commit message: Yuh
Parts:
- removed +12V1: +12V_TP, TestPoint:TestPoint_Pad_1.5x1.5mm, symbol Connector:TestPoint
- removed +5V1: +5V_TP, TestPoint:TestPoint_Pad_1.5x1.5mm, symbol Connector:TestPoint
- removed C1, C10: 1nF, Capacitor_SMD:C_0805_2012Metric, symbol Device:C
- removed C11: 100nF, Capacitor_SMD:C_0805_2012Metric, symbol Device:C
- removed C12: 0.1uf, Capacitor_SMD:C_0805_2012Metric, symbol Device:C
- removed C2: 10uF, Capacitor_SMD:C_0805_2012Metric, symbol Device:C
- removed C3: 1nf, Capacitor_SMD:C_0805_2012Metric, symbol Device:C
- removed C4, C5: 10uf, Capacitor_SMD:C_0805_2012Metric, symbol Device:C
- removed C6, C9: 100uF, Capacitor_SMD:C_0805_2012Metric, symbol Device:C
- removed C7, C8: 1uF, Capacitor_SMD:C_0805_2012Metric, symbol Device:C
- removed D1, D2, D3, D4: MBR, Diode_SMD:D_0805_2012Metric, symbol Device:D
- removed D6: SMD_0805, Diode_SMD:D_0805_2012Metric, symbol Device:LED
- removed D7: PESD15VL1BA, Diode_SMD:D_SOD-323, symbol Diode:SD12_SOD323
- removed GND1: GND_TP, TestPoint:TestPoint_Pad_1.5x1.5mm, symbol Connector:TestPoint
- removed GNDPWR1: GNDPWR_TP, TestPoint:TestPoint_Pad_1.5x1.5mm, symbol Connector:TestPoint
- removed J2: Accel Pos. Sensor, Connector_Molex:Molex_Micro-Fit_3.0_43045-0612_2x03_P3.00mm_Vertical, symbol Connector_Generic:Conn_02x03_Top_Bottom
- removed J4: Conn_01x02, Connector_Molex:Molex_Micro-Fit_3.0_43045-0212_2x01_P3.00mm_Vertical, symbol Connector_Generic:Conn_01x02
- removed R1: 20, Resistor_SMD:R_0805_2012Metric, symbol Device:R_US
- removed R2: 8.2k, Resistor_SMD:R_0805_2012Metric, symbol Device:R_US
- removed R3: 1.5k, Resistor_SMD:R_0805_2012Metric, symbol Device:R_US
- removed R4: 22k, Resistor_SMD:R_0805_2012Metric, symbol Device:R_US
- removed TP_3V3PWR1: +3V3PWR, TestPoint:TestPoint_Pad_1.5x1.5mm, symbol Connector:TestPoint
- removed U1: RI3-1205S, UTSVT_ICs:RI3_DC_Converter, symbol Dashboard-rescue:RI3-1205S-utsvt-power-regulators
- removed U3: TLV9301xDCK, Package_TO_SOT_SMD:SOT-353_SC-70-5, symbol Amplifier_Operational:TLV9301xDCK
- removed U4: AMC1300BDWV, Package_SO:SOIC-8_7.5x5.85mm_P1.27mm, symbol Amplifier_Difference:AMC1300BDWV
- removed U5: TLV70130DBVR, Package_TO_SOT_SMD:SOT-353_SC-70-5, symbol 2025-01-18_20-51-31:TLV70130DBVR
Connections:
- net Brake_Fl: now reaches U2.19 (SPI1_NSS)
- net Brake renamed Brake_Pot
- no-connect marks 17 -> 13
Other:
- added sheet Brake Fluid Sensor (Brake_Fl.kicad_sch)
- added sheet Pedals (untitled.kicad_sch)
- added sheet Power (power.kicad_sch)
- note removed: "0.5V - 4.5V Analog signal"
- note removed: "20ma -> ~0.4V (*8.2) -> 3.28v"
- note removed: "3V3 Pwr for Isolated Amp"
- note removed: "4.5V -> 3.278V"
- note removed: "Accel Pedal"
- note removed: "Based on: https://www.akao.co.uk/manuals/Link%20G4+%20Manual/nissan_vq35.htm"
- note removed: "Brake"
- note removed: "Break Pedal"
- note removed: "Break sensor gives current reading 4ma - 20ma"
- note removed: "For 5V needed for Accel Sensor"
- note removed: "ISOLATED PWR"
- note removed: "Isolated Amp"
- note removed: "Local (Leader Board) GND (Internal)"
- note removed: "Notes: · Motor + refers to the pin that has battery voltage applied to it to open the throttle. · It is recommended to use shielded cables for TPS and APS sensors. · To prevent back feeding, the throttle motor relay must be controlled from a non flywheeled output such as a spare Ignition or Injection channel. - If the sensor and microcontroller are powered from different systems or are physically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"
- note removed: "Power"
- note removed: "Power GND (External)"
- note removed: "Pwr LED"
- note removed: "Redundant Signal"
- note removed: "Schotky :)"
- note removed: "bypass :)"
- note removed: "x8.2 gain"
- moved on the sheet: J3, J5, U2

Commit message: Ravi <3
Changed lines of the file:
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@@
 	(paper "A4")
-	(junction
-		(at 223.52 73.66)
-		(diameter 0)
-		(color 0 0 0 0)
-	)
 	(junction
 		(at 185.42 124.46)
@@
 		(pts
 			(xy 162.56 92.71) (xy 162.56 90.17)
-		)
-		(stroke
-			(width 0)
-			(type default)
-		)
-	)
-	(wire
-		(pts
-			(xy 223.52 73.66) (xy 223.52 76.2)
 		)
 		(stroke
@@
 	)
 	(symbol
+		(lib_id "power:+3.3V")
+		(at 223.52 76.2 270)
+		(unit 1)
+		(exclude_from_sim no)
+		(in_bom yes)
+		(on_board yes)
+		(dnp no)
+		(fields_autoplaced yes)
+		(property "Reference" "#PWR054"
+			(at 219.71 76.2 0)
+			(effects
+				(font
+					(size 1.27 1.27)
+				)
+				(hide yes)
+			)
+		)
+		(property "Value" "+3V3"
+			(at 227.33 76.1999 90)
+			(effects
+				(font
+					(size 1.27 1.27)
+				)
+				(justify left)
+			)
+		)
+		(property "Footprint" ""
+			(at 223.52 76.2 0)
+			(effects
+				(font
+					(size 1.27 1.27)
+				)
+				(hide yes)
+			)
+		)
+		(property "Datasheet" ""
+			(at 223.52 76.2 0)
+			(effects
+				(font
+					(size 1.27 1.27)
+				)
+				(hide yes)
+			)
+		)
+		(property "Description" "Power symbol creates a global label with name \"+3.3V\""
+			(at 223.52 76.2 0)
+			(effects
+				(font
+					(size 1.27 1.27)
+				)
+				(hide yes)
+			)
+		)
+		(pin "1"
+		)
+		(instances
+			(project "Controls-PedalsDaughter"
+				(path "/30d77876-714b-4f1b-9bad-b74eb43ddcf6"
+					(reference "#PWR054")
+					(unit 1)
+				)
+			)
+		)
+	)
+	(symbol
 		(lib_id "utsvt-misc:PeripheralSOM")
 		(at 204.47 99.06 0)
@@
 	(symbol
 		(lib_id "power:+3.3V")
-		(at 223.52 73.66 0)
+		(at 223.52 73.66 270)
 		(unit 1)
 		(exclude_from_sim no)
@@
 		(fields_autoplaced yes)
 		(property "Reference" "#PWR022"
-			(at 223.52 77.47 0)
+			(at 219.71 73.66 0)
 			(effects
 				(font
@@
 		)
 		(property "Value" "+3V3"
-			(at 226.06 72.3899 0)
-			(effects
-				(font
+			(at 227.33 73.6599 90)
+			(effects
+				(font

Commit message: Fixed some stuff
Other:
- sheet Pedals: file untitled.kicad_sch -> pedals.kicad_sch
Changed lines of the file:
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@@
 			)
 		)
-		(property "Sheetfile" "untitled.kicad_sch"
+		(property "Sheetfile" "pedals.kicad_sch"
 			(at 63.5 100.9634 0)
 			(effects

Commit message: peapeapoohpooh
Connections:
- net +VDDA: now reaches U2.10 (VDDA(3.3V))
- net GNDA: now reaches U2.12 (GNDA)
- no-connect marks 13 -> 11

Commit message: new constraints
Parts:
- removed J3, J5: PeripheralCANConnector, UTSVT_Connectors:Molex_MicroFit3.0_1x4xP3.00mm_PolarizingPeg_Vertical, symbol utsvt-connectors:PeripheralCANConnector
- removed U2: PeripheralSOM, UTSVT_Special:PeripheralSOM, symbol utsvt-misc:PeripheralSOM
- added J1: MX150_02x03_Vertical, UTSVT_Connectors:CONN06_0757575131_MOL, symbol utsvt_connectors:MX150_02x03_Vertical
- added J6: MX150_02x10_Vertical, UTSVT_Connectors:CONN_SD-75757-002_2X10_F16p09_MOL, symbol utsvt_connectors:MX150_02x10_Vertical
- added J7: 53307-2471, UTSVT_Connectors:PeripheralSOM, symbol utsvt_connectors:PeripheralSOMConnector
Connections:
- no-connect marks 11 -> 0
Other:
- note removed: "Daisy Chain :)"
