File: Controls-PedalsDaughter.kicad_pcb (KiCad board)
At the start: 2 copper layers, 50.8 x 74.2 mm, 54 parts, among them J1 Brake Pos. Sensor, J2 Accel Pos. Sensor, J3 PeripheralCANConnector, J4 Conn_01x02, J5 PeripheralCANConnector, U1 RI3-1205S, U2 PeripheralSOM, U3 TLV9301xDCK, U4 TLV70130DBVR, U5 AMC1300BDWV, U6 TLV9301xDCK

Commit message: via fix
Routing:
- net +3V3: track 76.9 -> 79.3 mm, vias 7 -> 6
Changed lines of the file:
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@@
 		(fp_arc
 			(start 21.237742 18.612258)
-			(mid 20.300482 20.874999)
+			(mid 20.300481 20.874995)
 			(end 18.037742 21.812258)
 			(stroke
@@
 	)
 	(segment
-		(start 128.425 98.7625)
-		(end 127.25 99.9375)
-		(width 0.25)
-		(layer "F.Cu")
-		(net 8)
-	)
-	(segment
 		(start 152.525 93.7375)
 		(end 152.525 93.75)
@@
 	)
 	(segment
-		(start 150.1875 97.8125)
-		(end 152.12 97.8125)
+		(start 135.8125 113.8125)
+		(end 135.8125 115.75)
 		(width 0.25)
 		(layer "F.Cu")
@@
 	)
 	(segment
-		(start 144.6 98.7625)
-		(end 149.2375 98.7625)
+		(start 131.5 98.7625)
+		(end 128.425 98.7625)
 		(width 0.25)
 		(layer "F.Cu")
@@
 	)
 	(segment
-		(start 129.05 98.7625)
-		(end 128.425 98.7625)
+		(start 150.1875 97.8125)
+		(end 152.12 97.8125)
 		(width 0.25)
 		(layer "F.Cu")
@@
 	)
 	(segment
-		(start 127.25 105.25)
-		(end 135.8125 113.8125)
+		(start 144.6 98.7625)
+		(end 149.2375 98.7625)
 		(width 0.25)
 		(layer "F.Cu")
@@
 	)
 	(segment
-		(start 152.525 96.725)
-		(end 152.525 95.8375)
+		(start 127.25 105.25)
+		(end 135.8125 113.8125)
 		(width 0.25)
 		(layer "F.Cu")
@@
 	)
 	(segment
-		(start 129.05 98.7625)
-		(end 137 98.7625)
+		(start 152.525 96.725)
+		(end 152.525 95.8375)
 		(width 0.25)
 		(layer "F.Cu")
@@
 	)
 	(segment
-		(start 135.8125 113.8125)
-		(end 135.8125 115.75)
+		(start 128.425 98.7625)
+		(end 127.25 99.9375)
 		(width 0.25)
 		(layer "F.Cu")
@@
 	)
 	(via
-		(at 129.05 98.7625)
-		(size 0.6)
-		(drill 0.3)
-		(layers "F.Cu" "B.Cu")
-		(net 8)
-	)
-	(via
 		(at 144.6 98.7625)
 		(size 0.6)
@@
 	)
 	(via
-		(at 137 98.7625)
+		(at 131.5 98.7625)
 		(size 0.6)
 		(drill 0.3)
@@
 	)
 	(segment
-		(start 126.35625 95.5625)
-		(end 124.75 95.5625)
+		(start 131.5 98.7625)
+		(end 144.6 98.7625)
 		(width 0.25)
 		(layer "B.Cu")
@@
 	)
 	(segment
-		(start 143 84.225)
-		(end 143 82.6875)
+		(start 127 97.8625)
+		(end 127 96.20625)
 		(width 0.25)
 		(layer "B.Cu")
@@
 	)
 	(segment
-		(start 137 98.7625)
-		(end 144.6 98.7625)
+		(start 131.5 98.7625)
+		(end 127.9 98.7625)
 		(width 0.25)
 		(layer "B.Cu")
@@
 	)
 	(segment
-		(start 152.525 93.75)
-		(end 143 84.225)
+		(start 126.35625 95.5625)
+		(end 124.75 95.5625)
 		(width 0.25)
 		(layer "B.Cu")
@@
 	)
 	(segment
-		(start 127 97.8625)
-		(end 127 96.20625)
+		(start 143 84.225)
+		(end 143 82.6875)
 		(width 0.25)
 		(layer "B.Cu")
@@
 	)
 	(segment
-		(start 127.9 98.7625)
-		(end 127 97.8625)
+		(start 127 96.20625)
+		(end 126.35625 95.5625)
 		(width 0.25)
 		(layer "B.Cu")
@@
 	)
 	(segment
-		(start 127 96.20625)
-		(end 126.35625 95.5625)
+		(start 152.525 93.75)
+		(end 143 84.225)
 		(width 0.25)
 		(layer "B.Cu")
@@
 	)
 	(segment
-		(start 129.05 98.7625)
-		(end 127.9 98.7625)
+		(start 127.9 98.7625)
+		(end 127 97.8625)
 		(width 0.25)
 		(layer "B.Cu")

Commit message: Fixed some stuff
Parts:
- C5: value 10uf -> .1uf
- moved D3 4.00 mm to (152.0, 100.5), turned to 0 degrees
- moved D4 4.00 mm to (156.0, 100.5), turned to 0 degrees
- renumbered PWR_LED to PWR
Routing:
- net +3V3: track 79.3 -> 76.6 mm
- net /Brake_Pot: track 56.7 -> 58.5 mm
- net +3V3PWR: track 20.6 -> 22.3 mm
- net +12V: track 2.27 -> 3.80 mm
- net /Brake_Fl: track 66.8 -> 65.9 mm

Commit message: r
Parts:
- moved D7 7.22 mm to (128.4, 73.0)
- moved R3 7.22 mm to (126.6, 73.0)
- renumbered +12V to +12V1, +5V to +5V1, Accel_Raw to Accel_Raw1, Accel_TP to Accel_TP1, Brake_Fl_Sn to Brake_Fl_Sn1, Brake_Fl_Sn_Raw to Brake_Fl_Sn_Raw1, Brake_Raw to Brake_Raw1, Brake_TP to Brake_TP1, PWR to D7, GND to GND1, GNDPWR to GNDPWR1, TP_3V3PWR to TP_3V3PWR1
Connections:
- J4 pad 1: GNDPWR -> +12V
Changed lines of the file:
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@@
 	(footprint "Resistor_SMD:R_0805_2012Metric"
 		(layer "F.Cu")
-		(at 133.15 70)
+		(at 126.5875 73)
 		(descr "Resistor SMD 0805 (2012 Metric), square (rectangular) end terminal, IPC_7351 nominal, (Body size source: IPC-SM-782 page 72, https://www.pcb-3d.com/wordpress/wp-content/uploads/ipc-sm-782a_amendment_1_and_2.pdf), generated with kicad-footprint-generator")
 		(tags "resistor")
@@
 		(tags "diode")
 		(property "Reference" "D3"
-			(at -2.75 -0.05 360)
+			(at -2.75 -0.05 0)
 			(layer "B.SilkS")
 			(effects
@@
 		)
 		(property "Value" "MBR"
-			(at 0 -1.65 360)
+			(at 0 -1.65 0)
 			(layer "B.Fab")
 			(effects
@@
 		)
 		(fp_text user "${REFERENCE}"
-			(at 0 0 360)
+			(at 0 0 0)
 			(layer "B.Fab")
 			(effects
@@
 		(property ki_fp_filters "SOT*353*SC*70*")
 		(sheetname "Pedals")
-		(sheetfile "untitled.kicad_sch")
+		(sheetfile "pedals.kicad_sch")
 		(attr smd)
 		(fp_line
@@
 		(property ki_fp_filters "R_*")
 		(sheetname "Pedals")
-		(sheetfile "untitled.kicad_sch")
+		(sheetfile "pedals.kicad_sch")
 		(attr smd)
 		(fp_line
@@
 		(descr "THT rectangular pad as test Point, square 1.5mm side length, hole diameter 0.7mm")
 		(tags "test point THT pad rectangle square")
-		(property "Reference" "Accel_TP"
+		(property "Reference" "Accel_TP1"
 			(at -4.25 0.75 180)
 			(layer "B.SilkS")
@@
 		(property ki_fp_filters "Pin* Test*")
 		(sheetname "Pedals")
-		(sheetfile "untitled.kicad_sch")
+		(sheetfile "pedals.kicad_sch")
 		(attr exclude_from_pos_files)
 		(fp_line
@@
 		(tags "diode")
 		(property "Reference" "D4"
-			(at 2.75 0.05 360)
+			(at 2.75 0.05 0)
 			(layer "B.SilkS")
 			(effects
@@
 		)
 		(property "Value" "MBR"
-			(at 0 -1.65 360)
+			(at 0 -1.65 0)
 			(layer "B.Fab")
 			(effects
@@
 		)
 		(fp_text user "${REFERENCE}"
-			(at 0 0 360)
+			(at 0 0 0)
 			(layer "B.Fab")
 			(effects
@@
 	(footprint "Diode_SMD:D_0805_2012Metric"
 		(layer "B.Cu")
-		(at 135 70 180)
+		(at 128.4375 73 180)
 		(descr "Diode SMD 0805 (2012 Metric), square (rectangular) end terminal, IPC_7351 nominal, (Body size source: https://docs.google.com/spreadsheets/d/1BsfQQcO9C6DZCsRaXUlFlo91Tg2WpOkGARC1WS5S8t0/edit?usp=sharing), generated with kicad-footprint-generator")
 		(tags "diode")
-		(property "Reference" "PWR"
+		(property "Reference" "D7"
 			(at 0 1.75 180)
 			(layer "B.SilkS")
@@
 		(descr "SMD rectangular pad as test Point, square 1.5mm side length")
 		(tags "test point SMD pad rectangle square")
-		(property "Reference" "GNDPWR"
+		(property "Reference" "GNDPWR1"
 			(at -0.785 1.9 0)
 			(unlocked yes)
@@
 		(descr "THT rectangular pad as test Point, square 1.5mm side length, hole diameter 0.7mm")
 		(tags "test point THT pad rectangle square")
-		(property "Reference" "Brake_Fl_Sn_Raw"
+		(property "Reference" "Brake_Fl_Sn_Raw1"
 			(at -1.75 3.7 0)
 			(layer "B.SilkS")
@@
 		(property ki_fp_filters "C_*")
 		(sheetname "Pedals")
-		(sheetfile "untitled.kicad_sch")
+		(sheetfile "pedals.kicad_sch")
 		(attr smd)
 		(fp_line
@@
 		(property ki_fp_filters "Connector*:*_2x??_*")
 		(sheetname "Pedals")
-		(sheetfile "untitled.kicad_sch")
+		(sheetfile "pedals.kicad_sch")
 		(attr through_hole)
 		(fp_line
@@
 		(descr "SMD rectangular pad as test Point, square 1.5mm side length")
 		(tags "test point SMD pad rectangle square")
-		(property "Reference" "+5V"
+		(property "Reference" "+5V1"
 			(at 1.9 0.2 0)
 			(layer "B.SilkS")
@@
 		(descr "SMD rectangular pad as test Point, square 1.5mm side length")
 		(tags "test point SMD pad rectangle square")
-		(property "Reference" "GND"
+		(property "Reference" "GND1"
 			(at 0 1.9 0)
 			(layer "B.SilkS")
@@
 		(property ki_fp_filters "R_*")
 		(sheetname "Pedals")
-		(sheetfile "untitled.kicad_sch")
+		(sheetfile "pedals.kicad_sch")
 		(attr smd)
 		(fp_line
@@
 		(descr "THT rectangular pad as test Point, square 1.5mm side length, hole diameter 0.7mm")
 		(tags "test point THT pad rectangle square")
-		(property "Reference" "Brake_Fl_Sn"
+		(property "Reference" "Brake_Fl_Sn1"
 			(at 0 5.4 90)
 			(layer "B.SilkS")
@@
 		(descr "SMD rectangular pad as test Point, square 1.5mm side length")
 		(tags "test point SMD pad rectangle square")
-		(property "Reference" "+12V"
+		(property "Reference" "+12V1"
 			(at -0.3 1.9 180)
 			(layer "B.SilkS")
@@
 		(descr "THT rectangular pad as test Point, square 1.5mm side length, hole diameter 0.7mm")
 		(tags "test point THT pad rectangle square")
-		(property "Reference" "Accel_Raw"
+		(property "Reference" "Accel_Raw1"
 			(at -0.25 -1.8 180)
 			(layer "B.SilkS")
@@
 		(property ki_fp_filters "Pin* Test*")
 		(sheetname "Pedals")
-		(sheetfile "untitled.kicad_sch")
+		(sheetfile "pedals.kicad_sch")
 		(attr exclude_from_pos_files)
 		(fp_line
@@
 			(remove_unused_layers no)
 			(roundrect_rratio 0.166667)
-			(net 4 "GNDPWR")
+			(net 3 "+12V")
 			(pinfunction "Pin_1")
 			(pintype "passive")
@@
 		(property ki_fp_filters "R_*")
 		(sheetname "Pedals")
-		(sheetfile "untitled.kicad_sch")
+		(sheetfile "pedals.kicad_sch")
 		(attr smd)
 		(fp_line
@@
 		(property ki_fp_filters "SOT*353*SC*70*")
 		(sheetname "Pedals")
-		(sheetfile "untitled.kicad_sch")
+		(sheetfile "pedals.kicad_sch")
 		(attr smd)
 		(fp_line
@@
 		(property ki_fp_filters "TO-???* *_Diode_* *SingleDiode* D_*")
 		(sheetname "Pedals")
-		(sheetfile "untitled.kicad_sch")
+		(sheetfile "pedals.kicad_sch")
 		(attr smd)
 		(fp_line
@@
 		(property ki_fp_filters "TO-???* *_Diode_* *SingleDiode* D_*")
 		(sheetname "Pedals")
-		(sheetfile "untitled.kicad_sch")
+		(sheetfile "pedals.kicad_sch")
 		(attr smd)
 		(fp_line
@@
 		(descr "SMD rectangular pad as test Point, square 1.5mm side length")
 		(tags "test point SMD pad rectangle square")
-		(property "Reference" "TP_3V3PWR"
+		(property "Reference" "TP_3V3PWR1"
 			(at -5 0 90)
 			(layer "B.SilkS")
@@
 		(descr "THT rectangular pad as test Point, square 1.5mm side length, hole diameter 0.7mm")
 		(tags "test point THT pad rectangle square")
-		(property "Reference" "Brake_TP"
+		(property "Reference" "Brake_TP1"
 			(at 1.9 0 0)
 			(layer "B.SilkS")
@@
 		(property ki_fp_filters "Pin* Test*")
 		(sheetname "Pedals")
-		(sheetfile "untitled.kicad_sch")
+		(sheetfile "pedals.kicad_sch")
 		(attr exclude_from_pos_files)
 		(fp_line
@@
 		(property ki_fp_filters "C_*")
 		(sheetname "Pedals")
-		(sheetfile "untitled.kicad_sch")
+		(sheetfile "pedals.kicad_sch")
 		(attr smd)
 		(fp_line
@@
 		(property ki_fp_filters "TO-???* *_Diode_* *SingleDiode* D_*")
 		(sheetname "Pedals")
-		(sheetfile "untitled.kicad_sch")
+		(sheetfile "pedals.kicad_sch")
 		(attr smd)
 		(fp_line
@@
 		(property ki_fp_filters "C_*")
 		(sheetname "Pedals")
-		(sheetfile "untitled.kicad_sch")
+		(sheetfile "pedals.kicad_sch")
 		(attr smd)
 		(fp_line
@@
 		(property ki_fp_filters "Connector*:*_2x??_*")
 		(sheetname "Pedals")
-		(sheetfile "untitled.kicad_sch")
+		(sheetfile "pedals.kicad_sch")
 		(attr through_hole)
 		(fp_line
@@
 		(descr "THT rectangular pad as test Point, square 1.5mm side length, hole diameter 0.7mm")
 		(tags "test point THT pad rectangle square")
-		(property "Reference" "Brake_Raw"
+		(property "Reference" "Brake_Raw1"
 			(at 0 2 0)
 			(layer "B.SilkS")
@@
 		(property ki_fp_filters "Pin* Test*")
 		(sheetname "Pedals")
-		(sheetfile "untitled.kicad_sch")
+		(sheetfile "pedals.kicad_sch")
 		(attr exclude_from_pos_files)
 		(fp_line
@@
 		(property ki_fp_filters "R_*")
 		(sheetname "Pedals")
-		(sheetfile "untitled.kicad_sch")
+		(sheetfile "pedals.kicad_sch")
 		(attr smd)
 		(fp_line
@@
 		(property ki_fp_filters "TO-???* *_Diode_* *SingleDiode* D_*")
 		(sheetname "Pedals")
-		(sheetfile "untitled.kicad_sch")
+		(sheetfile "pedals.kicad_sch")
 		(attr smd)
 		(fp_line
@@
 		(property ki_fp_filters "C_*")
 		(sheetname "Pedals")
-		(sheetfile "untitled.kicad_sch")
+		(sheetfile "pedals.kicad_sch")
 		(attr smd)
 		(fp_line
@@
 	)
 	(via
-		(at 134.0625 70)
+		(at 127.5 73)
 		(size 0.6)
 		(drill 0.3)

Commit message: peapeapoohpooh
Parts:
- moved Brake_Fl_Raw 0.45 mm to (171.2, 75.0)
- turned C9 to 0 degrees
- renumbered +12V1 to +12V, +5V1 to +5V, TP_3V3PWR1 to 3V3PWR, Accel_TP1 to Accel, Accel_Raw1 to Accel_Raw, Brake_TP1 to Brake, Brake_Fl_Sn1 to Brake_Fl, Brake_Fl_Sn_Raw1 to Brake_Fl_Raw, Brake_Raw1 to Brake_Raw, GND1 to GND, GNDPWR1 to GNDPWR
Connections:
- C10 pad 1: +3V3 -> +VDDA
- C10 pad 2: GND -> GNDA
- C11 pad 1: +3V3 -> +VDDA
- C11 pad 2: GND -> GNDA
- C9 pad 2: GND -> GNDA
- D3 pad 1: +3V3 -> +VDDA
- D4 pad 2: GND -> GNDA
- U2 pad 10: unconnected-(U2-VDDA(3.3V)-Pad10) -> +VDDA
- U2 pad 12: unconnected-(U2-GNDA-Pad12) -> GNDA
- U5 pad 5: GND -> GNDA
- U5 pad 6: GND -> GNDA
- U5 pad 8: +3V3 -> +VDDA
Routing:
- net GNDA: track 0.00 -> 45.5 mm, vias 0 -> 3
- net +VDDA: track 0.00 -> 37.2 mm, vias 0 -> 3
- net +3V3: track 76.6 -> 54.2 mm, vias 6 -> 2
- net Net-(U3-+): track 19.8 -> 18.5 mm, vias 0 -> 1
- net +12V: track 3.80 -> 5.03 mm, vias 3 -> 4
- net /Brake_Fl: track 65.9 -> 64.8 mm
- net /CAN_H: track 66.8 -> 67.4 mm, vias 3 -> 1
- net GND: vias 3 -> 1
Other:
- board text added: "This area needs to be clear for USBC"
