File: Pedals.kicad_sch (KiCad schematic)
At the start: 42 parts, among them J1 PowerConn, J2 Throttle Body, J5 Accel Pos. Sensor, J6 Break_Pedal, J7 Gas_Pedal, U1 RI3-1205S

Commit message: Combined
Parts:
- removed C4, C5, C6, C7, C8: C, symbol Device:C
- removed D10, D11, D12, D13, D3, D5, D6, D7, D8, D9: D, symbol Device:D
- removed J2: Throttle Body, symbol Connector_Generic:Conn_02x03_Top_Bottom
- removed J6: Break_Pedal, symbol Connector_Generic:Conn_02x03_Top_Bottom
- removed J7: Gas_Pedal, symbol Connector_Generic:Conn_02x03_Top_Bottom
- removed R10, R2, R7, R8, R9: 1k, symbol Device:R_US
- removed R11, R12, R13, R14, R6: 2k, symbol Device:R_US
Other:
- note removed: "Based on: https://www.tbssowners.com/threads/need-help-0-5v-at-tps.244345/"
- note removed: "Pulldown Res, Filter Cap, Voltage spike and reverse polarity protection (?)"
- note removed: "TP1 vs TP2 may be reverse versions of each other (TP1 = true val, TP2 = Max - TP2)"
- note removed: "This will go to ADC input of Controller"
- note removed: "Throttle Position Sensor?"
- note removed: "Voltage Div [(2k)(1k)]/[2k+1k] 5V to 3.3V"
- moved on the sheet: C3, D2, D4, J5, R4, R5

Commit message: Fixed some stuff
Parts:
- removed C2: 10u, UTSVT_Passive:C_2220_5750Metric, symbol Device:C
- removed D4: D, symbol Device:D
- removed J1: PowerConn, UTSVT_Connectors:Molex_MicroFit3.0_1x2xP3.00mm_PolarizingPeg_Vertical, symbol Connector_Generic:Conn_01x02
- removed J5: Accel Pos. Sensor, symbol Connector_Generic:Conn_02x03_Top_Bottom
- removed TP1: +12V_TP, TestPoint:TestPoint_Pad_1.5x1.5mm, symbol Connector:TestPoint
- removed TP2: GNDPWR_TP, TestPoint:TestPoint_Pad_1.5x1.5mm, symbol Connector:TestPoint
- removed TP3: +5V_TP, TestPoint:TestPoint_Pad_1.5x1.5mm, symbol Connector:TestPoint
- removed TP4: GND_TP, TestPoint:TestPoint_Pad_1.5x1.5mm, symbol Connector:TestPoint
- removed U1: RI3-1205S, UTSVT_ICs:RI3_DC_Converter, symbol Dashboard-rescue:RI3-1205S-utsvt-power-regulators
- added Accel_Raw1: Accel_Raw_TP, TestPoint:TestPoint_THTPad_1.5x1.5mm_Drill0.7mm, symbol Connector:TestPoint
- added Accel_TP1: Accel, TestPoint:TestPoint_THTPad_1.5x1.5mm_Drill0.7mm, symbol Connector:TestPoint
- added Brake_Raw1: Brake_Raw_TP, TestPoint:TestPoint_THTPad_1.5x1.5mm_Drill0.7mm, symbol Connector:TestPoint
- added Brake_TP1: Brake, TestPoint:TestPoint_THTPad_1.5x1.5mm_Drill0.7mm, symbol Connector:TestPoint
- added C12, C14: 1nf, Capacitor_SMD:C_0805_2012Metric, symbol Device:C
- added C13: 0.1uf, Capacitor_SMD:C_0805_2012Metric, symbol Device:C
- added D5, D8: MBR, Diode_SMD:D_0805_2012Metric, symbol Device:D
- added J1: Brake Pos. Sensor, Connector_Molex:Molex_Micro-Fit_3.0_43045-0612_2x03_P3.00mm_Vertical, symbol Connector_Generic:Conn_02x03_Top_Bottom
- added J2: Accel Pos. Sensor, Connector_Molex:Molex_Micro-Fit_3.0_43045-0612_2x03_P3.00mm_Vertical, symbol Connector_Generic:Conn_02x03_Top_Bottom
- added R2: 8.2k, Resistor_SMD:R_0805_2012Metric, symbol Device:R_US
- added R6: 22k, Resistor_SMD:R_0805_2012Metric, symbol Device:R_US
- added U3, U6: TLV9301xDCK, Package_TO_SOT_SMD:SOT-353_SC-70-5, symbol Amplifier_Operational:TLV9301xDCK
- C3: value C -> 0.1uf; footprint (none) -> Capacitor_SMD:C_0805_2012Metric; P/N (none) -> pickle
- D1: value TVS -> MBR; footprint Diode_SMD:D_SOD-323 -> Diode_SMD:D_0805_2012Metric; P/N (none) -> MBR0520LT1G
- D2: value D -> MBR; footprint (none) -> Diode_SMD:D_0805_2012Metric; P/N (none) -> MBR0520LT1G
- R4: value 1k -> 22k; footprint (none) -> Resistor_SMD:R_0805_2012Metric; P/N (none) -> pickle
- R5: value 2k -> 8.2k; footprint (none) -> Resistor_SMD:R_0805_2012Metric; P/N (none) -> ERA-3ARB822V
Connections:
- net +5V: now also C3.2, C13.2, J1.4 (Pin_4), J1.6 (Pin_6), J2.4 (Pin_4), J2.6 (Pin_6), U3.5 (V+), U6.5 (V+)
- net GND: now also R4.2, C12.1, C13.1, C14.1, D8.2 (A), J1.1 (Pin_1), J1.3 (Pin_3), J2.1 (Pin_1), J2.3 (Pin_3), R6.2, U3.2 (V-), U6.2 (V-); no longer R5.2
- net +12V renamed +3V3
- net +3V3: now also D5.1 (K)
- net APS(Main): no longer names the net of R5.1
- net APS(Main): now also Brake_Raw1.1, R6.1, U6.1 (+); no longer R4.1
- net GNDPWR renamed Accel
- net Accel: now also D2.1 (K), Accel_TP1.1, C12.2, U3.3 (-), U3.4
- new net: J2.5 (Pin_5), R2.2
- new net: J1.5 (Pin_5), R5.2
- new net: Accel_Raw1.1, R2.1, R4.1, U3.1 (+)
- new net Brake_Pot: Brake_TP1.1, C14.2, D5.2 (A), D8.1 (K), U6.3 (-), U6.4
- no-connect marks 0 -> 2
Other:
- note added: "0.5V - 4.5V Analog signal"
- note added: "4.5V -> 3.278V"
- note added: "Accel Pedal"
- note added: "Brake Pedal"
- note added: "Notes: · Motor + refers to the pin that has battery voltage applied to it to open the throttle. · It is recommended to use shielded cables for TPS and APS sensors. · To prevent back feeding, the throttle motor relay must be controlled from a non flywheeled output such as a spare Ignition or Injection channel. - If the sensor and microcontroller are powered from different systems or are physically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"
- note added: "Redundant Signal"
- note added: "Schotky :)"
- note removed: "Accel Pedal Sensor?"
- note removed: "ISOLATED"
- note removed: "Local (Leader Board) GND (Internal)"
- note removed: "Not exactly sure what we'd use the TAC's for since we're wanting to use the direct sensor data output for controller (From what I understood)"
- note removed: "Notes: · Motor + refers to the pin that has battery voltage applied to it to open the throttle. · It is recommended to use shielded cables for TPS and APS sensors. · To prevent back feeding, the throttle motor relay must be controlled from a non flywheeled output such as a spare Ignition or Injection channel."
- note removed: "Pedals"
- note removed: "Power GND (External)"
- note removed: "TAC = Throttle Actuator Control Supposedly; electronically controls the throttle plate on a car with a drive-by-wire system"
- note removed: "TP = Throttle Position"

Commit message: new constraints
Parts:
- removed J1: Brake Pos. Sensor, Connector_Molex:Molex_Micro-Fit_3.0_43045-0612_2x03_P3.00mm_Vertical, symbol Connector_Generic:Conn_02x03_Top_Bottom
- removed J2: Accel Pos. Sensor, Connector_Molex:Molex_Micro-Fit_3.0_43045-0612_2x03_P3.00mm_Vertical, symbol Connector_Generic:Conn_02x03_Top_Bottom
