File: power.kicad_sch (KiCad schematic)
At the start: 11 parts, among them U1 RI3-1205S

Commit message: Ravi <3
Parts:
- C5: value 10uf -> .1uf
Changed lines of the file:
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@@
 			)
 		)
-		(property "Value" "10uf"
+		(property "Value" ".1uf"
 			(at 191.77 91.4399 0)
 			(effects

Commit message: Donesies?
Parts:
- R3: P/N pickle -> CRMA2512AF1K50FKEF
Changed lines of the file:
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@@
 			)
 		)
-		(property "P/N" "pickle"
+		(property "P/N" "CRMA2512AF1K50FKEF"
 			(at 180.34 114.3 0)
 			(effects

Commit message: new constraints
Parts:
- removed +12V1: +12V_TP, TestPoint:TestPoint_Pad_1.5x1.5mm, symbol Connector:TestPoint
- removed +5V1: +5V_TP, TestPoint:TestPoint_Pad_1.5x1.5mm, symbol Connector:TestPoint
- removed C2: 10uF, Capacitor_SMD:C_0805_2012Metric, symbol Device:C
- removed C4: 10uf, Capacitor_SMD:C_0805_2012Metric, symbol Device:C
- removed C5: .1uf, Capacitor_SMD:C_0805_2012Metric, symbol Device:C
- removed D6: PESD15VL1BA, Diode_SMD:D_SOD-323, symbol Diode:SD12_SOD323
- removed D7: SMD_0805, Diode_SMD:D_0805_2012Metric, symbol Device:LED
- removed GND1: GND_TP, TestPoint:TestPoint_Pad_1.5x1.5mm, symbol Connector:TestPoint
- removed GNDPWR1: GNDPWR_TP, TestPoint:TestPoint_Pad_1.5x1.5mm, symbol Connector:TestPoint
- removed R3: 1.5k, Resistor_SMD:R_0805_2012Metric, symbol Device:R_US
- removed U1: RI3-1205S, UTSVT_ICs:RI3_DC_Converter, symbol Dashboard-rescue:RI3-1205S-utsvt-power-regulators
Other:
- note removed: "For 5V needed for Accel Sensor"
- note removed: "ISOLATED PWR"
- note removed: "Local (Leader Board) GND (Internal)"
- note removed: "Power"
- note removed: "Power GND (External)"
- note removed: "Pwr LED"
- note removed: "bypass :)"
