File: hardware/VCAT-PedalBoxPCB/Controls-PedalsDaughter.kicad_sch (KiCad schematic)
At the start: 3 parts, among them J1 MX150_02x03_Vertical, J6 MX150_02x10_Vertical, J7 53307-2471

Commit message: sch too ez
Parts:
- added H1, H2, H3, H4: M.3, MountingHole:MountingHole_3.2mm_M3_Pad_TopBottom, symbol Mechanical:MountingHole
- added Raw3: BrakePotSig, TestPoint:TestPoint_THTPad_1.5x1.5mm_Drill0.7mm, symbol Connector:TestPoint
- added Raw4: AccelPotSig, TestPoint:TestPoint_THTPad_1.5x1.5mm_Drill0.7mm, symbol Connector:TestPoint
- added Raw5: BrakePressSig, TestPoint:TestPoint_THTPad_1.5x1.5mm_Drill0.7mm, symbol Connector:TestPoint
Connections:
- net +24V: now reaches J1.1 (+24V)
- net +24V: now also J7.24 (+24V_In)
- net CANH_IN: now reaches J1.2 (CANH_IN)
- net CANH_IN: now also J1.6 (CANL_OUT), J7.22 (CAN_H)
- net CANL_IN: now reaches J1.3 (CANL_IN)
- net CANL_IN: now also J1.5 (CANH_OUT), J7.20 (CAN_L)
- net GND: now reaches J1.4 (GND)
- net GND: now also J7.1 (GND), J7.3 (GND), J7.5 (GND)
- net GNDA: now reaches J7.10 (GNDA)
- net GNDA: now also J6.11 (BrakePot1-), J6.13 (BrakePot2-), J6.14 (AccelPot1-), J6.16 (AccelPot2-), J6.17 (BrakePressure1-), J6.19 (BrakePressure2-)
- net Accel_GPIO: now reaches J7.11 (ADC1_IN9)
- net BrakePot_GPIO: now reaches J7.13 (ADC1_IN10)
- net BrakeFL_GPIO: now reaches J7.15 (ADC1_IN11)
- net AccelPotRed: now reaches J7.19 (ADC_IN15)
- net AccelPotRed: now also J6.15 (AccelPotSig2), Raw4.1
- net +3.3V: now reaches J7.2 (+3.3v)
- net BrakePressRed: now reaches J7.7 (ACD1_IN5)
- net BrakePressRed: now also J6.18 (BrakePresSig2), Raw5.1
- net +VDDA: now reaches J7.8 (VDDA)
- net BrakePotRed: now reaches J7.9 (ADC1_IN7)
- net BrakePotRed: now also J6.12 (BrakePotSig2), Raw3.1
- net VoutAdj1: now reaches J6.1 (BrakePot1+)
- net VoutAdj1: now also J6.3 (BrakePot2+), J6.4 (AccelPot1+), J6.6 (AccelPot2+)
- net BrakePot_ADC: now reaches J6.2 (BrakePotSig1)
- net Accel_ADC: now reaches J6.5 (AccelPotSig1)
- net VoutAdj2: now reaches J6.7 (BrakePressure1+)
- net VoutAdj2: now also J6.9 (BrakePressure2+)
- net BrakeFL_ADC: now reaches J6.8 (BrakePressureSig1)
- no-connect marks 0 -> 15
Other:
- sheet Brake Fluid Sensor ports: added BrakeFL_ADC, BrakeFL_GPIO; removed Brake_Fl
- sheet Pedals ports: added Accel_GPIO, BrakePot, BrakePot_GPIO; removed Brake_Pot
- sheet Power ports: added VoutAdj1, VoutAdj2; removed none
- note added: "Made with sweat and tears by Sathvik Y :) (no blood yet)"
- moved on the sheet: J1, J7

Commit message: final review?? (plssss)
Parts:
- added D1, D19, D2: 0603_SMD, LED_SMD:LED_0603_1608Metric_Pad1.05x0.95mm_HandSolder, symbol Device:LED
- added D16: PedalsBoard_Status_Red, LED_SMD:LED_0603_1608Metric_Pad1.05x0.95mm_HandSolder, symbol Device:LED
- added R14, R15, R49: 120, Resistor_SMD:R_0603_1608Metric_Pad0.98x0.95mm_HandSolder, symbol Device:R
- added R47: 1.1k, Resistor_SMD:R_0603_1608Metric_Pad0.98x0.95mm_HandSolder, symbol Device:R
- renumbered J7 to PSOM
Connections:
- net +24V: now also D16.2 (A)
- net GND: now also R14.1, R15.1, R47.2, R49.1
- net AccelPotStatus: now reaches PSOM.14 (GPIO_PB14)
- net AccelPotStatus: now also D2.2 (A)
- net BrakeFluidStatus: now reaches PSOM.16 (GPIO_PB15)
- net BrakeFluidStatus: now also D1.2 (A)
- net BrakePotStatus: now reaches PSOM.17 (GPIO_PA12)
- net BrakePotStatus: now also D19.2 (A)
- net VoutAdj1 renamed +5V
- net VoutAdj2 renamed +9V
- new net: D19.1 (K), R49.2
- new net: D2.1 (K), R15.2
- new net: D16.1 (K), R47.1
- new net: D1.1 (K), R14.2
- no-connect marks 15 -> 12
Other:
- note added: "Green Programmable LEDs"
- note removed: "PSOM"
- moved on the sheet: J1, J6, PSOM

Commit message: PSOM pin layout pic
Other:
- note added: "Mx150 Connectors (Pedals + CAN)"
- note added: "PSOM"
- note added: "Status LEDs"
- note removed: "Pedal Board"
- moved on the sheet: D1, D16, D19, D2, H1, H2, H3, H4, J1, J6, PSOM, R14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

Commit message: pcb design review #1
Parts:
- renumbered PSOM to PSOM1
Connections:
- net CANH_IN: no longer J1.6 (CANL_OUT)
- net CANL_IN: no longer J1.5 (CANH_OUT)
- net GND: now also J1.5 (CANH_OUT)
- no-connect marks 12 -> 13
Changed lines of the file:
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@@
 		(color 0 0 0 0)
 	)
+	(junction
+		(at 164.465 106.68)
+		(diameter 0)
+		(color 0 0 0 0)
+	)
 	(no_connect
 		(at 234.315 86.36)
 	)
 	(no_connect
+		(at 153.035 107.95)
+	)
+	(no_connect
 		(at 198.755 90.17)
 	)
@@
 	(wire
 		(pts
+			(xy 161.925 100.33) (xy 164.465 102.87)
+		)
+		(stroke
+			(width 0)
+			(type default)
+		)
+	)
+	(wire
+		(pts
 			(xy 136.525 153.035) (xy 137.795 153.035)
 		)
@@
 	(wire
 		(pts
-			(xy 153.035 100.33) (xy 163.195 100.33)
-		)
-		(stroke
-			(width 0)
-			(type default)
-		)
-	)
-	(wire
-		(pts
 			(xy 103.505 73.025) (xy 103.505 73.66)
 		)
@@
 	(wire
 		(pts
-			(xy 164.465 101.6) (xy 164.465 102.87)
+			(xy 164.465 102.87) (xy 164.465 106.68)
 		)
 		(stroke
@@
 	(wire
 		(pts
-			(xy 163.195 100.33) (xy 164.465 101.6)
-		)
-		(stroke
-			(width 0)
-			(type default)
-		)
-	)
-	(wire
-		(pts
 			(xy 196.85 96.52) (xy 198.755 96.52)
 		)
@@
 	(wire
 		(pts
+			(xy 153.035 104.14) (xy 161.925 104.14)
+		)
+		(stroke
+			(width 0)
+			(type default)
+		)
+	)
+	(wire
+		(pts
 			(xy 66.675 130.175) (xy 64.77 130.175)
 		)
@@
 	(wire
 		(pts
-			(xy 154.94 104.14) (xy 153.035 104.14)
+			(xy 104.14 74.295) (xy 118.745 74.295)
 		)
 		(stroke
@@
 	(wire
 		(pts
-			(xy 104.14 74.295) (xy 118.745 74.295)
+			(xy 164.465 106.68) (xy 164.465 107.95)
 		)
 		(stroke
@@
 	(wire
 		(pts
-			(xy 154.94 107.95) (xy 153.035 107.95)
+			(xy 153.035 100.33) (xy 161.925 100.33)
 		)
 		(stroke
@@
 	(wire
 		(pts
+			(xy 161.925 104.14) (xy 164.465 106.68)
+		)
+		(stroke
+			(width 0)
+			(type default)
+		)
+	)
+	(wire
+		(pts
 			(xy 103.505 73.66) (xy 103.505 80.645)
 		)
@@
 		)
 	)
-	(label "CANL_IN"
-		(at 154.94 104.14 0)
-		(effects
-			(font
-				(size 1.27 1.27)
-			)
-			(justify left bottom)
-		)
-	)
 	(label "BrakePot_ADC"
 		(at 117.475 55.245 180)
@@
 	)
 	(label "CANH_IN"
-		(at 154.94 107.95 0)
-		(effects
-			(font
-				(size 1.27 1.27)
-			)
-			(justify left bottom)
-		)
-	)
-	(label "CANH_IN"
 		(at 123.19 104.14 180)
 		(effects
@@
 	(symbol
 		(lib_id "power:GND")
-		(at 164.465 102.87 0)
+		(at 164.465 107.95 0)
 		(unit 1)
 		(exclude_from_sim no)
@@
 		(fields_autoplaced yes)
 		(property "Reference" "#PWR016"
-			(at 164.465 109.22 0)
+			(at 164.465 114.3 0)
 			(effects
 				(font
@@
 		)
 		(property "Value" "GND"
-			(at 164.465 107.95 0)
+			(at 164.465 113.03 0)
 			(effects
 				(font
@@
 		)
 		(property "Footprint" ""
-			(at 164.465 102.87 0)
+			(at 164.465 107.95 0)
 			(effects
 				(font
@@
 		)
 		(property "Datasheet" ""
-			(at 164.465 102.87 0)
+			(at 164.465 107.95 0)
 			(effects
 				(font
@@
 		)
 		(property "Description" "Power symbol creates a global label with name \"GND\" , ground"
-			(at 164.465 102.87 0)
+			(at 164.465 107.95 0)
 			(effects
 				(font
@@
 		(dnp no)
 		(fields_autoplaced yes)
-		(property "Reference" "PSOM"
+		(property "Reference" "PSOM1"
 			(at 216.535 43.815 0)
 			(effects
@@
 			(project ""
 				(path "/30d77876-714b-4f1b-9bad-b74eb43ddcf6"
-					(reference "PSOM")
+					(reference "PSOM1")
 					(unit 1)
 				)
@@
 		(exclude_from_sim no)
 		(in_bom yes)
-		(on_board yes)
+		(on_board no)
 		(dnp no)
 		(property "Reference" "H2"
@@
 		(exclude_from_sim no)
 		(in_bom yes)
-		(on_board yes)
+		(on_board no)
 		(dnp no)
 		(fields_autoplaced yes)
@@
 		(exclude_from_sim no)
 		(in_bom yes)
-		(on_board yes)
+		(on_board no)
 		(dnp no)
 		(fields_autoplaced yes)
@@
 		(exclude_from_sim no)
 		(in_bom yes)
-		(on_board yes)
+		(on_board no)
 		(dnp no)
 		(fields_autoplaced yes)

Commit message: PCB review #2
Parts:
- added Raw6: ShieldGND, TestPoint:TestPoint_THTPad_1.5x1.5mm_Drill0.7mm, symbol Connector:TestPoint
- BrakeFL1: renamed from Raw5; value BrakePressSig -> BrakeFLSig; Silkscreen (none) -> Brake FL
- renumbered Raw4 to AccelPot1, D2 to AccelPotStat1, D1 to BrakeFLStat1, Raw3 to BrakePot1, D19 to BrakePotStat1, D16 to PWR_+24
Connections:
- net GND: now also Raw6.1
- net AccelPotRed renamed AccelPotRedundant
- net Accel_ADC renamed Accel_Main
- net BrakeFL_ADC renamed BrakeFL_Main
- net BrakePotRed renamed BrakePotRedundant
- net BrakePot_ADC renamed BrakePot_Main
- net BrakePressRed renamed BrakeFLRedundant
Other:
- moved on the sheet: PSOM1

Commit message: review #3
Parts:
- added R16, R17: 0, Resistor_SMD:R_0603_1608Metric_Pad0.98x0.95mm_HandSolder, symbol Device:R
Connections:
- net CANH_IN: now also J1.5 (CANH_OUT), R16.1
- net CANL_IN: now also J1.6 (CANL_OUT), R17.1
- net GND: now also R16.2, R17.2; no longer J1.5 (CANH_OUT)
- no-connect marks 13 -> 12

Commit message: review #5
Parts:
- removed H1: M.3, MountingHole:MountingHole_3.2mm_M3_Pad_TopBottom, symbol Mechanical:MountingHole
- added R18: 0, Resistor_SMD:R_0603_1608Metric_Pad0.98x0.95mm_HandSolder, symbol Device:R
- J1: footprint UTSVT_Connectors:CONN06_0757575131_MOL -> UTSVT_Connectors:MX150_02x03_Vertical
Connections:
- net GND: now also J6.20, R18.1; no longer R16.2, R17.2
- net CANH_IN renamed CANH
- net CANH: no longer J1.2 (CANH_IN)
- net CANL_IN renamed CANL
- net CANL: no longer J1.3 (CANL_IN)
- new net: J1.2 (CANH_IN), R16.2
- new net: J1.3 (CANL_IN), R17.2, R18.2
- no-connect marks 12 -> 11
Other:
- moved on the sheet: R16, R17
