File: hardware/VCAT-PedalBoxPCB/Controls-PedalsDaughter.kicad_sch (KiCad schematic)
At the start: 21 parts, among them J1 MX150_02x03_Vertical, J6 MX150_02x10_Vertical

Commit message: Lakshay approved - final review #6
Parts:
- removed R16: 0, Resistor_SMD:R_0603_1608Metric_Pad0.98x0.95mm_HandSolder, symbol Device:R
- added R19, R20: 0, Resistor_SMD:R_0603_1608Metric_Pad0.98x0.95mm_HandSolder, symbol Device:R
- R17: now not fitted
Connections:
- net CANH: now also R19.1
- net GND: now also R20.1
- net at J1.2 (CANH_IN): now also R19.2, R20.2

Commit message: updated mx150 pin order :( works now
Parts:
- PSOM1: P/N 53307-2471 -> (none)
- R14, R15, R49: P/N FC0402E65R0BGT0 -> (none)
- R17, R18, R19, R20: P/N CRCW12101K10FKEAHP -> (none)

Commit message: updated BOM
Parts:
- J6: footprint UTSVT_Connectors:CONN_SD-75757-002_2X10_F16p09_MOL -> UTSVT_Connectors:MX150_02x10_Vertical
- R14, R15, R49: P/N (none) -> CRCW0603120RFKEC
- R17, R18, R19, R20: P/N (none) -> CRCW06030000Z0EE
Changed lines of the file:
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@@
 			)
 		)
-		(property "Description" "prgm LED"
+		(property "Description" "Pedals Status LEDs"
 			(at 122.555 153.035 0)
 			(effects
@@
 			)
 		)
-		(property "Description" ""
+		(property "Description" "Pedals CAN conn"
 			(at 142.24 93.345 0)
 			(effects
@@
 			)
 		)
-		(property "Description" "prgm led R45"
+		(property "Description" "Pedals status LED resistor"
 			(at 132.715 161.925 0)
 			(effects
@@
 			)
 		)
-		(property "P/N" ""
+		(property "P/N" "CRCW0603120RFKEC "
 			(at 132.715 161.925 90)
 			(effects
@@
 			)
 		)
-		(property "Description" "Controls R47"
+		(property "Description" "Pedals goofy ah 0 ohms"
 			(at 113.03 103.505 0)
 			(effects
@@
 			)
 		)
-		(property "P/N" "~"
+		(property "P/N" "CRCW06030000Z0EE"
 			(at 113.03 103.505 90)
 			(effects
@@
 			)
 		)
-		(property "Description" "Board-to-board connector for Peripheral SOM daughterboards"
+		(property "Description" "PSOM"
 			(at 229.235 35.814 0)
 			(effects
@@
 			)
 		)
+		(property "P/N" "~"
+			(at 184.15 152.4 90)
+			(effects
+				(font
+					(size 1.27 1.27)
+				)
+				(hide yes)
+			)
+		)
 		(pin "1"
 		)
@@
 			)
 		)
-		(property "Description" "Controls Lead LED"
+		(property "Description" "Pedals PWR LED"
 			(at 121.92 141.605 0)
 			(effects
@@
 			)
 		)
-		(property "Description" "Controls R47"
+		(property "Description" "Pedals PWR LED R47"
 			(at 132.08 141.605 0)
 			(effects
@@
 			)
 		)
-		(property "Footprint" "UTSVT_Connectors:CONN_SD-75757-002_2X10_F16p09_MOL"
+		(property "Footprint" "UTSVT_Connectors:MX150_02x10_Vertical"
 			(at 132.715 45.085 0)
 			(effects
@@
 			)
 		)
-		(property "Description" ""
+		(property "Description" "Pedals MX150"
 			(at 132.715 45.085 0)
 			(effects
@@
 			)
 		)
-		(property "Description" "prgm LED"
+		(property "Description" "Pedals Status LEDs"
 			(at 122.555 161.925 0)
 			(effects
@@
 			)
 		)
-		(property "Description" "prgm led R45"
+		(property "Description" "Pedals status LED resistor"
 			(at 132.715 153.035 0)
 			(effects
@@
 			)
 		)
-		(property "P/N" ""
+		(property "P/N" "CRCW0603120RFKEC "
 			(at 132.715 153.035 90)
 			(effects
@@
 			)
 		)
-		(property "Description" "Controls R47"
+		(property "Description" "Pedals goofy ah 0 ohms"
 			(at 113.03 107.315 0)
 			(effects
@@
 			)
 		)
-		(property "P/N" "~"
+		(property "P/N" "CRCW06030000Z0EE"
 			(at 113.03 107.315 90)
 			(effects
@@
 			)
 		)
-		(property "Description" "prgm led R45"
+		(property "Description" "Pedals status LED resistor"
 			(at 133.35 170.18 0)
 			(effects
@@
 			)
 		)
-		(property "P/N" ""
+		(property "P/N" "CRCW0603120RFKEC "
 			(at 133.35 170.18 90)
 			(effects
@@
 			)
 		)
-		(property "Description" "prgm LED"
+		(property "Description" "Pedals Status LEDs"
 			(at 123.19 170.18 0)
 			(effects
@@
 			)
 		)
-		(property "Description" "Controls R47"
+		(property "Description" "Pedals goofy ah 0 ohms"
 			(at 113.03 111.125 0)
 			(effects
@@
 			)
 		)
-		(property "P/N" "~"
+		(property "P/N" "CRCW06030000Z0EE"
 			(at 113.03 111.125 90)
 			(effects
@@
 			)
 		)
-		(property "Description" "Controls R47"
+		(property "Description" "Pedals goofy ah 0 ohms"
 			(at 113.03 99.695 0)
 			(effects
@@
 			)
 		)
-		(property "P/N" "~"
+		(property "P/N" "CRCW06030000Z0EE"
 			(at 113.03 99.695 90)
 			(effects

Commit message: Final review..(?)
Parts:
- added H1: M.3, MountingHole:MountingHole_3.2mm_M3_Pad_TopBottom, symbol Mechanical:MountingHole
- PSOM1: P/N (none) -> 53307-2471
Connections:
- net AccelPotRedundant: now also PSOM1.15 (ADC1_IN11); no longer PSOM1.19 (ADC_IN15)
- net AccelPotStatus: now also PSOM1.4 (I2C1_SDA); no longer PSOM1.14 (GPIO_PB14)
- net BrakeFLRedundant: now also PSOM1.13 (ADC1_IN10); no longer PSOM1.7 (ACD1_IN5)
- net BrakeFL_GPIO: now also PSOM1.9 (ADC1_IN7); no longer PSOM1.15 (ADC1_IN11)
- net BrakeFluidStatus: now also PSOM1.6 (I2C1_SCL); no longer PSOM1.16 (GPIO_PB15)
- net BrakePotRedundant: now also PSOM1.19 (SPI1_NSS); no longer PSOM1.9 (ADC1_IN7)
- net BrakePotStatus: now also PSOM1.12 (SPI2_NSS); no longer PSOM1.17 (GPIO_PA12)
- net BrakePot_GPIO: now also PSOM1.7 (OPAMP1_VINP); no longer PSOM1.13 (ADC1_IN10)
- no-connect marks 11 -> 7
Other:
- note added: "Pins Changed"
- note added: "Stuff"
- moved on the sheet: AccelPotStat1, BrakeFLStat1, BrakePotStat1, H2, H3, H4, J1, J6, PWR_+24, R14, R15, R17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

Commit message: Rev B - Initial Layout
Parts:
- added J3: Conn_02x03_Top_Bottom, Connector_Molex:Molex_Nano-Fit_105310-xx06_2x03_P2.50mm_Vertical, symbol Connector_Generic:Conn_02x03_Top_Bottom
- added J4: Conn_02x06_Top_Bottom, Connector_Molex:Molex_Nano-Fit_105310-xx12_2x06_P2.50mm_Vertical, symbol Connector_Generic:Conn_02x06_Top_Bottom
- added J5: Conn_02x04_Top_Bottom, Connector_Molex:Molex_Nano-Fit_105310-xx08_2x04_P2.50mm_Vertical, symbol Connector_Generic:Conn_02x04_Top_Bottom
- J1, J6: now not fitted; now left out of the parts list
Connections:
- net +24V: now also J3.1 (Pin_1); no longer J1.1 (+24V)
- net +5V: now also J4.10 (Pin_10), J4.12 (Pin_12), J4.7 (Pin_7), J4.9 (Pin_9); no longer J6.1 (BrakePot1+), J6.3 (BrakePot2+), J6.4 (AccelPot1+), J6.6 (AccelPot2+)
- net +9V: now also J5.5 (Pin_5), J5.7 (Pin_7); no longer J6.7 (BrakePressure1+), J6.9 (BrakePressure2+)
- net BrakeFL_Main: now also J5.6 (Pin_6); no longer J6.8 (BrakePressureSig1)
- net CANH: now also J3.5 (Pin_5); no longer J1.5 (CANH_OUT)
- net CANL: now also J3.6 (Pin_6); no longer J1.6 (CANL_OUT)
- net GND: now also J3.4 (Pin_4), J5.4 (Pin_4), J5.8 (Pin_8); no longer J1.4 (GND), J6.20
- net GNDA: now also J4.1 (Pin_1), J4.3 (Pin_3), J4.4 (Pin_4), J4.6 (Pin_6), J5.1 (Pin_1), J5.2 (Pin_2); no longer J6.11 (BrakePot1-), J6.13 (BrakePot2-), J6.14 (AccelPot1-), J6.16 (AccelPot2-), J6.17 (BrakePressure1-), J6.19 (BrakePressure2-)
- net at R19.2, R20.2: now also J3.2 (Pin_2); no longer J1.2 (CANH_IN)
- net at R17.2, R18.2: now also J3.3 (Pin_3); no longer J1.3 (CANL_IN)
- removed net AccelPotRedundant: AccelPot1.1, J6.15 (AccelPotSig2), PSOM1.15 (ADC1_IN11)
- net Accel_GPIO renamed BrakeFL_Amp
- net Accel_Main: no longer names the net of J6.5 (AccelPotSig1)
- removed net BrakeFLRedundant: BrakeFL1.1, J6.18 (BrakePresSig2), PSOM1.13 (ADC1_IN10)
- net BrakeFL_GPIO renamed BrakePot_Buff
- removed net BrakePotRedundant: BrakePot1.1, J6.12 (BrakePotSig2), PSOM1.19 (SPI1_NSS)
- net BrakePot_GPIO renamed Accel_Buff
- net BrakePot_Main: no longer names the net of J6.2 (BrakePotSig1)
- new net AccelPotRed: AccelPot1.1, J4.11 (Pin_11)
- new net AccelPotRed_Buff: PSOM1.15 (ADC1_IN11)
- new net Accel_In: J4.5 (Pin_5)
- new net BrakeFLRed: BrakeFL1.1, J5.3 (Pin_3)
- new net BrakeFLRed_Amp: PSOM1.13 (ADC1_IN10)
- new net BrakePotRed: BrakePot1.1, J4.8 (Pin_8)
- new net BrakePotRed_Buff: PSOM1.19 (SPI1_NSS)
- new net BrakePot_In: J4.2 (Pin_2)
- no-connect marks 7 -> 6
Other:
- sheet Brake Fluid Sensor ports: added BrakeFL, BrakeFL_Amp, BrakeFL_Red, BrakeFL_RedAmp; removed BrakeFL_ADC, BrakeFL_GPIO
- sheet Pedals ports: added AccelRed, AccelRed_Buff, Accel_Buff, BrakePotRed, BrakePotRed_Buff, BrakePot_Buff; removed Accel_GPIO, BrakePot_GPIO
- note added: "Misc"
- note removed: "Stuff"
- moved on the sheet: AccelPotStat1, BrakeFLStat1, BrakePotStat1, PWR_+24, R14, R15, R17, R18, R19, R20, R47, R49

Commit message: Rev B - Layout Review
Connections:
- net +5V: now also J4.1 (Pin_1), J4.3 (Pin_3), J4.4 (Pin_4), J4.6 (Pin_6); no longer J4.10 (Pin_10), J4.12 (Pin_12), J4.7 (Pin_7), J4.9 (Pin_9)
- net +9V: now also J5.1 (Pin_1), J5.3 (Pin_3); no longer J5.5 (Pin_5), J5.7 (Pin_7)
- net AccelPotRed: now also J4.8 (Pin_8); no longer J4.11 (Pin_11)
- net Accel_In: now also J4.2 (Pin_2); no longer J4.5 (Pin_5)
- net BrakeFLRed: now also J5.7 (Pin_7); no longer J5.3 (Pin_3)
- net BrakeFL_Main: now also J5.2 (Pin_2); no longer J5.6 (Pin_6)
- net BrakePotRed: now also J4.11 (Pin_11); no longer J4.8 (Pin_8)
- net BrakePot_In: now also J4.5 (Pin_5); no longer J4.2 (Pin_2)
- net GNDA: now also J4.10 (Pin_10), J4.12 (Pin_12), J4.7 (Pin_7), J4.9 (Pin_9), J5.5 (Pin_5), J5.6 (Pin_6); no longer J4.1 (Pin_1), J4.3 (Pin_3), J4.4 (Pin_4), J4.6 (Pin_6), J5.1 (Pin_1), J5.2 (Pin_2)
Other:
- note added: "Nanofit Connectors (Pedals + CAN)"
- note removed: "Mx150 Connectors (Pedals + CAN)"

Commit message: Rev B Sch Review
Parts:
- J3: P/N (none) -> 1053101106
- J4: P/N (none) -> 1053101112
- J5: P/N (none) -> 1053101108
Connections:
- net +9V is gone; now on net +5V: J5.1 (Pin_1), J5.3 (Pin_3)
Changed lines of the file:
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@@
 			)
 		)
+		(property "P/N" "1053101112"
+			(at 140.208 49.022 0)
+			(effects
+				(font
+					(size 1.27 1.27)
+				)
+				(hide yes)
+			)
+		)
 		(pin "1"
 		)
@@
 			)
 		)
+		(property "P/N" "1053101108"
+			(at 140.208 67.818 0)
+			(effects
+				(font
+					(size 1.27 1.27)
+				)
+				(hide yes)
+			)
+		)
 		(pin "4"
 		)
@@
 	)
 	(symbol
+		(lib_id "power:+5V")
+		(at 116.84 63.246 0)
+		(unit 1)
+		(exclude_from_sim no)
+		(in_bom yes)
+		(on_board yes)
+		(dnp no)
+		(property "Reference" "#PWR034"
+			(at 116.84 67.056 0)
+			(effects
+				(font
+					(size 1.27 1.27)
+				)
+				(hide yes)
+			)
+		)
+		(property "Value" "+5V"
+			(at 114.3 60.706 0)
+			(effects
+				(font
+					(size 1.27 1.27)
+				)
+			)
+		)
+		(property "Footprint" ""
+			(at 116.84 63.246 0)
+			(effects
+				(font
+					(size 1.27 1.27)
+				)
+				(hide yes)
+			)
+		)
+		(property "Datasheet" ""
+			(at 116.84 63.246 0)
+			(effects
+				(font
+					(size 1.27 1.27)
+				)
+				(hide yes)
+			)
+		)
+		(property "Description" "Power symbol creates a global label with name \"+5V\""
+			(at 116.84 63.246 0)
+			(effects
+				(font
+					(size 1.27 1.27)
+				)
+				(hide yes)
+			)
+		)
+		(pin "1"
+		)
+		(instances
+			(project "Controls-PedalsDaughter"
+				(path "/30d77876-714b-4f1b-9bad-b74eb43ddcf6"
+					(reference "#PWR034")
+					(unit 1)
+				)
+			)
+		)
+	)
+	(symbol
 		(lib_id "power:GND")
 		(at 128.016 74.168 0)
@@
 	(symbol
 		(lib_id "power:+5V")
-		(at 116.84 41.656 0)
+		(at 61.976 138.43 0)
 		(unit 1)
 		(exclude_from_sim no)
@@
 		(on_board yes)
 		(dnp no)
-		(property "Reference" "#PWR033"
-			(at 116.84 45.466 0)
+		(fields_autoplaced yes)
+		(property "Reference" "#PWR031"
+			(at 61.976 142.24 0)
 			(effects
 				(font
@@
 		)
 		(property "Value" "+5V"
-			(at 114.3 39.116 0)
+			(at 61.976 133.985 0)
 			(effects
 				(font
@@
 		)
 		(property "Footprint" ""
-			(at 116.84 41.656 0)
+			(at 61.976 138.43 0)
 			(effects
 				(font
@@
 		)
 		(property "Datasheet" ""
-			(at 116.84 41.656 0)
+			(at 61.976 138.43 0)
 			(effects
 				(font
@@
 		)
 		(property "Description" "Power symbol creates a global label with name \"+5V\""
-			(at 116.84 41.656 0)
+			(at 61.976 138.43 0)
 			(effects
 				(font
@@
 			(project "Controls-PedalsDaughter"
 				(path "/30d77876-714b-4f1b-9bad-b74eb43ddcf6"
-					(reference "#PWR033")
+					(reference "#PWR031")
 					(unit 1)
 				)
@@
 	)
 	(symbol
-		(lib_id "power:GND")
-		(at 205.232 101.854 0)
+		(lib_id "power:+5V")
+		(at 116.84 41.656 0)
 		(unit 1)
 		(exclude_from_sim no)
@@
 		(on_board yes)
 		(dnp no)
-		(fields_autoplaced yes)
-		(property "Reference" "#PWR08"
-			(at 205.232 108.204 0)
+		(property "Reference" "#PWR033"
+			(at 116.84 45.466 0)
 			(effects
 				(font
@@
 			)
 		)
-		(property "Value" "GND"
-			(at 205.232 106.934 0)
+		(property "Value" "+5V"
+			(at 114.3 39.116 0)
 			(effects
 				(font
 					(size 1.27 1.27)
 				)
-				(hide yes)
 			)
 		)
 		(property "Footprint" ""
-			(at 205.232 101.854 0)
+			(at 116.84 41.656 0)
 			(effects
 				(font
@@
 		)
 		(property "Datasheet" ""
-			(at 205.232 101.854 0)
+			(at 116.84 41.656 0)
 			(effects
 				(font
@@
 			)
 		)
-		(property "Description" "Power symbol creates a global label with name \"GND\" , ground"
-			(at 205.232 101.854 0)
+		(property "Description" "Power symbol creates a global label with name \"+5V\""
+			(at 116.84 41.656 0)
 			(effects
 				(font
@@
 		)
 		(instances
-			(project ""
+			(project "Controls-PedalsDaughter"
 				(path "/30d77876-714b-4f1b-9bad-b74eb43ddcf6"
-					(reference "#PWR08")
+					(reference "#PWR033")
 					(unit 1)
 				)
@@
 	)
 	(symbol
-		(lib_id "power:+9V")
-		(at 61.976 138.43 0)
+		(lib_id "power:GND")
+		(at 205.232 101.854 0)
 		(unit 1)
 		(exclude_from_sim no)
@@
 		(dnp no)
 		(fields_autoplaced yes)
-		(property "Reference" "#PWR031"
-			(at 61.976 142.24 0)
+		(property "Reference" "#PWR08"
+			(at 205.232 108.204 0)
 			(effects
 				(font
@@
 			)
 		)
-		(property "Value" "+9V"
-			(at 61.976 133.985 0)
+		(property "Value" "GND"
+			(at 205.232 106.934 0)
 			(effects
 				(font
 					(size 1.27 1.27)
 				)
+				(hide yes)
 			)
 		)
 		(property "Footprint" ""
-			(at 61.976 138.43 0)
+			(at 205.232 101.854 0)
 			(effects
 				(font
@@
 		)
 		(property "Datasheet" ""
-			(at 61.976 138.43 0)
+			(at 205.232 101.854 0)
 			(effects
 				(font
@@
 			)
 		)
-		(property "Description" "Power symbol creates a global label with name \"+9V\""
-			(at 61.976 138.43 0)
+		(property "Description" "Power symbol creates a global label with name \"GND\" , ground"
+			(at 205.232 101.854 0)
 			(effects
 				(font
@@
 			(project ""
 				(path "/30d77876-714b-4f1b-9bad-b74eb43ddcf6"
-					(reference "#PWR031")
+					(reference "#PWR08")
 					(unit 1)
 				)
@@
 	)
 	(symbol
-		(lib_id "power:+9V")
-		(at 116.84 63.246 0)
-		(unit 1)
-		(exclude_from_sim no)
-		(in_bom yes)
-		(on_board yes)
-		(dnp no)
-		(property "Reference" "#PWR034"
-			(at 116.84 67.056 0)
-			(effects
-				(font
-					(size 1.27 1.27)
-				)
-				(hide yes)
-			)
-		)
-		(property "Value" "+9V"
-			(at 114.3 60.706 0)
-			(effects
-				(font
-					(size 1.27 1.27)
-				)
-			)
-		)
-		(property "Footprint" ""
-			(at 116.84 63.246 0)
-			(effects
-				(font
-					(size 1.27 1.27)
-				)
-				(hide yes)
-			)
-		)
-		(property "Datasheet" ""
-			(at 116.84 63.246 0)
-			(effects
-				(font
-					(size 1.27 1.27)
-				)
-				(hide yes)
-			)
-		)
-		(property "Description" "Power symbol creates a global label with name \"+9V\""
-			(at 116.84 63.246 0)
-			(effects
-				(font
-					(size 1.27 1.27)
-				)
-				(hide yes)
-			)
-		)
-		(pin "1"
-		)
-		(instances
-			(project "Controls-PedalsDaughter"
-				(path "/30d77876-714b-4f1b-9bad-b74eb43ddcf6"
-					(reference "#PWR034")
-					(unit 1)
-				)
-			)
-		)
-	)
-	(symbol
 		(lib_id "Connector:TestPoint")
 		(at 194.31 135.89 90)
@@
 			(at 147.574 87.884 0)
 			(effects
+				(font
+					(size 1.27 1.27)
+				)
+				(hide yes)
+			)
+		)
+		(property "P/N" "1053101106"
+			(at 147.574 87.884 0)
+			(effects

Commit message: Rev B Layout #2
Parts:
- removed AccelPot1: AccelPotSig, TestPoint:TestPoint_THTPad_1.5x1.5mm_Drill0.7mm, symbol Connector:TestPoint
- removed BrakeFL1: BrakeFLSig, TestPoint:TestPoint_THTPad_1.5x1.5mm_Drill0.7mm, symbol Connector:TestPoint
- removed BrakePot1: BrakePotSig, TestPoint:TestPoint_THTPad_1.5x1.5mm_Drill0.7mm, symbol Connector:TestPoint
Connections:
- net +5V: no longer J5.1 (Pin_1), J5.3 (Pin_3)
- new net 5V_BrakeFL: J5.1 (Pin_1), J5.3 (Pin_3)
- no-connect marks 6 -> 32
