File: hardware/VCAT-PedalBoxPCB/power.kicad_sch (KiCad schematic)
At the start: 0 parts

Commit message: sch too ez
Parts:
- added C13, C5: C, symbol Device:C
- added R6: 3.16k, symbol Device:R
- added R7, R9: 10k, symbol Device:R
- added R8: 1.54k, symbol Device:R
- added U2, U6: LDO40LPURY, Package_DFN_QFN:DFN-6-1EP_3x3mm_P0.95mm_EP1.7x2.6mm, symbol Regulator_Linear:LDO40LPURY
Connections:
- new net: R8.2, R9.1, U6.6 (ADJ)
- new net: R6.2, R7.1, U2.6 (ADJ)
- new net +24V: C13.1, C5.1, U2.3 (Vin), U6.3 (Vin)
- new net +3.3V: U2.2 (EN), U6.2 (EN)
- new net GND: C13.2, C5.2, R7.2, R9.2, U2.1 (GND), U2.7 (GND), U6.1 (GND), U6.7 (GND)
- new net VoutAdj1: R6.1, U2.4 (Vout), U2.5 (Vsense)
- new net VoutAdj2: R8.1, U6.4 (Vout), U6.5 (Vsense)
Other:
- note added: "1.11k -> 12V"
- note added: "1.54k -> 9V"
- note added: "3.16k -> 5V"
- note added: "5V"
- note added: "9V"
- note added: "R8 = -R9 + (R9/(1-(Vref/Vout)))"
- note added: "Vref = 1.2V Vref = Vout - Vadj Vout(R7/R6+R7) = Vadj Therefore, Vref/(1-(R7/R7+R6)) = Vout"

Commit message: final review?? (plssss)
Parts:
- removed C13: C, symbol Device:C
- added C4, C7, C8: 1uF, symbol Device:C
- added R10, R13: 1k, symbol Device:R
- C5: value C -> 1uF
Connections:
- net +24V: now also C7.1, R10.1, R13.1
- net GND: now also C4.2, C7.2, C8.2
- net VoutAdj1: now also C4.1
- net VoutAdj2: now also C8.1
- net +3.3V: no longer names the net of U2.2 (EN)
- net +3.3V: now also R10.2; no longer U6.2 (EN)
- new net: R13.2, U6.2 (EN)

Commit message: PSOM pin layout pic
Other:
- note added: "Adjustable LDOs"
Changed lines of the file:
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@@
 	(generator_version "9.0")
 	(paper "A4")
+	(rectangle
+		(start 88.265 60.325)
+		(end 217.17 137.16)
+		(stroke
+			(width 0)
+			(type default)
+		)
+		(fill
+			(type none)
+		)
+	)
 	(text "9V"
 		(exclude_from_sim no)
@@
 			)
 		)
+	)
+	(text "Adjustable LDOs"
+		(exclude_from_sim no)
+		(at 106.68 56.515 0)
+		(effects
+			(font
+				(size 3 3)
+				(thickness 0.4)
+				(bold yes)
+			)
+		)

Commit message: pcb design review #1
Parts:
- C4, C5, C7, C8: footprint (none) -> Capacitor_SMD:C_0603_1608Metric_Pad1.08x0.95mm_HandSolder
- R10, R13, R6, R7, R8, R9: footprint (none) -> Resistor_SMD:R_0603_1608Metric_Pad0.98x0.95mm_HandSolder
Changed lines of the file:
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@@
 			)
 		)
-		(property "Footprint" ""
+		(property "Footprint" "Resistor_SMD:R_0603_1608Metric_Pad0.98x0.95mm_HandSolder"
 			(at 104.267 74.295 90)
 			(effects
@@
 			)
 		)
-		(property "Footprint" ""
+		(property "Footprint" "Resistor_SMD:R_0603_1608Metric_Pad0.98x0.95mm_HandSolder"
 			(at 141.732 125.095 90)
 			(effects
@@
 			)
 		)
-		(property "Footprint" ""
+		(property "Footprint" "Resistor_SMD:R_0603_1608Metric_Pad0.98x0.95mm_HandSolder"
 			(at 141.097 84.455 90)
 			(effects
@@
 			)
 		)
-		(property "Footprint" ""
+		(property "Footprint" "Capacitor_SMD:C_0603_1608Metric_Pad1.08x0.95mm_HandSolder"
 			(at 101.9302 81.28 0)
 			(effects
@@
 			)
 		)
-		(property "Footprint" ""
+		(property "Footprint" "Capacitor_SMD:C_0603_1608Metric_Pad1.08x0.95mm_HandSolder"
 			(at 155.9052 122.555 0)
 			(effects
@@
 			)
 		)
-		(property "Footprint" ""
+		(property "Footprint" "Resistor_SMD:R_0603_1608Metric_Pad0.98x0.95mm_HandSolder"
 			(at 141.097 76.835 90)
 			(effects
@@
 			)
 		)
-		(property "Footprint" ""
+		(property "Footprint" "Capacitor_SMD:C_0603_1608Metric_Pad1.08x0.95mm_HandSolder"
 			(at 102.5652 121.92 0)
 			(effects
@@
 			)
 		)
-		(property "Footprint" ""
+		(property "Footprint" "Resistor_SMD:R_0603_1608Metric_Pad0.98x0.95mm_HandSolder"
 			(at 141.732 117.475 90)
 			(effects
@@
 			)
 		)
-		(property "Footprint" ""
+		(property "Footprint" "Capacitor_SMD:C_0603_1608Metric_Pad1.08x0.95mm_HandSolder"
 			(at 154.0002 81.915 0)
 			(effects
@@
 			)
 		)
-		(property "Footprint" ""
+		(property "Footprint" "Resistor_SMD:R_0603_1608Metric_Pad0.98x0.95mm_HandSolder"
 			(at 104.902 114.935 90)
 			(effects

Commit message: updated BOM
Parts:
- C4, C5, C7, C8: P/N (none) -> MLASU168SB5105KTNA01
- R10, R13: P/N (none) -> CRCW06031K00FKEI
- R6: P/N (none) -> ERJ-S03F3161V
- R7, R9: P/N (none) -> CRCW060310K0FKEI
- R8: P/N (none) -> CRCW06031K54FKEAC
- U2, U6: P/N (none) -> LDO40LPURY
Changed lines of the file:
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@@
 			)
 		)
-		(property "Description" "Resistor"
+		(property "Description" "Pedals 1k ohms"
 			(at 106.045 74.295 0)
 			(effects
@@
 		)
 		(property "p/n" ""
+			(at 106.045 74.295 0)
+			(effects
+				(font
+					(size 1.27 1.27)
+				)
+				(hide yes)
+			)
+		)
+		(property "P/N" "CRCW06031K00FKEI "
 			(at 106.045 74.295 0)
 			(effects
@@
 			)
 		)
-		(property "Description" "Resistor"
+		(property "Description" "Pedals 10K Ohms"
 			(at 143.51 125.095 0)
 			(effects
@@
 		)
 		(property "p/n" ""
+			(at 143.51 125.095 0)
+			(effects
+				(font
+					(size 1.27 1.27)
+				)
+				(hide yes)
+			)
+		)
+		(property "P/N" "CRCW060310K0FKEI "
 			(at 143.51 125.095 0)
 			(effects
@@
 			)
 		)
-		(property "Description" "Resistor"
+		(property "Description" "Pedals 10K Ohms"
 			(at 142.875 84.455 0)
 			(effects
@@
 		)
 		(property "p/n" ""
+			(at 142.875 84.455 0)
+			(effects
+				(font
+					(size 1.27 1.27)
+				)
+				(hide yes)
+			)
+		)
+		(property "P/N" "CRCW060310K0FKEI "
 			(at 142.875 84.455 0)
 			(effects
@@
 			)
 		)
-		(property "Description" "Unpolarized capacitor"
+		(property "Description" "Pedals 5v LDO C5 cap"
 			(at 100.965 77.47 0)
 			(effects
@@
 		)
 		(property "p/n" ""
+			(at 100.965 77.47 0)
+			(effects
+				(font
+					(size 1.27 1.27)
+				)
+				(hide yes)
+			)
+		)
+		(property "P/N" "MLASU168SB5105KTNA01"
 			(at 100.965 77.47 0)
 			(effects
@@
 			)
 		)
-		(property "Description" "Unpolarized capacitor"
+		(property "Description" "Pedals 5v LDO C5 cap"
 			(at 154.94 118.745 0)
 			(effects
@@
 		)
 		(property "p/n" ""
+			(at 154.94 118.745 0)
+			(effects
+				(font
+					(size 1.27 1.27)
+				)
+				(hide yes)
+			)
+		)
+		(property "P/N" "MLASU168SB5105KTNA01"
 			(at 154.94 118.745 0)
 			(effects
@@
 			)
 		)
-		(property "Description" "400mA, 3.5V-38V input, 2.5V-11V output, adjustable positive LDO regulator with enable, DFN-6"
+		(property "Description" "LDO40LPURY"
 			(at 127.635 116.205 0)
 			(effects
@@
 		)
 		(property "p/n" ""
+			(at 127.635 116.205 0)
+			(effects
+				(font
+					(size 1.27 1.27)
+				)
+				(hide yes)
+			)
+		)
+		(property "P/N" "LDO40LPURY"
 			(at 127.635 116.205 0)
 			(effects
@@
 			)
 		)
-		(property "Description" "Resistor"
+		(property "Description" "Pedals 5v LDO 3.16 ohms"
 			(at 142.875 76.835 0)
 			(effects
@@
 		)
 		(property "p/n" ""
+			(at 142.875 76.835 0)
+			(effects
+				(font
+					(size 1.27 1.27)
+				)
+				(hide yes)
+			)
+		)
+		(property "P/N" "ERJ-S03F3161V"
 			(at 142.875 76.835 0)
 			(effects
@@
 			)
 		)
-		(property "Description" "Unpolarized capacitor"
+		(property "Description" "Pedals 5v LDO C5 cap"
 			(at 101.6 118.11 0)
 			(effects
@@
 		)
 		(property "p/n" ""
+			(at 101.6 118.11 0)
+			(effects
+				(font
+					(size 1.27 1.27)
+				)
+				(hide yes)
+			)
+		)
+		(property "P/N" "MLASU168SB5105KTNA01"
 			(at 101.6 118.11 0)
 			(effects
@@
 			)
 		)
-		(property "Description" "400mA, 3.5V-38V input, 2.5V-11V output, adjustable positive LDO regulator with enable, DFN-6"
+		(property "Description" "LDO40LPURY"
 			(at 127 75.565 0)
 			(effects
@@
 		)
 		(property "p/n" ""
+			(at 127 75.565 0)
+			(effects
+				(font
+					(size 1.27 1.27)
+				)
+				(hide yes)
+			)
+		)
+		(property "P/N" "LDO40LPURY"
 			(at 127 75.565 0)
 			(effects
@@
 			)
 		)
-		(property "Description" "Resistor"
+		(property "Description" "Pedals 9v LDO 1.54 ohms"
 			(at 143.51 117.475 0)
 			(effects
@@
 		)
 		(property "p/n" ""
+			(at 143.51 117.475 0)
+			(effects
+				(font
+					(size 1.27 1.27)
+				)
+				(hide yes)
+			)
+		)
+		(property "P/N" "CRCW06031K54FKEAC"
 			(at 143.51 117.475 0)
 			(effects
@@
 			)
 		)
-		(property "Description" "Unpolarized capacitor"
+		(property "Description" "Pedals 5v LDO C5 cap"
 			(at 153.035 78.105 0)
 			(effects
@@
 		)
 		(property "p/n" ""
+			(at 153.035 78.105 0)
+			(effects
+				(font
+					(size 1.27 1.27)
+				)
+				(hide yes)
+			)
+		)
+		(property "P/N" "MLASU168SB5105KTNA01"
 			(at 153.035 78.105 0)
 			(effects
@@
 			)
 		)
-		(property "Description" "Resistor"
+		(property "Description" "Pedals 1k ohms"
 			(at 106.68 114.935 0)
 			(effects
@@
 			(at 106.68 114.935 0)
 			(effects
+				(font
+					(size 1.27 1.27)
+				)
+				(hide yes)
+			)
+		)
+		(property "P/N" "CRCW06031K00FKEI "
+			(at 106.68 114.935 0)
+			(effects

Commit message: bruh2
Parts:
- added TP1: Vin, TestPoint:TestPoint_Pad_1.0x1.0mm, symbol Connector:TestPoint
- added TP10: 9V_Out, TestPoint:TestPoint_Pad_1.0x1.0mm, symbol Connector:TestPoint
- added TP2: Enable5V, TestPoint:TestPoint_Pad_1.0x1.0mm, symbol Connector:TestPoint
- added TP3: GND, TestPoint:TestPoint_Pad_1.0x1.0mm, symbol Connector:TestPoint
- added TP5: Adj5V, TestPoint:TestPoint_Pad_1.0x1.0mm, symbol Connector:TestPoint
- added TP6: 5V_Out, TestPoint:TestPoint_Pad_1.0x1.0mm, symbol Connector:TestPoint
- added TP7: Enable9V, TestPoint:TestPoint_Pad_1.0x1.0mm, symbol Connector:TestPoint
- added TP9: Adj9V, TestPoint:TestPoint_Pad_1.0x1.0mm, symbol Connector:TestPoint
Connections:
- net +24V: now also TP1.1
- net GND: now also TP3.1
- net VoutAdj1: now also TP6.1
- net VoutAdj2: now also TP10.1
- net at R10.2, U2.2 (EN): now also TP2.1
- net at R8.2, R9.1, U6.6 (ADJ): now also TP9.1
- net at R6.2, R7.1, U2.6 (ADJ): now also TP5.1
- net at R13.2, U6.2 (EN): now also TP7.1

Commit message: Rev B Sch updates
Parts:
- removed TP10: 9V_Out, TestPoint:TestPoint_Pad_1.0x1.0mm, symbol Connector:TestPoint
- removed TP3: GND, TestPoint:TestPoint_Pad_1.0x1.0mm, symbol Connector:TestPoint
- removed TP7: Enable9V, TestPoint:TestPoint_Pad_1.0x1.0mm, symbol Connector:TestPoint
- removed TP9: Adj9V, TestPoint:TestPoint_Pad_1.0x1.0mm, symbol Connector:TestPoint
- added 9V_Out1: 5V_Out, TestPoint:TestPoint_Pad_1.0x1.0mm, symbol Connector:TestPoint
- added Adj9V1: Adj5V, TestPoint:TestPoint_Pad_1.0x1.0mm, symbol Connector:TestPoint
- added En9V1: Enable5V, TestPoint:TestPoint_Pad_1.0x1.0mm, symbol Connector:TestPoint
- added GND1: Vin, TestPoint:TestPoint_Pad_1.0x1.0mm, symbol Connector:TestPoint
- renumbered TP6 to 5V_Out1, TP5 to Adj5V1, TP2 to En5V1, TP1 to Vin1
Connections:
- net GND: now also GND1.1
- net VoutAdj2: now also 9V_Out1.1
- net at R8.2, R9.1, U6.6 (ADJ): now also Adj9V1.1
- net at R13.2, U6.2 (EN): now also En9V1.1
Other:
- moved on the sheet: C7, C8, R13, R8, R9, U6
