File: hardware/VCAT-PedalBoxPCB/power.kicad_sch (KiCad schematic)
At the start: 20 parts, among them U2 LDO40LPURY, U6 LDO40LPURY

Commit message: Rev B - Initial Layout
Changed lines of the file:
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@@
+	)
+	(junction
+		(at 100.838 109.474)
+		(diameter 0)
+		(color 0 0 0 0)
 	)
 	(junction
@@
 	)
 	(junction
-		(at 100.838 109.474)
-		(diameter 0)
-		(color 0 0 0 0)
-	)
-	(junction
 		(at 107.188 117.094)
 		(diameter 0)
@@
 	)
 	(junction
+		(at 101.092 70.612)
+		(diameter 0)
+		(color 0 0 0 0)
+	)
+	(junction
 		(at 127 88.392)
 		(diameter 0)
@@
 	)
 	(junction
-		(at 101.092 70.612)
-		(diameter 0)
-		(color 0 0 0 0)
-	)
-	(junction
 		(at 150.876 70.612)
 		(diameter 0)
@@
 	(wire
 		(pts
+			(xy 98.552 69.596) (xy 98.552 70.104)
+		)
+		(stroke
+			(width 0)
+			(type default)
+		)
+	)
+	(wire
+		(pts
+			(xy 98.552 70.104) (xy 99.06 70.612)
+		)
+		(stroke
+			(width 0)
+			(type default)
+		)
+	)
+	(wire
+		(pts
 			(xy 143.002 88.392) (xy 151.13 88.392)
 		)
@@
 	(wire
 		(pts
-			(xy 98.552 70.612) (xy 101.092 70.612)
-		)
-		(stroke
-			(width 0)
-			(type default)
-		)
-	)
-	(wire
-		(pts
 			(xy 150.368 109.474) (xy 154.178 109.474)
 		)
@@
 	(wire
 		(pts
-			(xy 98.298 109.474) (xy 100.838 109.474)
-		)
-		(stroke
-			(width 0)
-			(type default)
-		)
-	)
-	(wire
-		(pts
 			(xy 153.162 86.36) (xy 151.13 88.392)
 		)
@@
 	(wire
 		(pts
+			(xy 98.298 108.966) (xy 98.806 109.474)
+		)
+		(stroke
+			(width 0)
+			(type default)
+		)
+	)
+	(wire
+		(pts
 			(xy 110.744 70.612) (xy 114.3 70.612)
 		)
@@
 	(wire
 		(pts
+			(xy 99.06 70.612) (xy 101.092 70.612)
+		)
+		(stroke
+			(width 0)
+			(type default)
+		)
+	)
+	(wire
+		(pts
 			(xy 139.7 114.554) (xy 140.208 114.554)
 		)
@@
 	(wire
 		(pts
+			(xy 98.806 109.474) (xy 100.838 109.474)
+		)
+		(stroke
+			(width 0)
+			(type default)
+		)
+	)
+	(wire
+		(pts
 			(xy 139.7 70.612) (xy 140.462 70.612)
 		)
@@
 		(pts
 			(xy 101.092 70.612) (xy 101.092 73.66)
+		)
+		(stroke
+			(width 0)
+			(type default)
+		)
+	)
+	(wire
+		(pts
+			(xy 98.298 108.458) (xy 98.298 108.966)
 		)
 		(stroke
@@
 				(path "/30d77876-714b-4f1b-9bad-b74eb43ddcf6/6613b086-4f9a-483f-8869-58f1a430ca82"
 					(reference "C5")
-					(unit 1)
-				)
-			)
-		)
-	)
-	(symbol
-		(lib_id "power:+24V")
-		(at 98.552 70.612 0)
-		(unit 1)
-		(exclude_from_sim no)
-		(in_bom yes)
-		(on_board yes)
-		(dnp no)
-		(property "Reference" "#PWR018"
-			(at 98.552 74.422 0)
-			(effects
-				(font
-					(size 1.27 1.27)
-				)
-				(hide yes)
-			)
-		)
-		(property "Value" "+24V"
-			(at 94.742 68.072 0)
-			(effects
-				(font
-					(size 1.27 1.27)
-				)
-			)
-		)
-		(property "Footprint" ""
-			(at 98.552 70.612 0)
-			(effects
-				(font
-					(size 1.27 1.27)
-				)
-				(hide yes)
-			)
-		)
-		(property "Datasheet" ""
-			(at 98.552 70.612 0)
-			(effects
-				(font
-					(size 1.27 1.27)
-				)
-				(hide yes)
-			)
-		)
-		(property "Description" "Power symbol creates a global label with name \"+24V\""
-			(at 98.552 70.612 0)
-			(effects
-				(font
-					(size 1.27 1.27)
-				)
-				(hide yes)
-			)
-		)
-		(pin "1"
-		)
-		(instances
-			(project ""
-				(path "/30d77876-714b-4f1b-9bad-b74eb43ddcf6/6613b086-4f9a-483f-8869-58f1a430ca82"
-					(reference "#PWR018")
 					(unit 1)
 				)
@@
 	(symbol
 		(lib_id "power:+24V")
-		(at 98.298 109.474 0)
+		(at 98.298 108.458 0)
 		(unit 1)
 		(exclude_from_sim no)
@@
 		(dnp no)
 		(property "Reference" "#PWR022"
-			(at 98.298 113.284 0)
+			(at 98.298 112.268 0)
 			(effects
 				(font
@@
 		)
 		(property "Value" "+24V"
-			(at 94.488 106.934 0)
+			(at 94.488 105.918 0)
 			(effects
 				(font
@@
 		)
 		(property "Footprint" ""
-			(at 98.298 109.474 0)
+			(at 98.298 108.458 0)
 			(effects
 				(font
@@
 		)
 		(property "Datasheet" ""
-			(at 98.298 109.474 0)
+			(at 98.298 108.458 0)
 			(effects
 				(font
@@
 		)
 		(property "Description" "Power symbol creates a global label with name \"+24V\""
-			(at 98.298 109.474 0)
+			(at 98.298 108.458 0)
 			(effects
 				(font
@@
 					(unit 1)
 				)
+			)
+		)
+	)
+	(symbol
+		(lib_id "power:+24V")
+		(at 98.552 69.596 0)
+		(unit 1)
+		(exclude_from_sim no)
+		(in_bom yes)
+		(on_board yes)
+		(dnp no)
+		(property "Reference" "#PWR015"
+			(at 98.552 73.406 0)
+			(effects
+				(font
+					(size 1.27 1.27)
+				)
+				(hide yes)
+			)
+		)
+		(property "Value" "+24V"
+			(at 94.742 67.056 0)
+			(effects
+				(font
+					(size 1.27 1.27)
+				)
+			)
+		)
+		(property "Footprint" ""
+			(at 98.552 69.596 0)
+			(effects
+				(font
+					(size 1.27 1.27)
+				)
+				(hide yes)
+			)
+		)
+		(property "Datasheet" ""
+			(at 98.552 69.596 0)
+			(effects
+				(font
+					(size 1.27 1.27)
+				)
+				(hide yes)
+			)
+		)
+		(property "Description" "Power symbol creates a global label with name \"+24V\""
+			(at 98.552 69.596 0)
+			(effects
+				(font
+					(size 1.27 1.27)
+				)
+				(hide yes)
+			)
+		)
+		(pin "1"
+		)
+		(instances
+			(project "Controls-PedalsDaughter"
+				(path "/30d77876-714b-4f1b-9bad-b74eb43ddcf6/6613b086-4f9a-483f-8869-58f1a430ca82"
+					(reference "#PWR015")
+					(unit 1)
+				)

Commit message: Rev B - Layout Review
Parts:
- R6: value 3.16k -> 1.54k
- R8: value 1.54k -> 3.16k
- renumbered 9V_Out1 to 5V_Out1, 5V_Out1 to 9V_Out1, Adj9V1 to Adj5V1, Adj5V1 to Adj9V1, En9V1 to En5V1, En5V1 to En9V1
Connections:
- net VoutAdj1: now also 5V_Out1.1, C8.1, R8.1, U6.4 (Vout), U6.5 (Vsense); no longer 9V_Out1.1, C4.1, R6.1, U2.4 (Vout), U2.5 (Vsense)
- net VoutAdj2: now also 9V_Out1.1, C4.1, R6.1, U2.4 (Vout), U2.5 (Vsense); no longer 5V_Out1.1, C8.1, R8.1, U6.4 (Vout), U6.5 (Vsense)
Other:
- moved on the sheet: 5V_Out1, 9V_Out1
Changed lines of the file:
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@@
 	(text "9V"
 		(exclude_from_sim no)
-		(at 162.56 106.934 0)
+		(at 160.782 67.818 0)
 		(effects
 			(font
@@
 	(text "5V"
 		(exclude_from_sim no)
-		(at 160.782 68.072 0)
+		(at 162.814 106.934 0)
 		(effects
 			(font
@@
 	)
 	(junction
+		(at 148.336 70.612)
+		(diameter 0)
+		(color 0 0 0 0)
+	)
+	(junction
 		(at 140.208 109.474)
 		(diameter 0)
@@
 	)
 	(junction
-		(at 150.368 109.474)
+		(at 142.748 127.254)
 		(diameter 0)
 		(color 0 0 0 0)
 	)
 	(junction
-		(at 142.748 127.254)
+		(at 149.606 109.474)
 		(diameter 0)
 		(color 0 0 0 0)
@@
 	)
 	(junction
+		(at 107.442 78.232)
+		(diameter 0)
+		(color 0 0 0 0)
+	)
+	(junction
 		(at 107.188 117.094)
 		(diameter 0)
@@
 	)
 	(junction
-		(at 107.442 78.232)
-		(diameter 0)
-		(color 0 0 0 0)
-	)
-	(junction
 		(at 143.002 80.772)
 		(diameter 0)
@@
 	)
 	(junction
-		(at 150.876 70.612)
-		(diameter 0)
-		(color 0 0 0 0)
-	)
-	(junction
 		(at 154.178 109.474)
 		(diameter 0)
@@
 	(wire
 		(pts
-			(xy 142.748 109.474) (xy 150.368 109.474)
+			(xy 149.606 109.474) (xy 154.178 109.474)
+		)
+		(stroke
+			(width 0)
+			(type default)
+		)
+	)
+	(wire
+		(pts
+			(xy 142.748 109.474) (xy 149.606 109.474)
 		)
 		(stroke
@@
 	(wire
 		(pts
-			(xy 150.368 109.474) (xy 154.178 109.474)
-		)
-		(stroke
-			(width 0)
-			(type default)
-		)
-	)
-	(wire
-		(pts
 			(xy 153.162 86.36) (xy 151.13 88.392)
 		)
@@
 	(wire
 		(pts
-			(xy 150.876 70.612) (xy 153.162 70.612)
-		)
-		(stroke
-			(width 0)
-			(type default)
-		)
-	)
-	(wire
-		(pts
 			(xy 109.728 114.554) (xy 114.3 114.554)
 		)
@@
 	(wire
 		(pts
-			(xy 143.002 70.612) (xy 150.876 70.612)
+			(xy 143.002 70.612) (xy 148.336 70.612)
 		)
 		(stroke
@@
 		(pts
 			(xy 154.178 125.222) (xy 152.4 127.254)
+		)
+		(stroke
+			(width 0)
+			(type default)
+		)
+	)
+	(wire
+		(pts
+			(xy 148.336 70.612) (xy 153.162 70.612)
 		)
 		(stroke
@@
 	(hierarchical_label "VoutAdj2"
 		(shape output)
-		(at 157.988 109.474 0)
+		(at 155.702 70.612 0)
 		(effects
 			(font
@@
 	(hierarchical_label "VoutAdj1"
 		(shape output)
-		(at 155.702 70.612 0)
+		(at 157.988 109.474 0)
 		(effects
 			(font
@@
 		(on_board yes)
 		(dnp no)
-		(property "Reference" "Adj9V1"
+		(property "Reference" "Adj5V1"
 			(at 145.542 121.666 90)
 			(effects
@@
 			(project "Controls-PedalsDaughter"
 				(path "/30d77876-714b-4f1b-9bad-b74eb43ddcf6/6613b086-4f9a-483f-8869-58f1a430ca82"
-					(reference "Adj9V1")
+					(reference "Adj5V1")
 					(unit 1)
 				)
@@
 	(symbol
 		(lib_id "Connector:TestPoint")
-		(at 150.368 109.474 0)
+		(at 149.606 109.474 0)
 		(unit 1)
 		(exclude_from_sim no)
@@
 		(on_board yes)
 		(dnp no)
-		(property "Reference" "9V_Out1"
-			(at 153.924 103.378 0)
+		(property "Reference" "5V_Out1"
+			(at 153.162 103.378 0)
 			(effects
 				(font
@@
 		)
 		(property "Value" "5V_Out"
-			(at 153.162 103.886 0)
+			(at 152.4 103.886 0)
 			(effects
 				(font
@@
 		)
 		(property "Footprint" "TestPoint:TestPoint_Pad_1.0x1.0mm"
-			(at 155.448 109.474 0)
+			(at 154.686 109.474 0)
 			(effects
 				(font
@@
 		)
 		(property "Datasheet" "~"
-			(at 155.448 109.474 0)
+			(at 154.686 109.474 0)
 			(effects
 				(font
@@
 		)
 		(property "Description" "test point"
-			(at 150.368 109.474 0)
+			(at 149.606 109.474 0)
 			(effects
 				(font
@@
 			(project "Controls-PedalsDaughter"
 				(path "/30d77876-714b-4f1b-9bad-b74eb43ddcf6/6613b086-4f9a-483f-8869-58f1a430ca82"
-					(reference "9V_Out1")
+					(reference "5V_Out1")
 					(unit 1)
 				)
@@
 		(on_board yes)
 		(dnp no)
-		(property "Reference" "En9V1"
+		(property "Reference" "En5V1"
 			(at 109.474 122.936 0)
 			(effects
@@
 			(project "Controls-PedalsDaughter"
 				(path "/30d77876-714b-4f1b-9bad-b74eb43ddcf6/6613b086-4f9a-483f-8869-58f1a430ca82"
-					(reference "En9V1")
+					(reference "En5V1")
 					(unit 1)
 				)
@@
 		(fields_autoplaced yes)
 		(property "Reference" "R6"
-			(at 144.907 75.6919 0)
+			(at 144.78 75.6919 0)
 			(effects
 				(font
@@
 			)
 		)
-		(property "Value" "3.16k"
-			(at 144.907 78.2319 0)
+		(property "Value" "1.54k"
+			(at 144.78 78.2319 0)
 			(effects
 				(font
@@
 		(on_board yes)
 		(dnp no)
-		(property "Reference" "En5V1"
+		(property "Reference" "En9V1"
 			(at 109.728 84.074 0)
 			(effects
@@
 			(project "Controls-PedalsDaughter"
 				(path "/30d77876-714b-4f1b-9bad-b74eb43ddcf6/6613b086-4f9a-483f-8869-58f1a430ca82"
-					(reference "En5V1")
+					(reference "En9V1")
 					(unit 1)
 				)
@@
 		(on_board yes)
 		(dnp no)
-		(property "Reference" "Adj5V1"
+		(property "Reference" "Adj9V1"
 			(at 145.796 82.804 90)
 			(effects
@@
 			(project "Controls-PedalsDaughter"
 				(path "/30d77876-714b-4f1b-9bad-b74eb43ddcf6/6613b086-4f9a-483f-8869-58f1a430ca82"
-					(reference "Adj5V1")
+					(reference "Adj9V1")
 					(unit 1)
 				)
@@
 			)
 		)
-		(property "Value" "1.54k"
+		(property "Value" "3.16k"
 			(at 144.653 117.094 0)
 			(effects
@@
 	(symbol
 		(lib_id "Connector:TestPoint")
-		(at 150.876 70.612 0)
+		(at 148.336 70.612 0)
 		(unit 1)
 		(exclude_from_sim no)
@@
 		(on_board yes)
 		(dnp no)
-		(property "Reference" "5V_Out1"
-			(at 153.924 65.024 0)
+		(property "Reference" "9V_Out1"
+			(at 151.384 65.024 0)
 			(effects
 				(font
@@
 		)
 		(property "Value" "5V_Out"
-			(at 153.67 65.024 0)
+			(at 151.13 65.024 0)
 			(effects
 				(font
@@
 		)
 		(property "Footprint" "TestPoint:TestPoint_Pad_1.0x1.0mm"
-			(at 155.956 70.612 0)
+			(at 153.416 70.612 0)
 			(effects
 				(font
@@
 		)
 		(property "Datasheet" "~"
-			(at 155.956 70.612 0)
+			(at 153.416 70.612 0)
 			(effects
 				(font
@@
 		)
 		(property "Description" "test point"
-			(at 150.876 70.612 0)
+			(at 148.336 70.612 0)
 			(effects
 				(font
@@
 			(project "Controls-PedalsDaughter"
 				(path "/30d77876-714b-4f1b-9bad-b74eb43ddcf6/6613b086-4f9a-483f-8869-58f1a430ca82"
-					(reference "5V_Out1")
+					(reference "9V_Out1")
 					(unit 1)
 				)

Commit message: Layout DONEEEE
Parts:
- added IC1: ADP7182AUJZ-R7, ADP7182AUJZ-R7:SOT95P280X100-5N, symbol ADP7182AUJZ-R7:ADP7182AUJZ-R7
Connections:
- net VoutAdj1: no longer 5V_Out1.1, C8.1, R8.1, U6.4 (Vout), U6.5 (Vsense)
- net VoutAdj2: no longer 9V_Out1.1, C4.1, R6.1, U2.4 (Vout), U2.5 (Vsense)
- new net: 5V_Out1.1, C8.1, R8.1, U6.4 (Vout), U6.5 (Vsense)
- new net: 9V_Out1.1, C4.1, R6.1, U2.4 (Vout), U2.5 (Vsense)
Other:
- moved on the sheet: 5V_Out1, 9V_Out1, Adj5V1, Adj9V1, C4, C5, C7, C8, En5V1, En9V1, GND1, R10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

Commit message: uhh couple more changes, now its done
Parts:
- removed GND1: Vin, TestPoint:TestPoint_Pad_1.0x1.0mm, symbol Connector:TestPoint
- removed IC1: ADP7182AUJZ-R7, ADP7182AUJZ-R7:SOT95P280X100-5N, symbol ADP7182AUJZ-R7:ADP7182AUJZ-R7
- removed U2, U6: LDO40LPURY, Package_DFN_QFN:DFN-6-1EP_3x3mm_P0.95mm_EP1.7x2.6mm, symbol Regulator_Linear:LDO40LPURY
- added C15: 10uF, Capacitor_SMD:C_0603_1608Metric_Pad1.08x0.95mm_HandSolder, symbol Device:C
- added C16: 2.2uF, Capacitor_SMD:C_0603_1608Metric_Pad1.08x0.95mm_HandSolder, symbol Device:C
- added IC1, IC2: AP2205-W5-7, AP2205W57, symbol AP2205-W5-7:AP2205-W5-7
- C4: value 1uF -> 10uF
- C7: value 1uF -> 2.2uF
- R10: value 1k -> 10k
- R13: value 1k -> 10k; P/N CRCW06031K00FKEI -> CRCW060310K0FKEI
- R6: value 1.54k -> 30k; P/N ERJ-S03F3161V -> 0603WAJ0303T5E
- R8: value 3.16k -> 10k; P/N CRCW06031K54FKEAC -> CRCW06031K00FKEI
- R9: value 10k -> 63.4k; P/N CRCW060310K0FKEI -> RC0603FR-0763K4L
Connections:
- net +24V: now also C5.2, C8.2, R8.1, IC1.1 (VIN), IC2.1 (VIN); no longer C5.1, C7.1, R13.1
- net GND: now also C4.1, C5.1, C8.1, R13.2, C15.1, C16.2, IC1.2 (GND), IC2.2 (GND); no longer C4.2, C5.2, C8.2, R9.2
- net VoutAdj1: now also 5V_Out1.1, C7.1, R6.1, IC1.5 (VOUT)
- net VoutAdj2: now also 9V_Out1.1, R9.1, C16.1, IC2.5 (VOUT)
- net at R10.2: now also C4.2, En5V1.1, IC1.3 (EN); no longer En9V1.1
- net at R6.2, R7.1: now also Adj5V1.1, IC1.4 (ADJ); no longer Adj9V1.1
- new net: Adj9V1.1, IC2.4 (ADJ), R13.1, R9.2
- new net: C15.2, En9V1.1, IC2.3 (EN), R8.2
Other:
- note added: "Vout = Vref(1+(R6/R7)) Vref = 1.24 For VouT = 5v, r7 = 10K: R6 = ((Vout/Vref)-1)*R7 R6 = 30k"
- note added: "Vout = Vref(1+(R9/R13)) Vref = 1.24 For VouT = 9v, R13 = 10K: R9 = ((Vout/Vref)-1)*R13 R6 = 63.4k"
- note removed: "1.11k -> 12V"
- note removed: "1.54k -> 9V"
- note removed: "3.16k -> 5V"
- note removed: "R8 = -R9 + (R9/(1-(Vref/Vout)))"
- note removed: "Vref = 1.2V Vref = Vout - Vadj Vout(R7/R6+R7) = Vadj Therefore, Vref/(1-(R7/R7+R6)) = Vout"
- moved on the sheet: 5V_Out1, Adj5V1, Adj9V1, C4, C5, C7, En5V1, En9V1, R10, R6, R7, Vin1

Commit message: Rev B Sch Review
Parts:
- IC1, IC2: P/N (none) -> AP2205-W5-7
- R9: value 63.4k -> 30k
- renumbered 9V_Out1 to 5V_Out2, Adj9V1 to Adj5V2, En9V1 to En5V2
Other:
- note removed: "9V"
Changed lines of the file:
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@@
 		)
 	)
-	(text "9V"
+	(text "5V"
 		(exclude_from_sim no)
 		(at 161.798 85.852 0)
@@
 	)
 	(junction
+		(at 146.05 88.646)
+		(diameter 0)
+		(color 0 0 0 0)
+	)
+	(junction
 		(at 151.892 88.646)
 		(diameter 0)
@@
 	)
 	(junction
-		(at 146.05 88.646)
-		(diameter 0)
-		(color 0 0 0 0)
-	)
-	(junction
 		(at 150.622 70.358)
 		(diameter 0)
@@
 	(wire
 		(pts
-			(xy 146.05 88.646) (xy 151.892 88.646)
+			(xy 108.966 101.854) (xy 108.966 102.362)
 		)
 		(stroke
@@
 	(wire
 		(pts
-			(xy 108.966 101.854) (xy 108.966 102.362)
+			(xy 103.124 59.182) (xy 103.124 67.818)
 		)
 		(stroke
@@
 	(wire
 		(pts
-			(xy 103.124 59.182) (xy 103.124 67.818)
+			(xy 103.124 67.818) (xy 103.632 68.326)
 		)
 		(stroke
@@
 	(wire
 		(pts
-			(xy 103.124 67.818) (xy 103.632 68.326)
+			(xy 108.712 67.31) (xy 108.712 67.818)
 		)
 		(stroke
@@
 	(wire
 		(pts
-			(xy 108.712 67.31) (xy 108.712 67.818)
+			(xy 151.13 54.102) (xy 154.432 54.102)
 		)
 		(stroke
@@
 	(wire
 		(pts
-			(xy 151.13 54.102) (xy 154.432 54.102)
+			(xy 145.796 62.23) (xy 145.796 61.976)
 		)
 		(stroke
@@
 	(wire
 		(pts
-			(xy 145.796 62.23) (xy 145.796 61.976)
+			(xy 146.05 88.646) (xy 151.892 88.646)
 		)
 		(stroke
@@
 			)
 		)
+		(property "P/N" "~"
+			(at 151.13 54.102 0)
+			(effects
+				(font
+					(size 1.27 1.27)
+				)
+				(hide yes)
+			)
+		)
 		(pin "1"
 		)
@@
 		(on_board yes)
 		(dnp no)
-		(property "Reference" "9V_Out1"
+		(property "Reference" "5V_Out2"
 			(at 155.448 82.55 0)
 			(effects
@@
 			)
 		)
+		(property "P/N" "~"
+			(at 151.892 88.646 0)
+			(effects
+				(font
+					(size 1.27 1.27)
+				)
+				(hide yes)
+			)
+		)
 		(pin "1"
 		)
@@
 			(project "Controls-PedalsDaughter"
 				(path "/30d77876-714b-4f1b-9bad-b74eb43ddcf6/6613b086-4f9a-483f-8869-58f1a430ca82"
-					(reference "9V_Out1")
+					(reference "5V_Out2")
 					(unit 1)
 				)
@@
 			)
 		)
+		(property "P/N" "AP2205-W5-7"
+			(at 142.748 91.186 0)
+			(effects
+				(font
+					(size 1.27 1.27)
+				)
+				(hide yes)
+			)
+		)
 		(pin "1"
 		)
@@
 		(dnp no)
 		(property "Reference" "R9"
-			(at 147.574 90.932 0)
+			(at 141.986 89.916 0)
 			(effects
 				(font
@@
 			)
 		)
-		(property "Value" "63.4k"
-			(at 147.574 94.234 0)
+		(property "Value" "30k"
+			(at 146.05 94.488 90)
 			(effects
 				(font
@@
 			)
 		)
+		(property "P/N" "~"
+			(at 111.76 59.436 90)
+			(effects
+				(font
+					(size 1.27 1.27)
+				)
+				(hide yes)
+			)
+		)
 		(pin "1"
 		)
@@
 			)
 		)
+		(property "P/N" "AP2205-W5-7"
+			(at 142.494 56.642 0)
+			(effects
+				(font
+					(size 1.27 1.27)
+				)
+				(hide yes)
+			)
+		)
 		(pin "1"
 		)
@@
 		(on_board yes)
 		(dnp no)
-		(property "Reference" "En9V1"
+		(property "Reference" "En5V2"
 			(at 115.57 96.012 90)
 			(effects
@@
 			)
 		)
+		(property "P/N" "~"
+			(at 112.014 93.98 90)
+			(effects
+				(font
+					(size 1.27 1.27)
+				)
+				(hide yes)
+			)
+		)
 		(pin "1"
 		)
@@
 			(project "Controls-PedalsDaughter"
 				(path "/30d77876-714b-4f1b-9bad-b74eb43ddcf6/6613b086-4f9a-483f-8869-58f1a430ca82"
-					(reference "En9V1")
+					(reference "En5V2")
 					(unit 1)
 				)
@@
 		(on_board yes)
 		(dnp no)
-		(property "Reference" "Adj9V1"
+		(property "Reference" "Adj5V2"
 			(at 141.478 96.52 90)
 			(effects
@@
 			(project "Controls-PedalsDaughter"
 				(path "/30d77876-714b-4f1b-9bad-b74eb43ddcf6/6613b086-4f9a-483f-8869-58f1a430ca82"
-					(reference "Adj9V1")
+					(reference "Adj5V2")
 					(unit 1)
 				)
@@
 			(at 112.522 51.562 0)
 			(effects
+				(font
+					(size 1.27 1.27)
+				)
+				(hide yes)
+			)
+		)
+		(property "P/N" "~"
+			(at 112.522 51.562 0)
+			(effects

Commit message: Rev B Layout #2
Parts:
- IC1, IC2: footprint AP2205W57 -> AP2205-W5-7:AP2205W57
Changed lines of the file:
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@@
 			)
 		)
-		(property "Footprint" "AP2205W57"
+		(property "Footprint" "AP2205-W5-7:AP2205W57"
 			(at 118.618 -3.734 0)
 			(effects
@@
 			)
 		)
-		(property "Footprint" "AP2205W57"
+		(property "Footprint" "AP2205-W5-7:AP2205W57"
 			(at 118.364 -38.278 0)
 			(effects

Commit message: IM DONNEEEE
Parts:
- added F1, F2: 0603L025YR, 0603L025YR:FUSC1608X75N, symbol 0603L025YR:0603L025YR
Connections:
- net VoutAdj1: now also F2.2; no longer 5V_Out1.1, C7.1, IC1.5 (VOUT), R6.1
- net VoutAdj2: now also F1.2; no longer 5V_Out2.1, C16.1, IC2.5 (VOUT), R9.1
- new net: 5V_Out1.1, C7.1, F2.1, IC1.5 (VOUT), R6.1
- new net: 5V_Out2.1, C16.1, F1.1, IC2.5 (VOUT), R9.1
Other:
- note added: "------- For 9V ONLY ------- Vout = Vref(1+(R9/R13)) Vref = 1.24 For VouT = 9v, R13 = 10K: R9 = ((Vout/Vref)-1)*R13 R9 = 63.4k"
- note removed: "Vout = Vref(1+(R9/R13)) Vref = 1.24 For VouT = 9v, R13 = 10K: R9 = ((Vout/Vref)-1)*R13 R6 = 63.4k"

Commit message: Gerber + JLCpcb BOM :)
Parts:
- Adj5V1, Adj5V2: P/N (none) -> JLCJLCJLCJLC
