File: hardware/VCAT-PedalBoxPCB/Brake_Fl.kicad_sch (KiCad schematic)
At the start: 15 parts, among them U4 TLV70130DBVR, U5 AMC1300BDWV

Commit message: sch too ez
Parts:
- removed C1: 100nF, Capacitor_SMD:C_0805_2012Metric, symbol Device:C
- removed C10, C7: 1uF, Capacitor_SMD:C_0805_2012Metric, symbol Device:C
- removed C11, C6: 100uF, Capacitor_SMD:C_0805_2012Metric, symbol Device:C
- removed C8: 1nF, Capacitor_SMD:C_0805_2012Metric, symbol Device:C
- removed D3, D4: MBR, Diode_SMD:D_0805_2012Metric, symbol Device:D
- removed TP_3V3PWR1: +3V3PWR, TestPoint:TestPoint_Pad_1.5x1.5mm, symbol Connector:TestPoint
- removed U4: TLV70130DBVR, Package_TO_SOT_SMD:SOT-353_SC-70-5, symbol 2025-01-18_20-51-31:TLV70130DBVR
- removed U5: AMC1300BDWV, Package_SO:SOIC-8_7.5x5.85mm_P1.27mm, symbol Amplifier_Difference:AMC1300BDWV
- added U4: INA241A5xD, Package_SO:SOIC-8_3.9x4.9mm_P1.27mm, symbol Amplifier_Current:INA241A5xD
- added U5: REF5025AID, REF5025AID:SOIC127P599X175-8N, symbol REF5025AID:REF5025AID
- R1: value 20 -> 0.175
Connections:
- net GNDPWR is gone; now on net GNDA: R1.2
- net +VDDA: now also U4.6 (V+)
- net GNDA: now also U4.1 (-), U4.2 (GND), U4.4 (GND)
- net Brake_Fl renamed BrakeFL_GPIO
- net BrakeFL_GPIO: now also U4.5
- net INP renamed BrakeFL_ADC
- net BrakeFL_ADC: now also U4.8 (+)
- new net: U4.3 (REF2), U4.7 (REF1), U5.6 (VOUT)
- new net +3.3V: U5.2 (VIN)
- new net GND: U5.4 (GND)
- no-connect marks 2 -> 4
Other:
- note added: "0.7mV - 3.5mV"
- note added: "Break sensor gives current reading 4mA - 20mA"
- note added: "Current Sense Amplifier"
- note added: "Vout = G(Vin+ - Vin-) + (Vref1 +Vref2)/2 Vout = 200(ADC - 0) + (2.5) Vout = 200ADC + 2.5 Vout = [2.64v, 3.2v] ADC = [0.7mV, 3.5mV] Vref1 = Vref2 = 2.5v G = 200"
- note removed: "->"
- note removed: "20ma -> ~0.4V (*8.2) -> 3.28v"
- note removed: "3V3 Pwr for Isolated Amp"
- note removed: "Break sensor gives current reading 4ma - 20ma"
- note removed: "Isolated Amp"
- note removed: "x8.2 gain"
- moved on the sheet: Brake_Fl_Sn1, Brake_Fl_Sn_Raw1, C9, R1

Commit message: final review?? (plssss)
Connections:
- net +3.3V is gone; now on net +VDDA: U5.2 (VIN)
- net GND is gone; now on net GNDA: U5.4 (GND)
Changed lines of the file:
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@@
 	)
 	(symbol
-		(lib_id "power:GND")
-		(at 139.065 125.095 0)
-		(unit 1)
-		(exclude_from_sim no)
-		(in_bom yes)
-		(on_board yes)
-		(dnp no)
-		(fields_autoplaced yes)
-		(property "Reference" "#PWR032"
-			(at 139.065 131.445 0)
-			(effects
-				(font
-					(size 1.27 1.27)
-				)
-				(hide yes)
-			)
-		)
-		(property "Value" "GND"
-			(at 139.065 130.175 0)
-			(effects
-				(font
-					(size 1.27 1.27)
-				)
-				(hide yes)
+		(lib_name "+3V3_1")
+		(lib_id "power:+3V3")
+		(at 181.61 106.045 0)
+		(unit 1)
+		(exclude_from_sim no)
+		(in_bom yes)
+		(on_board yes)
+		(dnp no)
+		(property "Reference" "#PWR01"
+			(at 181.61 109.855 0)
+			(effects
+				(font
+					(size 1.27 1.27)
+				)
+				(hide yes)
+			)
+		)
+		(property "Value" "+VDDA"
+			(at 181.61 100.965 0)
+			(effects
+				(font
+					(size 1.27 1.27)
+				)
 			)
 		)
 		(property "Footprint" ""
-			(at 139.065 125.095 0)
+			(at 181.61 106.045 0)
 			(effects
 				(font
@@
 		)
 		(property "Datasheet" ""
-			(at 139.065 125.095 0)
-			(effects
-				(font
-					(size 1.27 1.27)
-				)
-				(hide yes)
-			)
-		)
-		(property "Description" "Power symbol creates a global label with name \"GND\" , ground"
-			(at 139.065 125.095 0)
+			(at 181.61 106.045 0)
+			(effects
+				(font
+					(size 1.27 1.27)
+				)
+				(hide yes)
+			)
+		)
+		(property "Description" "Power symbol creates a global label with name \"+3V3\""
+			(at 181.61 106.045 0)
 			(effects
 				(font
@@
 			(project "Controls-PedalsDaughter"
 				(path "/30d77876-714b-4f1b-9bad-b74eb43ddcf6/7d1ff2c9-efd0-48ce-add2-9372a4e6c13a"
-					(reference "#PWR032")
+					(reference "#PWR01")
 					(unit 1)
 				)
@@
 	)
 	(symbol
-		(lib_id "power:+3.3V")
-		(at 181.61 106.045 0)
+		(lib_id "power:GND")
+		(at 139.065 125.095 0)
 		(unit 1)
 		(exclude_from_sim no)
@@
 		(fields_autoplaced yes)
 		(property "Reference" "#PWR029"
-			(at 181.61 109.855 0)
-			(effects
-				(font
-					(size 1.27 1.27)
-				)
-				(hide yes)
-			)
-		)
-		(property "Value" "+3.3V"
-			(at 181.61 100.965 0)
+			(at 139.065 131.445 0)
+			(effects
+				(font
+					(size 1.27 1.27)
+				)
+				(hide yes)
+			)
+		)
+		(property "Value" "GNDA"
+			(at 139.065 130.175 0)
 			(effects
 				(font
@@
 		)
 		(property "Footprint" ""
-			(at 181.61 106.045 0)
+			(at 139.065 125.095 0)
 			(effects
 				(font
@@
 		)
 		(property "Datasheet" ""
-			(at 181.61 106.045 0)
-			(effects
-				(font
-					(size 1.27 1.27)
-				)
-				(hide yes)
-			)
-		)
-		(property "Description" "Power symbol creates a global label with name \"+3.3V\""
-			(at 181.61 106.045 0)
-			(effects
-				(font
+			(at 139.065 125.095 0)
+			(effects
+				(font
+					(size 1.27 1.27)
+				)
+				(hide yes)
+			)
+		)
+		(property "Description" "Power symbol creates a global label with name \"GND\" , ground"
+			(at 139.065 125.095 0)
+			(effects
+				(font

Commit message: PSOM pin layout pic
Other:
- note added: "Brake Fluid Sensor"
- note removed: "Break Fluid Sensor"
Changed lines of the file:
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@@
 	(generator_version "9.0")
 	(paper "A4")
-	(text "Break Fluid Sensor"
+	(rectangle
+		(start 57.785 64.77)
+		(end 248.92 133.985)
+		(stroke
+			(width 0)
+			(type default)
+		)
+		(fill
+			(type none)
+		)
+	)
+	(text "Brake Fluid Sensor"
 		(exclude_from_sim no)
-		(at 71.755 60.325 0)
+		(at 79.375 60.96 0)
 		(effects
 			(font
-				(size 2 2)
+				(size 3 3)
 				(thickness 0.4)
 				(bold yes)

Commit message: pcb design review #1
Parts:
- removed U5: REF5025AID, REF5025AID:SOIC127P599X175-8N, symbol REF5025AID:REF5025AID
- C9: footprint Capacitor_SMD:C_0805_2012Metric -> Capacitor_SMD:C_0603_1608Metric_Pad1.08x0.95mm_HandSolder
- R1: footprint Resistor_SMD:R_0805_2012Metric -> Resistor_SMD:R_0603_1608Metric_Pad0.98x0.95mm_HandSolder
Connections:
- net GNDA: now also U4.3 (REF2), U4.7 (REF1)
- no-connect marks 4 -> 0
Other:
- moved on the sheet: U4

Commit message: review #3
Parts:
- added C10: 1nF, Capacitor_SMD:C_0603_1608Metric_Pad1.08x0.95mm_HandSolder, symbol Device:C
Connections:
- net BrakeFL_ADC: now also C10.1
- net GNDA: now also C10.2
Changed lines of the file:
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@@
+	)
+	(junction
+		(at 99.06 88.9)
+		(diameter 0)
+		(color 0 0 0 0)
 	)
 	(junction
@@
 	(wire
 		(pts
-			(xy 87.63 88.9) (xy 92.71 88.9)
-		)
-		(stroke
-			(width 0)
-			(type default)
-		)
-	)
-	(wire
-		(pts
 			(xy 227.33 92.075) (xy 228.6 92.075)
 		)
@@
 	(wire
 		(pts
-			(xy 142.24 107.95) (xy 144.78 107.95)
+			(xy 141.605 107.95) (xy 144.78 107.95)
 		)
 		(stroke
@@
 	(wire
 		(pts
+			(xy 87.63 88.9) (xy 99.06 88.9)
+		)
+		(stroke
+			(width 0)
+			(type default)
+		)
+	)
+	(wire
+		(pts
 			(xy 87.63 86.36) (xy 87.63 88.9)
 		)
@@
 		(pts
 			(xy 81.28 88.9) (xy 87.63 88.9)
+		)
+		(stroke
+			(width 0)
+			(type default)
+		)
+	)
+	(wire
+		(pts
+			(xy 105.41 88.9) (xy 99.06 88.9)
 		)
 		(stroke
@@
 	)
 	(label "BrakeFL_ADC"
-		(at 92.71 88.9 0)
+		(at 105.41 88.9 0)
 		(effects
 			(font
@@
 	)
 	(symbol
+		(lib_id "Device:C")
+		(at 99.06 92.71 0)
+		(unit 1)
+		(exclude_from_sim no)
+		(in_bom yes)
+		(on_board yes)
+		(dnp no)
+		(property "Reference" "C10"
+			(at 102.87 91.44 0)
+			(effects
+				(font
+					(size 1.27 1.27)
+				)
+				(justify left)
+			)
+		)
+		(property "Value" "1nF"
+			(at 102.87 93.98 0)
+			(effects
+				(font
+					(size 1.27 1.27)
+				)
+				(justify left)
+			)
+		)
+		(property "Footprint" "Capacitor_SMD:C_0603_1608Metric_Pad1.08x0.95mm_HandSolder"
+			(at 100.0252 96.52 0)
+			(effects
+				(font
+					(size 1.27 1.27)
+				)
+				(hide yes)
+			)
+		)
+		(property "Datasheet" "~"
+			(at 99.06 92.71 0)
+			(effects
+				(font
+					(size 1.27 1.27)
+				)
+				(hide yes)
+			)
+		)
+		(property "Description" "Unpolarized capacitor"
+			(at 99.06 92.71 0)
+			(effects
+				(font
+					(size 1.27 1.27)
+				)
+				(hide yes)
+			)
+		)
+		(property "P/N" "pickle"
+			(at 99.06 92.71 0)
+			(effects
+				(font
+					(size 1.27 1.27)
+				)
+				(hide yes)
+			)
+		)
+		(pin "2"
+		)
+		(pin "1"
+		)
+		(instances
+			(project "Controls-PedalsDaughter"
+				(path "/30d77876-714b-4f1b-9bad-b74eb43ddcf6/7d1ff2c9-efd0-48ce-add2-9372a4e6c13a"
+					(reference "C10")
+					(unit 1)
+				)
+			)
+		)
+	)
+	(symbol
 		(lib_id "power:GND")
 		(at 153.67 120.65 0)
@@
 	(symbol
 		(lib_id "power:GNDA")
-		(at 142.24 107.95 0)
+		(at 141.605 107.95 0)
 		(unit 1)
 		(exclude_from_sim no)
@@
 		(dnp no)
 		(property "Reference" "#PWR010"
-			(at 142.24 114.3 0)
+			(at 141.605 114.3 0)
 			(effects
 				(font
@@
 		)
 		(property "Value" "GNDA"
-			(at 142.24 112.395 0)
+			(at 141.605 112.395 0)
 			(effects
 				(font
@@
 		)
 		(property "Footprint" ""
-			(at 142.24 107.95 0)
+			(at 141.605 107.95 0)
 			(effects
 				(font
@@
 		)
 		(property "Datasheet" ""
-			(at 142.24 107.95 0)
+			(at 141.605 107.95 0)
 			(effects
 				(font
@@
 		)
 		(property "Description" "Power symbol creates a global label with name \"GNDA\" , analog ground"
-			(at 142.24 107.95 0)
+			(at 141.605 107.95 0)
 			(effects
 				(font
@@
 					(unit 1)
 				)
+			)
+		)
+	)
+	(symbol
+		(lib_id "power:GND")
+		(at 99.06 96.52 0)
+		(unit 1)
+		(exclude_from_sim no)
+		(in_bom yes)
+		(on_board yes)
+		(dnp no)
+		(fields_autoplaced yes)
+		(property "Reference" "#PWR015"
+			(at 99.06 102.87 0)
+			(effects
+				(font
+					(size 1.27 1.27)
+				)
+				(hide yes)
+			)
+		)
+		(property "Value" "GNDA"
+			(at 99.06 101.6 0)
+			(effects
+				(font
+					(size 1.27 1.27)
+				)
+			)
+		)
+		(property "Footprint" ""
+			(at 99.06 96.52 0)
+			(effects
+				(font
+					(size 1.27 1.27)
+				)
+				(hide yes)
+			)
+		)
+		(property "Datasheet" ""
+			(at 99.06 96.52 0)
+			(effects
+				(font
+					(size 1.27 1.27)
+				)
+				(hide yes)
+			)
+		)
+		(property "Description" "Power symbol creates a global label with name \"GND\" , ground"
+			(at 99.06 96.52 0)
+			(effects
+				(font
+					(size 1.27 1.27)
+				)
+				(hide yes)
+			)
+		)
+		(pin "1"
+		)
+		(instances
+			(project "Controls-PedalsDaughter"
+				(path "/30d77876-714b-4f1b-9bad-b74eb43ddcf6/7d1ff2c9-efd0-48ce-add2-9372a4e6c13a"
+					(reference "#PWR015")
+					(unit 1)
+				)

Commit message: updated mx150 pin order :( works now
Parts:
- C10, C9: P/N pickle -> (none)
- R1: P/N ERJ-UP6D20R0V -> (none)

Commit message: updated BOM
Parts:
- added R16: 0.075, Resistor_SMD:R_0603_1608Metric_Pad0.98x0.95mm_HandSolder, symbol Device:R_US
- C10, C9: P/N (none) -> MLASU063SB7102KFNA01
- R1: value 0.175 -> 0.1; P/N (none) -> WSL0603R1000FEA
- U4: P/N (none) -> INA241A5IDR
Connections:
- net GNDA: now also R16.2; no longer R1.2
- new net: R1.2, R16.1
Changed lines of the file:
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@@
 	(text "Break sensor gives current\nreading 4mA - 20mA"
 		(exclude_from_sim no)
-		(at 87.63 109.22 0)
+		(at 86.995 114.3 0)
 		(effects
 			(font
@@
 	(text "Break psi is 25 - 600\nSensor range is 25 - 2500 psi"
 		(exclude_from_sim no)
-		(at 87.63 114.3 0)
+		(at 86.995 119.38 0)
 		(effects
 			(font
@@
 	(wire
 		(pts
+			(xy 87.63 105.41) (xy 87.63 104.14)
+		)
+		(stroke
+			(width 0)
+			(type default)
+		)
+	)
+	(wire
+		(pts
 			(xy 141.605 107.95) (xy 144.78 107.95)
 		)
@@
 		(pts
 			(xy 105.41 88.9) (xy 99.06 88.9)
-		)
-		(stroke
-			(width 0)
-			(type default)
-		)
-	)
-	(wire
-		(pts
-			(xy 87.63 97.155) (xy 87.63 96.52)
 		)
 		(stroke
@@
 			)
 			(justify left)
+		)
+	)
+	(symbol
+		(lib_id "Device:R_US")
+		(at 87.63 100.33 0)
+		(unit 1)
+		(exclude_from_sim no)
+		(in_bom yes)
+		(on_board yes)
+		(dnp no)
+		(fields_autoplaced yes)
+		(property "Reference" "R16"
+			(at 90.17 99.0599 0)
+			(effects
+				(font
+					(size 1.27 1.27)
+				)
+				(justify left)
+			)
+		)
+		(property "Value" "0.075"
+			(at 90.17 101.5999 0)
+			(effects
+				(font
+					(size 1.27 1.27)
+				)
+				(justify left)
+			)
+		)
+		(property "Footprint" "Resistor_SMD:R_0603_1608Metric_Pad0.98x0.95mm_HandSolder"
+			(at 88.646 100.584 90)
+			(effects
+				(font
+					(size 1.27 1.27)
+				)
+				(hide yes)
+			)
+		)
+		(property "Datasheet" "https://www.mouser.com/ProductDetail/Eaton-Electronics/MSMA2512R1750FEN?qs=By6Nw2ByBD3oOZ3TJVhB2g%3D%3D"
+			(at 87.63 100.33 0)
+			(effects
+				(font
+					(size 1.27 1.27)
+				)
+				(hide yes)
+			)
+		)
+		(property "Description" "Pedals BrakeFL R16 current sense"
+			(at 87.63 100.33 0)
+			(effects
+				(font
+					(size 1.27 1.27)
+				)
+				(hide yes)
+			)
+		)
+		(property "P/N" "RCWE060375L0FNEA"
+			(at 87.63 100.33 0)
+			(effects
+				(font
+					(size 1.27 1.27)
+				)
+				(hide yes)
+			)
+		)
+		(property "Height" ""
+			(at 87.63 100.33 0)
+			(effects
+				(font
+					(size 1.27 1.27)
+				)
+				(hide yes)
+			)
+		)
+		(property "Inventory" ""
+			(at 87.63 100.33 0)
+			(effects
+				(font
+					(size 1.27 1.27)
+				)
+				(hide yes)
+			)
+		)
+		(property "Mfg" ""
+			(at 87.63 100.33 0)
+			(effects
+				(font
+					(size 1.27 1.27)
+				)
+				(hide yes)
+			)
+		)
+		(property "Mouser Part Number" ""
+			(at 87.63 100.33 0)
+			(effects
+				(font
+					(size 1.27 1.27)
+				)
+				(hide yes)
+			)
+		)
+		(property "Mouser Price/Stock" ""
+			(at 87.63 100.33 0)
+			(effects
+				(font
+					(size 1.27 1.27)
+				)
+				(hide yes)
+			)
+		)
+		(property "PN" ""
+			(at 87.63 100.33 0)
+			(effects
+				(font
+					(size 1.27 1.27)
+				)
+				(hide yes)
+			)
+		)
+		(property "Sim.Device" ""
+			(at 87.63 100.33 0)
+			(effects
+				(font
+					(size 1.27 1.27)
+				)
+				(hide yes)
+			)
+		)
+		(property "p/n" ""
+			(at 87.63 100.33 0)
+			(effects
+				(font
+					(size 1.27 1.27)
+				)
+				(hide yes)
+			)
+		)
+		(pin "2"
+		)
+		(pin "1"
+		)
+		(instances
+			(project "Controls-PedalsDaughter"
+				(path "/30d77876-714b-4f1b-9bad-b74eb43ddcf6/7d1ff2c9-efd0-48ce-add2-9372a4e6c13a"
+					(reference "R16")
+					(unit 1)
+				)
+			)
 		)
 	)
@@
 			)
 		)
-		(property "Value" "0.175"
+		(property "Value" "0.1"
 			(at 90.17 93.9799 0)
 			(effects
@@
 			)
 		)
-		(property "Description" "Resistor, US symbol"
+		(property "Description" "Pedals BrakeFL R1 current sense"
 			(at 87.63 92.71 0)
 			(effects
@@
 			)
 		)
-		(property "P/N" ""
+		(property "P/N" "WSL0603R1000FEA"
 			(at 87.63 92.71 0)
 			(effects
@@
 			)
 		)
-		(property "Description" "Unpolarized capacitor"
+		(property "Description" "Pedals BrakeFL C10 cap"
 			(at 99.06 92.71 0)
 			(effects
@@
 			)
 		)
-		(property "P/N" ""
+		(property "P/N" "MLASU063SB7102KFNA01"
 			(at 99.06 92.71 0)
 			(effects
@@
 	(symbol
 		(lib_id "power:GND")
-		(at 87.63 97.155 0)
+		(at 87.63 105.41 0)
 		(unit 1)
 		(exclude_from_sim no)
@@
 		(fields_autoplaced yes)
 		(property "Reference" "#PWR012"
-			(at 87.63 103.505 0)
+			(at 87.63 111.76 0)
 			(effects
 				(font
@@
 		)
 		(property "Value" "GNDA"
-			(at 87.63 102.235 0)
+			(at 87.63 110.49 0)
 			(effects
 				(font
@@
 		)
 		(property "Footprint" ""
-			(at 87.63 97.155 0)
+			(at 87.63 105.41 0)
 			(effects
 				(font
@@
 		)
 		(property "Datasheet" ""
-			(at 87.63 97.155 0)
+			(at 87.63 105.41 0)
 			(effects
 				(font
@@
 		)
 		(property "Description" "Power symbol creates a global label with name \"GND\" , ground"
-			(at 87.63 97.155 0)
+			(at 87.63 105.41 0)
 			(effects
 				(font
@@
 			)
 		)
-		(property "Description" "High- and Low-Side, Bidirectional, Zero-Drift, Current-Sense Amplifier With Enhanced PWM Rejection, 200V/V, ±0.01% Gain Accuracy, ±10 μV Offset Voltage, SOIC-8"
+		(property "Description" "INA241A5IDR"
 			(at 152.4 105.41 0)
 			(effects
@@
 		)
 		(property "p/n" ""
+			(at 152.4 105.41 0)
+			(effects
+				(font
+					(size 1.27 1.27)
+				)
+				(hide yes)
+			)
+		)
+		(property "P/N" "INA241A5IDR"
 			(at 152.4 105.41 0)
 			(effects
@@
 			)
 		)
-		(property "Description" "Unpolarized capacitor"
+		(property "Description" "Pedals BrakeFL C10 cap"
 			(at 205.74 95.885 0)
 			(effects
@@
 			)
 		)
-		(property "P/N" ""
+		(property "P/N" "MLASU063SB7102KFNA01"
 			(at 205.74 95.885 0)
 			(effects

Commit message: Rev B - Initial Layout
Parts:
- added Brake_Fl_Sn2: Brake_Fl_Sn_TP, TestPoint:TestPoint_THTPad_1.5x1.5mm_Drill0.7mm, symbol Connector:TestPoint
- added Brake_Fl_Sn_Raw2: Brake_Fl_Sn_Raw_TP, TestPoint:TestPoint_THTPad_1.5x1.5mm_Drill0.7mm, symbol Connector:TestPoint
- added C13, C14: 1nF, Capacitor_SMD:C_0603_1608Metric_Pad1.08x0.95mm_HandSolder, symbol Device:C
- added R27: 1, Resistor_SMD:R_0603_1608Metric_Pad0.98x0.95mm_HandSolder, symbol Device:R_US
- added R28: 4.7, Resistor_SMD:R_0603_1608Metric_Pad0.98x0.95mm_HandSolder, symbol Device:R_US
- added R29, R30: 0.825, Resistor_SMD:R_0603_1608Metric_Pad0.98x0.95mm_HandSolder, symbol Device:R_US
- added U5: INA241A5xD, Package_SO:SOIC-8_3.9x4.9mm_P1.27mm, symbol Amplifier_Current:INA241A5xD
- R1: value 0.1 -> 1
- R16: value 0.075 -> 4.7
Connections:
- net +VDDA: now also U5.6 (V+)
- net GNDA: now also C13.2, C14.2, U5.1 (-), U5.2 (GND), U5.3 (REF2), U5.4 (GND), U5.7 (REF1); no longer R16.2
- net at R1.2: now also C10.1, R16.2, U4.8 (+); no longer R16.1
- net BrakeFL_ADC renamed BrakeFL
- net BrakeFL: now also R16.1; no longer C10.1, U4.8 (+)
- net BrakeFL_GPIO renamed BrakeFL_Amp
- new net: C13.1, R27.2, R28.2, U5.8 (+)
- new net BrakeFL_Red: Brake_Fl_Sn_Raw2.1, R27.1, R28.1
- new net BrakeFL_RedAmp: Brake_Fl_Sn2.1, C14.1, U5.5
Other:
- note added: "0.66V - 3.3V"
- note added: "3.3mV - 16.5mV"
- note added: "I V"
- note added: "V Ouput Range"
- note added: "V+ Input Range"
- note added: "Vout = G(Vin+ - Vin-) + (Vref1 +Vref2)/2 Vout = 200(ADC - 0) + (2.5) Vout = 200ADC Vout = [0.66v, 3.3v] ADC = [3.3mV, 16.5mV] Vref1 = Vref2 = GNDA = 0.0V G = 200"
- note removed: "0.7mV - 3.5mV"
- note removed: "Brake"
- note removed: "Vout = G(Vin+ - Vin-) + (Vref1 +Vref2)/2 Vout = 200(ADC - 0) + (2.5) Vout = 200ADC + 2.5 Vout = [2.64v, 3.2v] ADC = [0.7mV, 3.5mV] Vref1 = Vref2 = 2.5v G = 200"
- moved on the sheet: Brake_Fl_Sn1, Brake_Fl_Sn_Raw1, C10, C9, R1, R16, U4
