File: hardware/VCAT-PedalBoxPCB/Brake_Fl.kicad_sch (KiCad schematic)
At the start: 16 parts, among them U4 INA241A5xD, U5 INA241A5xD

Commit message: Layout DONEEEE
Parts:
- removed Brake_Fl_Sn_Raw2: Brake_Fl_Sn_Raw_TP, TestPoint:TestPoint_THTPad_1.5x1.5mm_Drill0.7mm, symbol Connector:TestPoint
Changed lines of the file:
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@@
 	)
 	(junction
-		(at 98.298 102.87)
-		(diameter 0)
-		(color 0 0 0 0)
-	)
-	(junction
 		(at 188.976 105.41)
 		(diameter 0)
@@
 	(wire
 		(pts
-			(xy 100.838 102.87) (xy 98.298 102.87)
+			(xy 91.948 102.87) (xy 100.838 102.87)
 		)
 		(stroke
@@
 	(wire
 		(pts
-			(xy 91.948 102.87) (xy 98.298 102.87)
-		)
-		(stroke
-			(width 0)
-			(type default)
-		)
-	)
-	(wire
-		(pts
 			(xy 98.044 60.452) (xy 98.044 62.484)
 		)
@@
 	(wire
 		(pts
-			(xy 98.298 100.838) (xy 98.298 102.87)
-		)
-		(stroke
-			(width 0)
-			(type default)
-		)
-	)
-	(wire
-		(pts
 			(xy 101.092 62.484) (xy 101.092 69.342)
 		)
@@
 					(unit 1)
 				)
-			)
-		)
-	)
-	(symbol
-		(lib_id "Connector:TestPoint")
-		(at 98.298 100.838 0)
-		(unit 1)
-		(exclude_from_sim no)
-		(in_bom yes)
-		(on_board yes)
-		(dnp no)
-		(property "Reference" "Brake_Fl_Sn_Raw2"
-			(at 100.076 96.774 0)
-			(effects
-				(font
-					(size 1.27 1.27)
-				)
-				(justify left)
-			)
-		)
-		(property "Value" "Brake_Fl_Sn_Raw_TP"
-			(at 76.708 97.028 0)
-			(effects
-				(font
-					(size 1.27 1.27)
-				)
-				(justify left)
-			)
-		)
-		(property "Footprint" "TestPoint:TestPoint_THTPad_1.5x1.5mm_Drill0.7mm"
-			(at 103.378 100.838 0)
-			(effects
-				(font
-					(size 1.27 1.27)
-				)
-				(hide yes)
-			)
-		)
-		(property "Datasheet" "~"
-			(at 103.378 100.838 0)
-			(effects
-				(font
-					(size 1.27 1.27)
-				)
-				(hide yes)
-			)
-		)
-		(property "Description" ""
-			(at 98.298 100.838 0)
-			(effects
-				(font
-					(size 1.27 1.27)
-				)
-				(hide yes)
-			)
-		)
-		(property "Height" ""
-			(at 98.298 100.838 0)
-			(effects
-				(font
-					(size 1.27 1.27)
-				)
-				(hide yes)
-			)
-		)
-		(property "Inventory" ""
-			(at 98.298 100.838 0)
-			(effects
-				(font
-					(size 1.27 1.27)
-				)
-				(hide yes)
-			)
-		)
-		(property "Mfg" ""
-			(at 98.298 100.838 0)
-			(effects
-				(font
-					(size 1.27 1.27)
-				)
-				(hide yes)
-			)
-		)
-		(property "Mouser Part Number" ""
-			(at 98.298 100.838 0)
-			(effects
-				(font
-					(size 1.27 1.27)
-				)
-				(hide yes)
-			)
-		)
-		(property "Mouser Price/Stock" ""
-			(at 98.298 100.838 0)
-			(effects
-				(font
-					(size 1.27 1.27)
-				)
-				(hide yes)
-			)
-		)
-		(property "P/N" "~"
-			(at 98.298 100.838 0)
-			(effects
-				(font
-					(size 1.27 1.27)
-				)
-				(hide yes)
-			)
-		)
-		(property "PN" ""
-			(at 98.298 100.838 0)
-			(effects
-				(font
-					(size 1.27 1.27)
-				)
-				(hide yes)
-			)
-		)
-		(property "Sim.Device" ""
-			(at 98.298 100.838 0)
-			(effects
-				(font
-					(size 1.27 1.27)
-				)
-				(hide yes)
-			)
-		)
-		(property "p/n" ""
-			(at 98.298 100.838 0)
-			(effects
-				(font
-					(size 1.27 1.27)
-				)
-				(hide yes)
-			)
-		)
-		(pin "1"
-		)
-		(instances
-			(project "Controls-PedalsDaughter"
-				(path "/30d77876-714b-4f1b-9bad-b74eb43ddcf6/7d1ff2c9-efd0-48ce-add2-9372a4e6c13a"
-					(reference "Brake_Fl_Sn_Raw2")
-					(unit 1)
-				)

Commit message: Rev B Sch Review
Parts:
- removed Brake_Fl_Sn1, Brake_Fl_Sn2: Brake_Fl_Sn_TP, TestPoint:TestPoint_THTPad_1.5x1.5mm_Drill0.7mm, symbol Connector:TestPoint
- removed Brake_Fl_Sn_Raw1: Brake_Fl_Sn_Raw_TP, TestPoint:TestPoint_THTPad_1.5x1.5mm_Drill0.7mm, symbol Connector:TestPoint
- removed C10, C13, C14, C9: 1nF, Capacitor_SMD:C_0603_1608Metric_Pad1.08x0.95mm_HandSolder, symbol Device:C
- removed R1, R27: 1, Resistor_SMD:R_0603_1608Metric_Pad0.98x0.95mm_HandSolder, symbol Device:R_US
- removed R16, R28: 4.7, Resistor_SMD:R_0603_1608Metric_Pad0.98x0.95mm_HandSolder, symbol Device:R_US
- removed R29, R30: 0.825, Resistor_SMD:R_0603_1608Metric_Pad0.98x0.95mm_HandSolder, symbol Device:R_US
- removed U4, U5: INA241A5xD, Package_SO:SOIC-8_3.9x4.9mm_P1.27mm, symbol Amplifier_Current:INA241A5xD
- added BrakeFLredRaw1, BrakeFlRaw1: Raw_TP, TestPoint:TestPoint_THTPad_1.5x1.5mm_Drill0.7mm, symbol Connector:TestPoint
- added R27, R28, R37, R38, R41, R42, R43, R44: 0, Resistor_SMD:R_0603_1608Metric_Pad0.98x0.95mm_HandSolder, symbol Device:R
- added R31, R32: 10k, Resistor_SMD:R_0603_1608Metric_Pad0.98x0.95mm_HandSolder, symbol Device:R_US
- added R33, R34: 5.6k, Resistor_SMD:R_0603_1608Metric_Pad0.98x0.95mm_HandSolder, symbol Device:R_US
Connections:
- net BrakeFL: now also R37.2, R41.2
- net BrakeFL_Amp: now also R38.1, R44.1
- net BrakeFL_Red: now also R27.2, R42.2
- net BrakeFL_RedAmp: now also R28.1, R43.1
- net GNDA: now also R31.1, R32.1
- new net: R33.1, R41.1
- new net: BrakeFlRaw1.1, R31.2, R33.2
- new net: R34.1, R42.1
- new net: BrakeFLredRaw1.1, R32.2, R34.2
- new net Brake Fluid Current Sense Amp/FL Sensor: R37.1
- new net Brake Fluid Current Sense Amp/Voltage output: R38.2
- new net Brake Fluid Current Sense Amp1/FL Sensor: R27.1
- new net Brake Fluid Current Sense Amp1/Voltage output: R28.2
- new net Dual Op Amp Buffer/MainSignalOut: R44.2
- new net Dual Op Amp Buffer/RedSignalOut: R43.2
Other:
- added sheet Brake Fluid Current Sense Amp (FL_CS.kicad_sch)
- added sheet Brake Fluid Current Sense Amp1 (FL_CS.kicad_sch)
- added sheet Dual Op Amp Buffer (untitled.kicad_sch)
- note added: "0.32v - 3.205v"
- note added: "0.5v - 5v"
- note added: "Main Signal"
- note added: "New Brake Fluid Sensor (Voltage Output)"
- note added: "OLD Brake Fluid Sensor (current output) - Backup"
- note added: "Redundant Signal"
- note added: "V Input Range"
- note added: "V Output Range"
- note added: "Vin = [0.5, 5] Vdivider = Vin * 10/(10+5.6) Vdivider_low = 0.5 * 10/15.6 = 0.32v Vdivider_high = 5 * 10/15.6 = 3.205v"
- note removed: "0.66V - 3.3V"
- note removed: "3.3mV - 16.5mV"
- note removed: "Brake Fluid Sensor"
- note removed: "Break psi is 25 - 600 Sensor range is 25 - 2500 psi"
- note removed: "Break sensor gives current reading 4mA - 20mA"
- note removed: "Current Sense Amplifier"
- note removed: "I V"
- note removed: "V Ouput Range"
- note removed: "V+ Input Range"
- note removed: "Vout = G(Vin+ - Vin-) + (Vref1 +Vref2)/2 Vout = 200(ADC - 0) + (2.5) Vout = 200ADC Vout = [0.66v, 3.3v] ADC = [3.3mV, 16.5mV] Vref1 = Vref2 = GNDA = 0.0V G = 200"

Commit message: Rev B Layout #2
Parts:
- removed BrakeFLredRaw1, BrakeFlRaw1: Raw_TP, TestPoint:TestPoint_THTPad_1.5x1.5mm_Drill0.7mm, symbol Connector:TestPoint
- removed R31, R32: 10k, Resistor_SMD:R_0603_1608Metric_Pad0.98x0.95mm_HandSolder, symbol Device:R_US
- removed R33, R34: 5.6k, Resistor_SMD:R_0603_1608Metric_Pad0.98x0.95mm_HandSolder, symbol Device:R_US
- R27, R28, R37, R38: now not fitted
Connections:
- net Dual Op Amp Buffer/Signal1_In: now reaches R41.1
- net Dual Op Amp Buffer/Signal2_In: now reaches R42.1
- net Dual Op Amp Buffer/MainSignalOut renamed Dual Op Amp Buffer/Signal1_Out
- net Dual Op Amp Buffer/RedSignalOut renamed Dual Op Amp Buffer/Signal2_Out
Other:
- sheet Dual Op Amp Buffer ports: added Signal1_In, Signal1_Out, Signal2_In, Signal2_Out; removed MainSignalIn, MainSignalOut, RedSignalIn, RedSignalOut
- moved on the sheet: R41, R42, R43, R44

Commit message: IM DONNEEEE
Other:
- sheet Dual Op Amp Buffer: file untitled.kicad_sch -> OpAmpBuffer.kicad_sch
Changed lines of the file:
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@@
 			)
 		)
-		(property "Sheetfile" "untitled.kicad_sch"
+		(property "Sheetfile" "OpAmpBuffer.kicad_sch"
 			(at 124.968 65.8626 0)
 			(effects
