File: hardware/VCAT-PedalBoxPCB/untitled.kicad_sch (KiCad schematic)
At the start: 8 parts, among them U1 TLV9002QDRQ1

Commit message: Rev B Layout #2
Parts:
- removed BrakeFLRed_Buff2, BrakeFL_Buff1: Accel, TestPoint:TestPoint_THTPad_1.5x1.5mm_Drill0.7mm, symbol Connector:TestPoint
- added R31, R32: 10k, Resistor_SMD:R_0603_1608Metric_Pad0.98x0.95mm_HandSolder, symbol Device:R_US
- added R33, R34: 5.6k, Resistor_SMD:R_0603_1608Metric_Pad0.98x0.95mm_HandSolder, symbol Device:R_US
- added TP1: Raw_TP, TestPoint:TestPoint_Pad_1.0x1.0mm, symbol Connector:TestPoint
- added TP12, TP6, TP9: Raw_TP, TestPoint:TestPoint_THTPad_1.5x1.5mm_Drill0.7mm, symbol Connector:TestPoint
Connections:
- net GNDA: now also R31.1, R32.1
- net MainSignalIn renamed In1+
- net In1+: now also R31.2, R33.2, TP6.1
- net MainSignalOut renamed Signal1_Out
- net Signal1_Out: now also TP9.1
- net RedSignalIn renamed In2+
- net In2+: now also R32.2, R34.2, TP1.1
- net RedSignalOut renamed Signal2_Out
- net Signal2_Out: now also TP12.1
- new net Signal1_In: R33.1
- new net Signal2_In: R34.1
Other:
- moved on the sheet: C17, C18, C19, R35, R36, U1A, U1B, U1C
