File: hardware/VCAT-PedalBoxPCB/Pedals.kicad_sch (KiCad schematic)
At the start: 18 parts, among them U3 TLV9301xDCK, U6 TLV9301xDCK

Commit message: sch too ez
Parts:
- removed Accel_Raw1: Accel_Raw_TP, TestPoint:TestPoint_THTPad_1.5x1.5mm_Drill0.7mm, symbol Connector:TestPoint
- removed Accel_TP1: Accel, TestPoint:TestPoint_THTPad_1.5x1.5mm_Drill0.7mm, symbol Connector:TestPoint
- removed Brake_Raw1: Brake_Raw_TP, TestPoint:TestPoint_THTPad_1.5x1.5mm_Drill0.7mm, symbol Connector:TestPoint
- removed Brake_TP1: Brake, TestPoint:TestPoint_THTPad_1.5x1.5mm_Drill0.7mm, symbol Connector:TestPoint
- removed C12, C14: 1nf, Capacitor_SMD:C_0805_2012Metric, symbol Device:C
- removed C13, C3: 0.1uf, Capacitor_SMD:C_0805_2012Metric, symbol Device:C
- removed D1, D2, D5, D8: MBR, Diode_SMD:D_0805_2012Metric, symbol Device:D
- removed R2, R5: 8.2k, Resistor_SMD:R_0805_2012Metric, symbol Device:R_US
- removed R4, R6: 22k, Resistor_SMD:R_0805_2012Metric, symbol Device:R_US
- removed U3, U6: TLV9301xDCK, Package_TO_SOT_SMD:SOT-353_SC-70-5, symbol Amplifier_Operational:TLV9301xDCK
Connections:
- no-connect marks 2 -> 0
Other:
- added sheet Unity Gain Buffer (UnityGainBuffer.kicad_sch)
- added sheet Unity Gain Buffer1 (UnityGainBuffer.kicad_sch)
- note removed: "0.5V - 4.5V Analog signal"
- note removed: "4.5V -> 3.278V"
- note removed: "Based on: https://www.akao.co.uk/manuals/Link%20G4+%20Manual/nissan_vq35.htm"
- note removed: "Redundant Signal"
- note removed: "Schotky :)"

Commit message: bruh
Other:
- removed sheet Unity Gain Buffer1
- sheet Unity Gain Buffer ports: added Accel_ADC, Accel_Raw, BrakePot_Raw, Brake_ADC; removed ADC_GPIO, ADC_Raw
- note added: "Accel & Brake Pedal"
- note removed: "Accel Pedal"
- note removed: "Brake Pedal"
Changed lines of the file:
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@@
 		)
 	)
-	(text "Brake Pedal"
+	(text "Accel & Brake Pedal"
 		(exclude_from_sim no)
-		(at 171.45 76.2 0)
-		(effects
-			(font
-				(size 3 3)
-				(thickness 0.4)
-				(bold yes)
-			)
-		)
-	)
-	(text "Accel Pedal"
-		(exclude_from_sim no)
-		(at 114.935 76.835 0)
+		(at 140.716 76.2 0)
 		(effects
 			(font
@@
 	(wire
 		(pts
-			(xy 159.385 88.9) (xy 161.29 88.9)
+			(xy 152.146 89.154) (xy 155.448 89.154)
 		)
 		(stroke
@@
 	(wire
 		(pts
-			(xy 102.235 88.9) (xy 104.14 88.9)
+			(xy 152.146 96.774) (xy 155.194 96.774)
 		)
 		(stroke
@@
 	(wire
 		(pts
-			(xy 126.365 88.9) (xy 129.54 88.9)
+			(xy 128.27 86.614) (xy 130.048 86.614)
 		)
 		(stroke
@@
 	(wire
 		(pts
-			(xy 183.515 88.9) (xy 188.595 88.9)
+			(xy 128.016 93.218) (xy 130.048 93.218)
 		)
 		(stroke
@@
 	(hierarchical_label "BrakePot"
 		(shape input)
-		(at 159.385 88.9 180)
+		(at 128.016 93.218 180)
 		(effects
 			(font
@@
 	(hierarchical_label "Accel"
 		(shape input)
-		(at 102.235 88.9 180)
+		(at 128.27 86.614 180)
 		(effects
 			(font
@@
 	(hierarchical_label "Accel_GPIO"
 		(shape output)
-		(at 129.54 88.9 0)
+		(at 155.448 89.154 0)
 		(effects
 			(font
@@
 	(hierarchical_label "BrakePot_GPIO"
 		(shape output)
-		(at 188.595 88.9 0)
+		(at 155.194 96.774 0)
 		(effects
 			(font
@@
 	)
 	(sheet
-		(at 161.29 85.09)
-		(size 22.225 6.985)
-		(exclude_from_sim no)
-		(in_bom yes)
-		(on_board yes)
-		(dnp no)
-		(stroke
-			(width 0.1524)
-			(type solid)
-		)
-		(fill
-			(color 0 0 0 0.0000)
-		)
-		(property "Sheetname" "Unity Gain Buffer1"
-			(at 161.29 84.3784 0)
-			(effects
-				(font
-					(size 1.27 1.27)
-				)
-				(justify left bottom)
-			)
-		)
-		(property "Sheetfile" "UnityGainBuffer.kicad_sch"
-			(at 158.115 94.615 0)
-			(effects
-				(font
-					(size 1.27 1.27)
-				)
-				(justify left top)
-			)
-		)
-		(pin "ADC_GPIO" output
-			(at 183.515 88.9 0)
-			(effects
-				(font
-					(size 1.27 1.27)
-				)
-				(justify right)
-			)
-		)
-		(pin "ADC_Raw" input
-			(at 161.29 88.9 180)
-			(effects
-				(font
-					(size 1.27 1.27)
-				)
-				(justify left)
-			)
-		)
-		(instances
-			(project "Controls-PedalsDaughter"
-				(path "/30d77876-714b-4f1b-9bad-b74eb43ddcf6/ba8b1230-57a3-4f16-bcdd-31b6729b5a2c"
-					(page "6")
-				)
-			)
-		)
-	)
-	(sheet
-		(at 104.14 85.09)
-		(size 22.225 6.985)
+		(at 130.048 84.328)
+		(size 22.098 14.732)
 		(exclude_from_sim no)
 		(in_bom yes)
@@
 		)
 		(property "Sheetname" "Unity Gain Buffer"
-			(at 104.14 84.3784 0)
+			(at 130.048 83.6164 0)
 			(effects
 				(font
@@
 		)
 		(property "Sheetfile" "UnityGainBuffer.kicad_sch"
-			(at 100.965 94.615 0)
+			(at 126.873 100.838 0)
 			(effects
 				(font
@@
 			)
 		)
-		(pin "ADC_GPIO" output
-			(at 126.365 88.9 0)
+		(pin "Accel_ADC" output
+			(at 152.146 89.154 0)
 			(effects
 				(font
@@
 			)
 		)
-		(pin "ADC_Raw" input
-			(at 104.14 88.9 180)
+		(pin "Accel_Raw" input
+			(at 130.048 86.614 180)
 			(effects
 				(font
@@
 			)
 		)
+		(pin "BrakePot_Raw" input
+			(at 130.048 93.218 180)
+			(effects
+				(font
+					(size 1.27 1.27)
+				)
+				(justify left)
+			)
+		)
+		(pin "Brake_ADC" output
+			(at 152.146 96.774 0)
+			(effects
+				(font
+					(size 1.27 1.27)
+				)
+				(justify right)
+			)
+		)

Commit message: Rev B Sch updates
Parts:
- added AccelRaw1, BrakeRaw1: Raw_TP, TestPoint:TestPoint_THTPad_1.5x1.5mm_Drill0.7mm, symbol Connector:TestPoint
- added Accel_GPIO1, BrakePot_GPIO1: Accel, TestPoint:TestPoint_THTPad_1.5x1.5mm_Drill0.7mm, symbol Connector:TestPoint
- added C11: 0.1uF, Capacitor_SMD:C_0603_1608Metric_Pad1.08x0.95mm_HandSolder, symbol Device:C
- added C2, C6: 0.01uf, Capacitor_SMD:C_0603_1608Metric_Pad1.08x0.95mm_HandSolder, symbol Device:C
- added R12, R3: 10k, Resistor_SMD:R_0603_1608Metric_Pad0.98x0.95mm_HandSolder, symbol Device:R_US
- added R21, R5: 22k, Resistor_SMD:R_0603_1608Metric_Pad0.98x0.95mm_HandSolder, symbol Device:R_US
- added R22, R23: 100, Resistor_SMD:R_0603_1608Metric_Pad0.98x0.95mm_HandSolder, symbol Device:R_US
- added U1: TLV9002QDRQ1, TLV9002QDRQ1:SOIC8_D_TEX, symbol Device:Opamp_Dual
Connections:
- net Accel: now also R3.2
- net Accel_GPIO: now also Accel_GPIO1.1, C2.2, R22.1
- net BrakePot: now also R12.2
- net BrakePot_GPIO: now also BrakePot_GPIO1.1, C6.2, R23.1
- new net +VDDA: C11.1, U1.8 (V+)
- new net GNDA: C11.2, C2.1, C6.1, R21.2, R5.2, U1.4 (V-)
- new net In1+: AccelRaw1.1, R3.1, R5.1, U1.3 (+)
- new net In1-: R22.2, U1.1, U1.2 (-)
- new net In2+: BrakeRaw1.1, R12.1, R21.1, U1.5 (+)
- new net In2-: R23.2, U1.6 (-), U1.7
Other:
- removed sheet Unity Gain Buffer
- note added: "Accel & Brake ADC Signal Buffer"
- note added: "Pedals Potentiometer Datasheet https://www.ttelectronics.com/TTElectronics/media/ProductFiles/Datasheet/6120.pdf"
- note removed: "Accel & Brake Pedal"

Commit message: Rev B - Initial Layout
Parts:
- removed U1: TLV9002QDRQ1, TLV9002QDRQ1:SOIC8_D_TEX, symbol Device:Opamp_Dual
- added AccelRaw2, BrakeRaw2: Raw_TP, TestPoint:TestPoint_THTPad_1.5x1.5mm_Drill0.7mm, symbol Connector:TestPoint
- added Accel_GPIO2, BrakePot_GPIO2: Accel, TestPoint:TestPoint_THTPad_1.5x1.5mm_Drill0.7mm, symbol Connector:TestPoint
- added C1: 0.1uF, Capacitor_SMD:C_0603_1608Metric_Pad1.08x0.95mm_HandSolder, symbol Device:C
- added C12, C3: 0.01uf, Capacitor_SMD:C_0603_1608Metric_Pad1.08x0.95mm_HandSolder, symbol Device:C
- added R11, R24: 22k, Resistor_SMD:R_0603_1608Metric_Pad0.98x0.95mm_HandSolder, symbol Device:R_US
- added R2, R4: 10k, Resistor_SMD:R_0603_1608Metric_Pad0.98x0.95mm_HandSolder, symbol Device:R_US
- added R25, R26: 100, Resistor_SMD:R_0603_1608Metric_Pad0.98x0.95mm_HandSolder, symbol Device:R_US
- added U3: TLV9002QDRQ1, TLV9002QDRQ1:SOIC8_D_TEX, symbol Device:Opamp_Dual
- added U7: TLV9002QDRQ1, Package_SO:SOIC-8_3.9x4.9mm_P1.27mm, symbol utsvt_misc:TLV9002QDRQ1
Connections:
- net +VDDA: now also C1.1, U3.8 (V+), U7.8 (V+)
- net GNDA: now also C1.2, C12.1, C3.1, R11.2, R24.2, U3.4 (V-), U7.4 (V-)
- net In1+: now also U7.3 (+)
- net In1-: now also U7.1, U7.2 (-)
- net In2+: now also U7.5 (+)
- net In2-: now also U7.6 (-), U7.7
- net Accel_GPIO renamed Accel_Buff
- net BrakePot_GPIO renamed BrakePot_Buff
- new net AccelRed: R2.2
- new net AccelRed_Buff: Accel_GPIO2.1, C3.2, R25.1
- new net BrakePotRed: R4.2
- new net BrakePotRed_Buff: BrakePot_GPIO2.1, C12.2, R26.1
- new net In3+: AccelRaw2.1, R11.1, R2.1, U3.3 (+)
- new net In3-: R25.2, U3.1, U3.2 (-)
- new net In4+: BrakeRaw2.1, R24.1, R4.1, U3.5 (+)
- new net In4-: R26.2, U3.6 (-), U3.7
Other:
- moved on the sheet: AccelRaw1, Accel_GPIO1, BrakePot_GPIO1, BrakeRaw1, C11, C2, C6, R12, R21, R22, R23, R3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

Commit message: Rev B Sch Review
Parts:
- removed Accel_GPIO1, Accel_GPIO2, BrakePot_GPIO1, BrakePot_GPIO2: Accel, TestPoint:TestPoint_THTPad_1.5x1.5mm_Drill0.7mm, symbol Connector:TestPoint
- removed C1, C11: 0.1uF, Capacitor_SMD:C_0603_1608Metric_Pad1.08x0.95mm_HandSolder, symbol Device:C
- removed C12, C2, C3, C6: 0.01uf, Capacitor_SMD:C_0603_1608Metric_Pad1.08x0.95mm_HandSolder, symbol Device:C
- removed R22, R23, R25, R26: 100, Resistor_SMD:R_0603_1608Metric_Pad0.98x0.95mm_HandSolder, symbol Device:R_US
- removed U3: TLV9002QDRQ1, TLV9002QDRQ1:SOIC8_D_TEX, symbol Device:Opamp_Dual
- removed U7: TLV9002QDRQ1, Package_SO:SOIC-8_3.9x4.9mm_P1.27mm, symbol utsvt_misc:TLV9002QDRQ1
Connections:
- net In1+ renamed Dual Op Amp Buffer/MainSignalIn
- net In2+ renamed Dual Op Amp Buffer/RedSignalIn
- net In3+ renamed Dual Op Amp Buffer1/MainSignalIn
- net In4+ renamed Dual Op Amp Buffer1/RedSignalIn
Other:
- added sheet Dual Op Amp Buffer (untitled.kicad_sch)
- added sheet Dual Op Amp Buffer1 (untitled.kicad_sch)
- moved on the sheet: R11, R12, R2, R21, R24, R3, R4, R5

Commit message: Rev B Layout #2
Parts:
- removed AccelRaw1, AccelRaw2, BrakeRaw1, BrakeRaw2: Raw_TP, TestPoint:TestPoint_THTPad_1.5x1.5mm_Drill0.7mm, symbol Connector:TestPoint
- removed R11, R21, R24, R5: 22k, Resistor_SMD:R_0603_1608Metric_Pad0.98x0.95mm_HandSolder, symbol Device:R_US
- removed R12, R2, R3, R4: 10k, Resistor_SMD:R_0603_1608Metric_Pad0.98x0.95mm_HandSolder, symbol Device:R_US
Other:
- sheet Dual Op Amp Buffer ports: added Signal1_In, Signal1_Out, Signal2_In, Signal2_Out; removed MainSignalIn, MainSignalOut, RedSignalIn, RedSignalOut
- sheet Dual Op Amp Buffer1 ports: added Signal1_In, Signal1_Out, Signal2_In, Signal2_Out; removed MainSignalIn, MainSignalOut, RedSignalIn, RedSignalOut
- note added: "Vin = [0.25, 5] Vdivider = Vin * 10/(10+5.6) Vdivider_low = 0.25 * 10/15.6 = 0.16v Vdivider_high = 5 * 10/15.6 = 3.205v"

Commit message: IM DONNEEEE
Other:
- sheet Dual Op Amp Buffer renamed Dual Op Amp Buffer Pots (main)
- sheet Dual Op Amp Buffer1 renamed Dual Op Amp Buffer Pots (Redundant)
- sheet Dual Op Amp Buffer Pots (Redundant): file untitled.kicad_sch -> OpAmpBuffer.kicad_sch
- sheet Dual Op Amp Buffer Pots (main): file untitled.kicad_sch -> OpAmpBuffer.kicad_sch
Changed lines of the file:
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@@
 			(color 0 0 0 0.0000)
 		)
-		(property "Sheetname" "Dual Op Amp Buffer1"
+		(property "Sheetname" "Dual Op Amp Buffer Pots (Redundant)"
 			(at 127.254 79.2984 0)
 			(effects
@@
 			)
 		)
-		(property "Sheetfile" "untitled.kicad_sch"
+		(property "Sheetfile" "OpAmpBuffer.kicad_sch"
 			(at 127.254 92.5326 0)
 			(effects
@@
 			(color 0 0 0 0.0000)
 		)
-		(property "Sheetname" "Dual Op Amp Buffer"
+		(property "Sheetname" "Dual Op Amp Buffer Pots (main)"
 			(at 127 51.8664 0)
 			(effects
@@
 			)
 		)
-		(property "Sheetfile" "untitled.kicad_sch"
+		(property "Sheetfile" "OpAmpBuffer.kicad_sch"
 			(at 127 65.1006 0)
 			(effects
