File: hardware/VCAT-PedalBoxPCB/FL_CS.kicad_sch (KiCad schematic)
At the start: 7 parts, among them U4 INA241A5xD

Commit message: Rev B Layout #2
Parts:
- removed Brake_Fl_Sn_Raw1: Brake_Fl_Sn_Raw_TP, TestPoint:TestPoint_THTPad_1.5x1.5mm_Drill0.7mm, symbol Connector:TestPoint
- added TP4: Raw_TP, TestPoint:TestPoint_THTPad_1.5x1.5mm_Drill0.7mm, symbol Connector:TestPoint
Connections:
- net FL Sensor: now also TP4.1
- no-connect marks 0 -> 2
Changed lines of the file:
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@@
-	)
-	(junction
-		(at 91.186 86.868)
-		(diameter 0)
-		(color 0 0 0 0)
 	)
 	(junction
@@
 		(color 0 0 0 0)
 	)
+	(junction
+		(at 91.186 86.106)
+		(diameter 0)
+		(color 0 0 0 0)
+	)
+	(no_connect
+		(at 84.074 108.966)
+	)
+	(no_connect
+		(at 84.074 116.586)
+	)
 	(wire
 		(pts
@@
 	(wire
 		(pts
-			(xy 91.186 80.264) (xy 91.186 86.868)
-		)
-		(stroke
-			(width 0)
-			(type default)
-		)
-	)
-	(wire
-		(pts
 			(xy 83.566 97.282) (xy 84.328 98.044)
 		)
@@
 	(wire
 		(pts
+			(xy 91.186 86.106) (xy 91.186 89.662)
+		)
+		(stroke
+			(width 0)
+			(type default)
+		)
+	)
+	(wire
+		(pts
 			(xy 91.186 89.662) (xy 96.012 89.662)
 		)
@@
 	(wire
 		(pts
-			(xy 91.186 86.868) (xy 91.186 89.662)
+			(xy 91.186 80.264) (xy 91.186 86.106)
 		)
 		(stroke
@@
 	)
 	(symbol
+		(lib_id "Connector:TestPoint")
+		(at 91.186 86.106 90)
+		(unit 1)
+		(exclude_from_sim no)
+		(in_bom yes)
+		(on_board yes)
+		(dnp no)
+		(property "Reference" "TP4"
+			(at 82.804 88.646 0)
+			(effects
+				(font
+					(size 1.27 1.27)
+				)
+				(justify left)
+				(hide yes)
+			)
+		)
+		(property "Value" "Raw_TP"
+			(at 85.1154 88.646 0)
+			(effects
+				(font
+					(size 1.27 1.27)
+				)
+				(justify left)
+				(hide yes)
+			)
+		)
+		(property "Footprint" "TestPoint:TestPoint_THTPad_1.5x1.5mm_Drill0.7mm"
+			(at 91.186 81.026 0)
+			(effects
+				(font
+					(size 1.27 1.27)
+				)
+				(hide yes)
+			)
+		)
+		(property "Datasheet" "~"
+			(at 91.186 81.026 0)
+			(effects
+				(font
+					(size 1.27 1.27)
+				)
+				(hide yes)
+			)
+		)
+		(property "Description" ""
+			(at 91.186 86.106 0)
+			(effects
+				(font
+					(size 1.27 1.27)
+				)
+				(hide yes)
+			)
+		)
+		(property "Height" ""
+			(at 91.186 86.106 0)
+			(effects
+				(font
+					(size 1.27 1.27)
+				)
+				(hide yes)
+			)
+		)
+		(property "Inventory" ""
+			(at 91.186 86.106 0)
+			(effects
+				(font
+					(size 1.27 1.27)
+				)
+				(hide yes)
+			)
+		)
+		(property "Mfg" ""
+			(at 91.186 86.106 0)
+			(effects
+				(font
+					(size 1.27 1.27)
+				)
+				(hide yes)
+			)
+		)
+		(property "Mouser Part Number" ""
+			(at 91.186 86.106 0)
+			(effects
+				(font
+					(size 1.27 1.27)
+				)
+				(hide yes)
+			)
+		)
+		(property "Mouser Price/Stock" ""
+			(at 91.186 86.106 0)
+			(effects
+				(font
+					(size 1.27 1.27)
+				)
+				(hide yes)
+			)
+		)
+		(property "P/N" "~"
+			(at 91.186 86.106 0)
+			(effects
+				(font
+					(size 1.27 1.27)
+				)
+				(hide yes)
+			)
+		)
+		(property "PN" ""
+			(at 91.186 86.106 0)
+			(effects
+				(font
+					(size 1.27 1.27)
+				)
+				(hide yes)
+			)
+		)
+		(property "Sim.Device" ""
+			(at 91.186 86.106 0)
+			(effects
+				(font
+					(size 1.27 1.27)
+				)
+				(hide yes)
+			)
+		)
+		(property "p/n" ""
+			(at 91.186 86.106 0)
+			(effects
+				(font
+					(size 1.27 1.27)
+				)
+				(hide yes)
+			)
+		)
+		(pin "1"
+		)
+		(instances
+			(project "Controls-PedalsDaughter"
+				(path "/30d77876-714b-4f1b-9bad-b74eb43ddcf6/7d1ff2c9-efd0-48ce-add2-9372a4e6c13a/4f4b66ca-ebef-4dbc-af03-510cf70c75cb"
+					(reference "TP5")
+					(unit 1)
+				)
+				(path "/30d77876-714b-4f1b-9bad-b74eb43ddcf6/7d1ff2c9-efd0-48ce-add2-9372a4e6c13a/5ee0acff-6668-4939-819e-7e9025ec765c"
+					(reference "TP4")
+					(unit 1)
+				)
+			)
+		)
+	)
+	(symbol
 		(lib_id "power:GND")
 		(at 106.172 108.712 0)
@@
 					(unit 1)
 				)
-			)
-		)
-	)
-	(symbol
-		(lib_id "Connector:TestPoint")
-		(at 91.186 86.868 90)
-		(unit 1)
-		(exclude_from_sim no)
-		(in_bom yes)
-		(on_board yes)
-		(dnp no)
-		(property "Reference" "Brake_Fl_Sn_Raw1"
-			(at 87.63 84.582 90)
-			(effects
-				(font
-					(size 1.27 1.27)
-				)
-				(justify left)
-			)
-		)
-		(property "Value" "Brake_Fl_Sn_Raw_TP"
-			(at 87.122 86.614 90)
-			(effects
-				(font
-					(size 1.27 1.27)
-				)
-				(justify left)
-			)
-		)
-		(property "Footprint" "TestPoint:TestPoint_THTPad_1.5x1.5mm_Drill0.7mm"
-			(at 91.186 81.788 0)
-			(effects
-				(font
-					(size 1.27 1.27)
-				)
-				(hide yes)
-			)
-		)
-		(property "Datasheet" "~"
-			(at 91.186 81.788 0)
-			(effects
-				(font
-					(size 1.27 1.27)
-				)
-				(hide yes)
-			)
-		)
-		(property "Description" ""
-			(at 91.186 86.868 0)
-			(effects
-				(font
-					(size 1.27 1.27)
-				)
-				(hide yes)
-			)
-		)
-		(property "Height" ""
-			(at 91.186 86.868 0)
-			(effects
-				(font
-					(size 1.27 1.27)
-				)
-				(hide yes)
-			)
-		)
-		(property "Inventory" ""
-			(at 91.186 86.868 0)
-			(effects
-				(font
-					(size 1.27 1.27)
-				)
-				(hide yes)
-			)
-		)
-		(property "Mfg" ""
-			(at 91.186 86.868 0)
-			(effects
-				(font
-					(size 1.27 1.27)
-				)
-				(hide yes)
-			)
-		)
-		(property "Mouser Part Number" ""
-			(at 91.186 86.868 0)
-			(effects
-				(font
-					(size 1.27 1.27)
-				)
-				(hide yes)
-			)
-		)
-		(property "Mouser Price/Stock" ""
-			(at 91.186 86.868 0)
-			(effects
-				(font
-					(size 1.27 1.27)
-				)
-				(hide yes)
-			)
-		)
-		(property "P/N" "~"
-			(at 91.186 86.868 0)
-			(effects
-				(font
-					(size 1.27 1.27)
-				)
-				(hide yes)
-			)
-		)
-		(property "PN" ""
-			(at 91.186 86.868 0)
-			(effects
-				(font
-					(size 1.27 1.27)
-				)
-				(hide yes)
-			)
-		)
-		(property "Sim.Device" ""
-			(at 91.186 86.868 0)
-			(effects
-				(font
-					(size 1.27 1.27)
-				)
-				(hide yes)
-			)
-		)
-		(property "p/n" ""
-			(at 91.186 86.868 0)
-			(effects
-				(font
-					(size 1.27 1.27)
-				)
-				(hide yes)
-			)
-		)
-		(pin "1"
-		)
-		(instances
-			(project "Controls-PedalsDaughter"
-				(path "/30d77876-714b-4f1b-9bad-b74eb43ddcf6/7d1ff2c9-efd0-48ce-add2-9372a4e6c13a/4f4b66ca-ebef-4dbc-af03-510cf70c75cb"
-					(reference "Brake_Fl_Sn_Raw2")
-					(unit 1)
-				)
-				(path "/30d77876-714b-4f1b-9bad-b74eb43ddcf6/7d1ff2c9-efd0-48ce-add2-9372a4e6c13a/5ee0acff-6668-4939-819e-7e9025ec765c"
-					(reference "Brake_Fl_Sn_Raw1")
-					(unit 1)
-				)

Commit message: IM DONNEEEE
Parts:
- Brake_Fl_Sn1, TP4: footprint TestPoint:TestPoint_THTPad_1.5x1.5mm_Drill0.7mm -> TestPoint:TestPoint_Keystone_5005-5009_Compact
Changed lines of the file:
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@@
 			)
 		)
-		(property "Footprint" "TestPoint:TestPoint_THTPad_1.5x1.5mm_Drill0.7mm"
+		(property "Footprint" "TestPoint:TestPoint_Keystone_5005-5009_Compact"
 			(at 91.186 81.026 0)
 			(effects
@@
 			)
 		)
-		(property "Footprint" "TestPoint:TestPoint_THTPad_1.5x1.5mm_Drill0.7mm"
+		(property "Footprint" "TestPoint:TestPoint_Keystone_5005-5009_Compact"
 			(at 149.606 92.202 0)
 			(effects

Commit message: change VDDA to 3v3 on sch
Connections:
- net +VDDA renamed +3.3V
- net GNDA renamed GND
Other:
- note added: "Vout = G(Vin+ - Vin-) + (Vref1 +Vref2)/2 Vout = 200(ADC - 0) + (2.5) Vout = 200ADC Vout = [0.66v, 3.3v] ADC = [3.3mV, 16.5mV] Vref1 = Vref2 = GND = 0.0V G = 200"
- note removed: "Vout = G(Vin+ - Vin-) + (Vref1 +Vref2)/2 Vout = 200(ADC - 0) + (2.5) Vout = 200ADC Vout = [0.66v, 3.3v] ADC = [3.3mV, 16.5mV] Vref1 = Vref2 = GNDA = 0.0V G = 200"
Changed lines of the file:
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@@
 		)
 	)
-	(text "Vout = G(Vin+ - Vin-) + (Vref1 +Vref2)/2\nVout = 200(ADC - 0) + (2.5)\nVout = 200ADC\nVout = [0.66v, 3.3v]\n\nADC = [3.3mV, 16.5mV]\nVref1 = Vref2 = GNDA = 0.0V\nG = 200"
+	(text "Vout = G(Vin+ - Vin-) + (Vref1 +Vref2)/2\nVout = 200(ADC - 0) + (2.5)\nVout = 200ADC\nVout = [0.66v, 3.3v]\n\nADC = [3.3mV, 16.5mV]\nVref1 = Vref2 = GND = 0.0V\nG = 200"
 		(exclude_from_sim no)
 		(at 192.786 118.872 0)
@@
 			)
 		)
-		(property "Value" "+VDDA"
+		(property "Value" "+3.3V"
 			(at 102.362 78.232 0)
 			(effects
@@
 			)
 		)
-		(property "Value" "GNDA"
+		(property "Value" "GND"
 			(at 106.172 113.792 0)
 			(effects
@@
 			)
 		)
-		(property "Value" "GNDA"
+		(property "Value" "GND"
 			(at 91.186 105.283 0)
 			(effects
@@
 			)
 		)
-		(property "Value" "GNDA"
+		(property "Value" "GND"
 			(at 134.366 106.172 0)
 			(effects
