File: hardware/VCAT-PedalBoxPCB/OpAmpBuffer.kicad_sch (KiCad schematic)
At the start: 14 parts, among them U1 TLV9002QDRQ1

Commit message: mikea
Parts:
- R35, R36: value 100 -> 120
Changed lines of the file:
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@@
 			)
 		)
-		(property "Value" "100"
+		(property "Value" "120"
 			(at 194.818 109.474 90)
 			(effects
@@
 			)
 		)
-		(property "Value" "100"
+		(property "Value" "120"
 			(at 194.818 81.534 90)
 			(effects

Commit message: change VDDA to 3v3 on sch
Connections:
- net +VDDA renamed +3.3V
- net GNDA renamed GND
Changed lines of the file:
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@@
 			)
 		)
-		(property "Value" "+VDDA"
+		(property "Value" "+3.3V"
 			(at 84.328 80.264 0)
 			(effects
@@
 			)
 		)
-		(property "Value" "GNDA"
+		(property "Value" "GND"
 			(at 206.375 122.809 0)
 			(effects
@@
 			)
 		)
-		(property "Value" "GNDA"
+		(property "Value" "GND"
 			(at 206.375 94.869 0)
 			(effects
@@
 			)
 		)
-		(property "Value" "GNDA"
+		(property "Value" "GND"
 			(at 84.328 116.84 0)
 			(effects
@@
 			)
 		)
-		(property "Value" "GNDA"
+		(property "Value" "GND"
 			(at 130.683 97.155 0)
 			(effects
@@
 			)
 		)
-		(property "Value" "GNDA"
+		(property "Value" "GND"
 			(at 123.952 125.73 0)
 			(effects
